File: leds.sch (KiCad schematic (older format))
At the start: 4 parts

Commit message: Update leds.sch
Connections:
- net labels added: DSP_GPIO16
- net labels removed: DSP_GPIO
Changed lines of the file:
@@
 	7650 3650 7100 3650
 Text GLabel 7650 4100 2    50   Input ~ 0
-DSP_GPIO
+DSP_GPIO16
 Wire Wire Line
 	7650 3650 7650 4500
