File: MC-FO.sch (KiCad schematic (older format))
At the start: 9 parts, among them J1 DB25_Female

Commit message: pull down resistor footprint
Parts:
- R11, R12, R13, R14, R15, R16, R17, R18: footprint (none) -> Resistor_SMD:R_0603_1608Metric
Changed lines of the file:
@@
 F 0 "R11" H 2918 1996 50  0000 L CNN
 F 1 "10K" H 2918 1905 50  0000 L CNN
-F 2 "" H 2850 1950 50  0001 C CNN
+F 2 "Resistor_SMD:R_0603_1608Metric" H 2850 1950 50  0001 C CNN
 F 3 "~" H 2850 1950 50  0001 C CNN
 	1    2850 1950
@@
 F 0 "R12" H 2918 2946 50  0000 L CNN
 F 1 "10K" H 2918 2855 50  0000 L CNN
-F 2 "" H 2850 2900 50  0001 C CNN
+F 2 "Resistor_SMD:R_0603_1608Metric" H 2850 2900 50  0001 C CNN
 F 3 "~" H 2850 2900 50  0001 C CNN
 	1    2850 2900
@@
 F 0 "R13" H 2918 4046 50  0000 L CNN
 F 1 "10K" H 2918 3955 50  0000 L CNN
-F 2 "" H 2850 4000 50  0001 C CNN
+F 2 "Resistor_SMD:R_0603_1608Metric" H 2850 4000 50  0001 C CNN
 F 3 "~" H 2850 4000 50  0001 C CNN
 	1    2850 4000
@@
 F 0 "R14" H 2918 4996 50  0000 L CNN
 F 1 "10K" H 2918 4905 50  0000 L CNN
-F 2 "" H 2850 4950 50  0001 C CNN
+F 2 "Resistor_SMD:R_0603_1608Metric" H 2850 4950 50  0001 C CNN
 F 3 "~" H 2850 4950 50  0001 C CNN
 	1    2850 4950
@@
 F 0 "R15" H 2918 5996 50  0000 L CNN
 F 1 "10K" H 2918 5905 50  0000 L CNN
-F 2 "" H 2850 5950 50  0001 C CNN
+F 2 "Resistor_SMD:R_0603_1608Metric" H 2850 5950 50  0001 C CNN
 F 3 "~" H 2850 5950 50  0001 C CNN
 	1    2850 5950
@@
 F 0 "R16" H 2918 6946 50  0000 L CNN
 F 1 "10K" H 2918 6855 50  0000 L CNN
-F 2 "" H 2850 6900 50  0001 C CNN
+F 2 "Resistor_SMD:R_0603_1608Metric" H 2850 6900 50  0001 C CNN
 F 3 "~" H 2850 6900 50  0001 C CNN
 	1    2850 6900
@@
 F 0 "R17" H 4518 4996 50  0000 L CNN
 F 1 "10K" H 4518 4905 50  0000 L CNN
-F 2 "" H 4450 4950 50  0001 C CNN
+F 2 "Resistor_SMD:R_0603_1608Metric" H 4450 4950 50  0001 C CNN
 F 3 "~" H 4450 4950 50  0001 C CNN
 	1    4450 4950
@@
 F 0 "R18" H 4518 5996 50  0000 L CNN
 F 1 "10K" H 4518 5905 50  0000 L CNN
-F 2 "" H 4450 5950 50  0001 C CNN
+F 2 "Resistor_SMD:R_0603_1608Metric" H 4450 5950 50  0001 C CNN
 F 3 "~" H 4450 5950 50  0001 C CNN
 	1    4450 5950
