File: MC-FO/Detector_Circuits.sch (KiCad schematic (older format))
At the start: 8 parts, among them IC1 TLV3501AID, J1 IFE98

Commit message: moved FO Board to using hierarchical sheets
Connections:
- net labels added: Regulated_5V
- wire segments 43 -> 46
Changed lines of the file:
@@
 	7350 3500 7250 3500
 Wire Wire Line
-	5750 2400 6850 2400
+	5750 2400 6250 2400
 Wire Wire Line
 	6850 2450 6850 2400
@@
 Text Notes 8200 4150 0    50   ~ 0
 Is an additional opamp needed? The typical configuration includes \nthe one I placed in this schematic -- zach
+Text GLabel 6000 2000 0    50   Input ~ 0
+Regulated_5V
+Wire Wire Line
+	6000 2000 6250 2000
+Wire Wire Line
+	6250 2000 6250 2400
+Connection ~ 6250 2400
+Wire Wire Line
+	6250 2400 6850 2400
 $EndSCHEMATC
