File: MC-FO/Detector_Circuits.sch (KiCad schematic (older format))
At the start: 8 parts, among them U15 IFD97, U16 TLV3501AID

Commit message: Add files via upload
Parts:
- removed C55, C57: 0.1 uF, symbol Device:C_Small
- added C28, C30: 0.1 uF, symbol Device:C_Small
- added U17: 74LVC1G32SE-7, symbol Existing_IC_Models:74LVC1G32SE-7
- renumbered C56 to C29, R50 to R16, R51 to R17, R52 to R18, U15 to U16, U16 to U18
Connections:
- net labels removed: GND
- wire segments 40 -> 50
Other:
- note added: "added a 5V tolerant OR gate\nthat will output 3.3V so the\nsignal is safe for DSP"
- note removed: "could add a stage to make 3.3 v. or a different comparator. Or resistor devider"
- moved on the sheet: R18, U18
Changed lines of the file:
@@
 Detector CKT
 $Comp
-L Device:C_Small C57
-U 1 1 6171F0C9
+L Device:C_Small C30
+U 1 1 6178E7F5
 P 7350 2500
-AR Path="/6171C819/6171F0C9" Ref="C57"  Part="1"
-AR Path="/61724A08/6171F0C9" Ref="C62"  Part="1"
-F 0 "C57" H 7450 2550 50  0000 L CNN
+AR Path="/6171C819/6178E7F5" Ref="C30"  Part="1"
+AR Path="/61724A08/6178E7F5" Ref="C27"  Part="1"
+F 0 "C30" H 7450 2550 50  0000 L CNN
 F 1 "0.1 uF" H 7450 2450 50  0000 L CNN
 F 2 "" H 7350 2500 50  0001 C CNN
@@
 $EndComp
 $Comp
-L Device:C_Small C55
-U 1 1 61733718
+L Device:C_Small C28
+U 1 1 6178E7F6
 P 4700 2600
-AR Path="/6171C819/61733718" Ref="C55"  Part="1"
-AR Path="/61724A08/61733718" Ref="C60"  Part="1"
-F 0 "C55" H 4800 2650 50  0000 L CNN
+AR Path="/6171C819/6178E7F6" Ref="C28"  Part="1"
+AR Path="/61724A08/6178E7F6" Ref="C25"  Part="1"
+F 0 "C28" H 4800 2650 50  0000 L CNN
 F 1 "0.1 uF" H 4800 2550 50  0000 L CNN
 F 2 "" H 4700 2600 50  0001 C CNN
@@
 $EndComp
 $Comp
-L power:GND #PWR?
-U 1 1 61735A2B
-P 4950 2850
-AR Path="/6171C819/61735A2B" Ref="#PWR?"  Part="1"
-AR Path="/61724A08/61735A2B" Ref="#PWR?"  Part="1"
-F 0 "#PWR?" H 4950 2600 50  0001 C CNN
-F 1 "GND" H 4955 2677 50  0000 C CNN
-F 2 "" H 4950 2850 50  0001 C CNN
-F 3 "" H 4950 2850 50  0001 C CNN
-	1    4950 2850
-	1    0    0    -1
-$EndComp
-$Comp
-L power:GND #PWR?
-U 1 1 6173205B
-P 7350 2750
-AR Path="/6171C819/6173205B" Ref="#PWR?"  Part="1"
-AR Path="/61724A08/6173205B" Ref="#PWR?"  Part="1"
-F 0 "#PWR?" H 7350 2500 50  0001 C CNN
-F 1 "GND" H 7355 2577 50  0000 C CNN
-F 2 "" H 7350 2750 50  0001 C CNN
-F 3 "" H 7350 2750 50  0001 C CNN
-	1    7350 2750
-	1    0    0    -1
-$EndComp
-$Comp
-L Device:R_Small_US R50
+L Device:R_Small_US R16
 U 1 1 6174EB5A
 P 5750 3950
-AR Path="/6171C819/6174EB5A" Ref="R50"  Part="1"
-AR Path="/61724A08/6174EB5A" Ref="R60"  Part="1"
-F 0 "R50" H 5850 3900 50  0000 L CNN
+AR Path="/6171C819/6174EB5A" Ref="R16"  Part="1"
+AR Path="/61724A08/6174EB5A" Ref="R13"  Part="1"
+F 0 "R16" H 5850 3900 50  0000 L CNN
 F 1 "2.4 K" H 5850 4000 50  0000 L CNN
 F 2 "" H 5750 3950 50  0001 C CNN
@@
 $EndComp
 $Comp
-L Device:CP1_Small C56
+L Device:CP1_Small C29
 U 1 1 61720E6A
 P 5200 2600
-AR Path="/6171C819/61720E6A" Ref="C56"  Part="1"
-AR Path="/61724A08/61720E6A" Ref="C61"  Part="1"
-F 0 "C56" H 5291 2646 50  0000 L CNN
+AR Path="/6171C819/61720E6A" Ref="C29"  Part="1"
+AR Path="/61724A08/61720E6A" Ref="C26"  Part="1"
+F 0 "C29" H 5291 2646 50  0000 L CNN
 F 1 "10 uF" H 5291 2555 50  0000 L CNN
 F 2 "" H 5200 2600 50  0001 C CNN
@@
 	4700 2400 5200 2400
 Wire Wire Line
-	4950 2850 5200 2850
-Wire Wire Line
-	4950 2850 4700 2850
-Wire Wire Line
 	4700 2850 4700 2700
-Connection ~ 4950 2850
-$Comp
-L power:GND #PWR?
-U 1 1 6174213D
-P 6650 4100
-AR Path="/6171C819/6174213D" Ref="#PWR?"  Part="1"
-AR Path="/61724A08/6174213D" Ref="#PWR?"  Part="1"
-F 0 "#PWR?" H 6650 3850 50  0001 C CNN
-F 1 "GND" H 6655 3927 50  0000 C CNN
-F 2 "" H 6650 4100 50  0001 C CNN
-F 3 "" H 6650 4100 50  0001 C CNN
-	1    6650 4100
-	1    0    0    -1
-$EndComp
-$Comp
-L Device:R_Small_US R51
+$Comp
+L Device:R_Small_US R17
 U 1 1 617451F8
 P 5750 4900
-AR Path="/6171C819/617451F8" Ref="R51"  Part="1"
-AR Path="/61724A08/617451F8" Ref="R61"  Part="1"
-F 0 "R51" H 5850 4850 50  0000 L CNN
+AR Path="/6171C819/617451F8" Ref="R17"  Part="1"
+AR Path="/61724A08/617451F8" Ref="R14"  Part="1"
+F 0 "R17" H 5850 4850 50  0000 L CNN
 F 1 "1 K" H 5850 4950 50  0000 L CNN
 F 2 "" H 5750 4900 50  0001 C CNN
@@
 $EndComp
 $Comp
-L Device:R_Small_US R52
+L Device:R_Small_US R18
 U 1 1 61745A42
-P 7050 4600
-AR Path="/6171C819/61745A42" Ref="R52"  Part="1"
-AR Path="/61724A08/61745A42" Ref="R62"  Part="1"
-F 0 "R52" V 7250 4550 50  0000 L CNN
-F 1 "47 K" V 7150 4550 50  0000 L CNN
-F 2 "" H 7050 4600 50  0001 C CNN
-F 3 "~" H 7050 4600 50  0001 C CNN
-	1    7050 4600
+P 7050 4650
+AR Path="/6171C819/61745A42" Ref="R18"  Part="1"
+AR Path="/61724A08/61745A42" Ref="R15"  Part="1"
+F 0 "R18" V 7250 4600 50  0000 L CNN
+F 1 "47 K" V 7150 4600 50  0000 L CNN
+F 2 "" H 7050 4650 50  0001 C CNN
+F 3 "~" H 7050 4650 50  0001 C CNN
+	1    7050 4650
 	0    -1   -1   0
 $EndComp
@@
 	5750 5150 5750 5000
 Wire Wire Line
-	5750 4800 5750 4600
-Wire Wire Line
-	5750 4600 5750 4050
-Connection ~ 5750 4600
-Wire Wire Line
-	5750 2400 5750 3850
+	5750 4800 5750 4650
+Wire Wire Line
+	5750 4650 5750 4050
+Connection ~ 5750 4650
+Wire Wire Line
+	5750 2400 5750 3000
 Wire Wire Line
 	5200 2400 5750 2400
@@
 Wire Wire Line
 	4300 3600 4300 3700
-$Comp
-L power:GND #PWR?
-U 1 1 6176C799
-P 4300 3700
-AR Path="/6171C819/6176C799" Ref="#PWR?"  Part="1"
-AR Path="/61724A08/6176C799" Ref="#PWR?"  Part="1"
-F 0 "#PWR?" H 4300 3450 50  0001 C CNN
-F 1 "GND" H 4305 3527 50  0000 C CNN
-F 2 "" H 4300 3700 50  0001 C CNN
-F 3 "" H 4300 3700 50  0001 C CNN
-	1    4300 3700
-	1    0    0    -1
-$EndComp
 Wire Wire Line
 	4300 2400 4300 3300
@@
 	6250 2400 6700 2400
 Wire Wire Line
-	6700 3300 6700 2400
+	6700 3350 6700 2400
 Connection ~ 6700 2400
 Wire Wire Line
 	6700 2400 7350 2400
-Connection ~ 6200 4600
-Wire Wire Line
-	6200 4600 6950 4600
-Wire Wire Line
-	5750 4600 6200 4600
-Wire Wire Line
-	7800 3600 8100 3600
-Wire Wire Line
-	6200 3600 6450 3600
-Wire Wire Line
-	6200 3600 6200 4600
-Wire Wire Line
-	7800 4600 7800 3600
-Wire Wire Line
-	7150 4600 7800 4600
-Wire Wire Line
-	7100 3600 7800 3600
-$Comp
-L Existing_IC_Models:IFD97 U15
+Connection ~ 6200 4650
+Wire Wire Line
+	6200 4650 6950 4650
+Wire Wire Line
+	5750 4650 6200 4650
+Wire Wire Line
+	7800 3650 8100 3650
+Wire Wire Line
+	6200 3650 6450 3650
+Wire Wire Line
+	6200 3650 6200 4650
+Wire Wire Line
+	7800 4650 7800 3650
+Wire Wire Line
+	7150 4650 7800 4650
+Wire Wire Line
+	7100 3650 7800 3650
+$Comp
+L Existing_IC_Models:IFD97 U16
 U 1 1 61758365
 P 3700 3900
-AR Path="/6171C819/61758365" Ref="U15"  Part="1"
-AR Path="/61724A08/61758365" Ref="U17"  Part="1"
-F 0 "U15" H 3700 4715 50  0000 C CNN
+AR Path="/6171C819/61758365" Ref="U16"  Part="1"
+AR Path="/61724A08/61758365" Ref="U13"  Part="1"
+F 0 "U16" H 3700 4715 50  0000 C CNN
 F 1 "IFD97" H 3700 4624 50  0000 C CNN
 F 2 "" H 3700 4700 50  0001 C CNN
@@
 	1    0    0    -1
 $EndComp
-Text HLabel 8100 3600 2    50   Input ~ 0
+Text HLabel 8100 3650 2    50   Input ~ 0
 DPWM
-Text Notes 10650 3250 2    50   ~ 0
-could add a stage to make 3.3 v. or a different comparator. Or resistor devider
 Text HLabel 6000 2000 0    50   Input ~ 0
 5V
-Wire Wire Line
-	4000 3500 6450 3500
-$Comp
-L Existing_IC_Models:TLV3501AID U16
+$Comp
+L Existing_IC_Models:TLV3501AID U18
 U 1 1 61744BAA
-P 6600 3900
-AR Path="/6171C819/61744BAA" Ref="U16"  Part="1"
-AR Path="/61724A08/61744BAA" Ref="U18"  Part="1"
-F 0 "U16" H 7100 3800 50  0000 L CNN
-F 1 "TLV3501AID" H 6950 3700 50  0000 L CNN
-F 2 "" H 6600 3900 50  0001 C CNN
-F 3 "" H 6600 3900 50  0001 C CNN
-	1    6600 3900
+P 6600 3950
+AR Path="/6171C819/61744BAA" Ref="U18"  Part="1"
+AR Path="/61724A08/61744BAA" Ref="U15"  Part="1"
+F 0 "U18" H 7100 3850 50  0000 L CNN
+F 1 "TLV3501AID" H 6950 3750 50  0000 L CNN
+F 2 "" H 6600 3950 50  0001 C CNN
+F 3 "" H 6600 3950 50  0001 C CNN
+	1    6600 3950
 	1    0    0    1
 $EndComp
 Wire Wire Line
-	6800 3800 6800 4000
-Wire Wire Line
-	6800 4000 6650 4000
-Wire Wire Line
-	6650 4000 6650 4100
-Wire Wire Line
-	6650 3900 6650 4000
-Connection ~ 6650 4000
-Connection ~ 7800 3600
-Wire Wire Line
-	7800 3600 7800 3550
+	6800 3850 6800 4050
+Wire Wire Line
+	6800 4050 6650 4050
+Wire Wire Line
+	6650 4050 6650 4150
+Wire Wire Line
+	6650 3950 6650 4050
+Connection ~ 6650 4050
+Connection ~ 7800 3650
+Wire Wire Line
+	7800 3650 7800 3600
 Text HLabel 5750 5150 3    50   Input ~ 0
 GND2
+$Comp
+L Existing_IC_Models:74LVC1G32SE-7 U17
+U 1 1 6177D138
+P 5100 3550
+AR Path="/6171C819/6177D138" Ref="U17"  Part="1"
+AR Path="/61724A08/6177D138" Ref="U14"  Part="1"
+F 0 "U17" H 5400 3800 50  0000 C CNN
+F 1 "74LVC1G32SE-7" H 5400 3700 50  0000 C CNN
+F 2 "" H 5100 3550 50  0001 C CNN
+F 3 "http://www.ti.com/lit/sg/scyt129e/scyt129e.pdf" H 5100 3550 50  0001 C CNN
+	1    5100 3550
+	1    0    0    -1
+$EndComp
+Wire Wire Line
+	4000 3500 4800 3500
+Wire Wire Line
+	5100 3650 5100 3850
+Wire Wire Line
+	5100 3850 4800 3850
+Wire Wire Line
+	4800 3850 4800 3600
+Wire Wire Line
+	5100 3850 5100 4000
+Connection ~ 5100 3850
+Text HLabel 5100 4000 0    50   Input ~ 0
+GND2
+Wire Wire Line
+	5350 3550 6450 3550
+Text HLabel 6650 4150 0    50   Input ~ 0
+GND2
+Wire Wire Line
+	5750 3000 5100 3000
+Wire Wire Line
+	5100 3000 5100 3450
+Connection ~ 5750 3000
+Wire Wire Line
+	5750 3000 5750 3850
+Text HLabel 4950 2900 3    50   Input ~ 0
+GND2
+Text HLabel 4300 3700 0    50   Input ~ 0
+GND2
+Text HLabel 7300 2750 0    50   Input ~ 0
+GND2
+Wire Wire Line
+	7300 2750 7350 2750
+Text Notes 4050 4400 0    50   ~ 0
+added a 5V tolerant OR gate\nthat will output 3.3V so the\nsignal is safe for DSP
+Wire Wire Line
+	4700 2850 4950 2850
+Wire Wire Line
+	4950 2850 4950 2900
+Connection ~ 4950 2850
+Wire Wire Line
+	4950 2850 5200 2850
 $EndSCHEMATC

Commit message: a few more FO tweaks 10-26
Parts:
- C28, C29, C30: footprint (none) -> Capacitor_SMD:C_0603_1608Metric
Changed lines of the file:
@@
 F 0 "C30" H 7450 2550 50  0000 L CNN
 F 1 "0.1 uF" H 7450 2450 50  0000 L CNN
-F 2 "" H 7350 2500 50  0001 C CNN
+F 2 "Capacitor_SMD:C_0603_1608Metric" H 7350 2500 50  0001 C CNN
 F 3 "~" H 7350 2500 50  0001 C CNN
 	1    7350 2500
@@
 F 0 "C28" H 4800 2650 50  0000 L CNN
 F 1 "0.1 uF" H 4800 2550 50  0000 L CNN
-F 2 "" H 4700 2600 50  0001 C CNN
+F 2 "Capacitor_SMD:C_0603_1608Metric" H 4700 2600 50  0001 C CNN
 F 3 "~" H 4700 2600 50  0001 C CNN
 	1    4700 2600
@@
 F 0 "C29" H 5291 2646 50  0000 L CNN
 F 1 "10 uF" H 5291 2555 50  0000 L CNN
-F 2 "" H 5200 2600 50  0001 C CNN
+F 2 "Capacitor_SMD:C_0603_1608Metric" H 5200 2600 50  0001 C CNN
 F 3 "~" H 5200 2600 50  0001 C CNN
 	1    5200 2600

Commit message: added footprints and reference
Parts:
- R16, R17, R18: footprint (none) -> Resistor_SMD:R_0603_1608Metric
- U16: footprint (none) -> Footprints_MC-FO:IFD97
- U17: footprint (none) -> Package_TO_SOT_SMD:SOT-353_SC-70-5_Handsoldering
- U18: footprint (none) -> Package_SO:SOIC-8_3.9x4.9mm_P1.27mm
Changed lines of the file:
@@
 F 0 "R16" H 5850 3900 50  0000 L CNN
 F 1 "2.4 K" H 5850 4000 50  0000 L CNN
-F 2 "" H 5750 3950 50  0001 C CNN
+F 2 "Resistor_SMD:R_0603_1608Metric" H 5750 3950 50  0001 C CNN
 F 3 "~" H 5750 3950 50  0001 C CNN
 	1    5750 3950
@@
 F 0 "R17" H 5850 4850 50  0000 L CNN
 F 1 "1 K" H 5850 4950 50  0000 L CNN
-F 2 "" H 5750 4900 50  0001 C CNN
+F 2 "Resistor_SMD:R_0603_1608Metric" H 5750 4900 50  0001 C CNN
 F 3 "~" H 5750 4900 50  0001 C CNN
 	1    5750 4900
@@
 F 0 "R18" V 7250 4600 50  0000 L CNN
 F 1 "47 K" V 7150 4600 50  0000 L CNN
-F 2 "" H 7050 4650 50  0001 C CNN
+F 2 "Resistor_SMD:R_0603_1608Metric" H 7050 4650 50  0001 C CNN
 F 3 "~" H 7050 4650 50  0001 C CNN
 	1    7050 4650
@@
 F 0 "U16" H 3700 4715 50  0000 C CNN
 F 1 "IFD97" H 3700 4624 50  0000 C CNN
-F 2 "" H 3700 4700 50  0001 C CNN
+F 2 "Footprints_MC-FO:IFD97" H 3700 4700 50  0001 C CNN
 F 3 "" H 3700 4700 50  0001 C CNN
 	1    3700 3900
@@
 F 0 "U18" H 7100 3850 50  0000 L CNN
 F 1 "TLV3501AID" H 6950 3750 50  0000 L CNN
-F 2 "" H 6600 3950 50  0001 C CNN
+F 2 "Package_SO:SOIC-8_3.9x4.9mm_P1.27mm" H 6600 3950 50  0001 C CNN
 F 3 "" H 6600 3950 50  0001 C CNN
 	1    6600 3950
@@
 F 0 "U17" H 5400 3800 50  0000 C CNN
 F 1 "74LVC1G32SE-7" H 5400 3700 50  0000 C CNN
-F 2 "" H 5100 3550 50  0001 C CNN
+F 2 "Package_TO_SOT_SMD:SOT-353_SC-70-5_Handsoldering" H 5100 3550 50  0001 C CNN
 F 3 "http://www.ti.com/lit/sg/scyt129e/scyt129e.pdf" H 5100 3550 50  0001 C CNN
 	1    5100 3550
