File: MC-FO/Detector_Circuits.sch (KiCad schematic (older format))
At the start: 11 parts, among them U141 IFD97, U142 TLV3501AID, U143 74LVC1G32SE-7

Commit message: Add files via upload
Parts:
- removed C144: 0.1 uF, Capacitor_SMD:C_0603_1608Metric, symbol Device:C_Small
- removed R141: 2.4K, Resistor_SMD:R_0603_1608Metric, symbol Device:R_Small_US
- removed R142: 1K, Resistor_SMD:R_0603_1608Metric, symbol Device:R_Small_US
- removed R143: 10K, Resistor_SMD:R_0603_1608Metric, symbol Device:R_Small_US
- removed R144: 47K, Resistor_SMD:R_0603_1608Metric, symbol Device:R_Small_US
- removed U141: IFD97, Footprints_MC-FO:IFE98, symbol Existing_IC_Models:IFD97
- removed U142: TLV3501AID, Package_SO:SOIC-8_3.9x4.9mm_P1.27mm, symbol Existing_IC_Models:TLV3501AID
- removed U143: 74LVC1G32SE-7, Package_TO_SOT_SMD:SOT-353_SC-70-5, symbol Existing_IC_Models:74LVC1G32SE-7
- added R161: 2.4K, Resistor_SMD:R_0603_1608Metric, symbol Device:R_Small_US
- added R162: 47K, Resistor_SMD:R_0603_1608Metric, symbol Device:R_Small_US
- added R163: 10K, Resistor_SMD:R_0603_1608Metric, symbol Device:R_Small_US
- added U?: IFD97, Footprints_MC-FO:IFE98, symbol Existing_IC_Models:IFD97
- added U?: 74LVC1G32SE-7, Package_TO_SOT_SMD:SOT-353_SC-70-5, symbol Existing_IC_Models:74LVC1G32SE-7
Connections:
- net 5V: now also U?.4 (Vcc); no longer C143.1
- net GND: now also R163.2, U?.1 (GND), U?.2 (B), U?.3 (GND), U?.3 (GND)
- net VCC: now also C143.1, U?.5 (VCC)
- new net: R161.1, U?.2 (Q)
- new net: R161.2, R162.2, U?.1 (A)
- new net STATUS1_gpio: R162.1, R163.1, U?.4 (Y)
Other:
- note removed: "added a 5V tolerant(at logic input) OR gate to output\nof the comparator that will output 3.3V signal to DSP\n\n"
- note removed: "on one detector do or gate and the other using the comparator"
