File: MC-FO/Emitter_Circuits.sch (KiCad schematic (older format))
At the start: 9 parts, among them IC1 74ACT08SCX, J1 IFE98, U1 OPA356xxD

Commit message: moved FO Board to using hierarchical sheets
Parts:
- U1: renamed from IC1; Arrow Part Number 74ACT08SCX -> (none); Arrow Price/Stock https://www.arrow.com/en/products/74act08scx/on-semiconduct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 -> (none); Description AND Gate Quad 2 Input CMOS SOIC14 -> (none); Height 1.75 -> (none); Manufacturer_Name ON Semiconductor -> (none); Manufacturer_Part_Number 74ACT08SCX -> (none); Mouser Part Number 512-74ACT08SCX -> (none); Mouser Price/Stock https://www.mouser.com/Search/Refine.aspx?Keyword=512-74ACT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 -> (none)
- renumbered C1 to C11, C2 to C12, C3 to C13, C4 to C14, J1 to J?, R1 to R?, R2 to R?, U1 to U?
Connections:
- net labels added: 3V3, 5V, EPWM
- net labels removed: EPWM1A, Regulated_3.3V, Regulated_5V
Other:
- note removed: "Unsure of MH1 pin purpose"
Changed lines of the file:
@@
 $Descr A4 11693 8268
 encoding utf-8
-Sheet 1 1
+Sheet 2 6
 Title ""
 Date ""
@@
 Comment4 ""
 $EndDescr
-Text Notes 5350 5600 0    50   ~ 10
+Text Notes 5350 5450 0    50   ~ 10
 Emitter CKT
 Wire Wire Line
@@
 U 1 1 617046FE
 P 3100 5250
+AR Path="/61717EAF/617046FE" Ref="#PWR?"  Part="1"
+AR Path="/617509F7/617046FE" Ref="#PWR?"  Part="1"
+AR Path="/61750A2A/617046FE" Ref="#PWR?"  Part="1"
 F 0 "#PWR?" H 3100 5000 50  0001 C CNN
 F 1 "GND" H 3105 5077 50  0000 C CNN
@@
 $EndComp
 $Comp
-L Amplifier_Operational:OPA356xxD U1
+L Amplifier_Operational:OPA356xxD U?
 U 1 1 617059F7
 P 3200 4950
-F 0 "U1" H 3150 5250 50  0000 L CNN
+AR Path="/61717EAF/617059F7" Ref="U?"  Part="1"
+AR Path="/617509F7/617059F7" Ref="U?"  Part="1"
+AR Path="/61750A2A/617059F7" Ref="U?"  Part="1"
+F 0 "U?" H 3150 5250 50  0000 L CNN
 F 1 "OPA356xxD" H 3150 5150 50  0000 L CNN
 F 2 "Package_SO:SOIC-8_3.9x4.9mm_P1.27mm" H 3100 4750 50  0001 L CNN
@@
 	1    0    0    -1
 $EndComp
-Text GLabel 2950 4600 0    50   Input ~ 0
-Regulated_3.3V
 Wire Wire Line
 	2950 4600 3100 4600
@@
 U 1 1 61717683
 P 4950 4750
+AR Path="/61717EAF/61717683" Ref="#PWR?"  Part="1"
+AR Path="/617509F7/61717683" Ref="#PWR?"  Part="1"
+AR Path="/61750A2A/61717683" Ref="#PWR?"  Part="1"
 F 0 "#PWR?" H 4950 4500 50  0001 C CNN
 F 1 "GND" H 4955 4577 50  0000 C CNN
@@
 	4700 3800 4700 3950
 $Comp
-L Device:C_Small C1
+L Device:C_Small C11
 U 1 1 6171F0C9
 P 4700 4050
-F 0 "C1" H 4750 3950 50  0000 L CNN
+AR Path="/61717EAF/6171F0C9" Ref="C11"  Part="1"
+AR Path="/617509F7/6171F0C9" Ref="C21"  Part="1"
+AR Path="/61750A2A/6171F0C9" Ref="C?"  Part="1"
+F 0 "C11" H 4750 3950 50  0000 L CNN
 F 1 "0.1 uF" H 4750 3850 50  0000 L CNN
 F 2 "" H 4700 4050 50  0001 C CNN
@@
 Text Notes 2700 4400 0    50   ~ 0
 Unity Gain Buffer
-Text GLabel 2050 4850 0    50   Input ~ 0
-EPWM1A
 Wire Wire Line
 	2900 4850 2050 4850
@@
 Wire Wire Line
 	4400 4600 4450 4600
-Text GLabel 4300 4600 0    50   Input ~ 0
-Regulated_5V
-$Comp
-L Device:C_Small C2
+$Comp
+L Device:C_Small C12
 U 1 1 61730A88
 P 5750 3150
-F 0 "C2" H 5800 3050 50  0000 L CNN
+AR Path="/61717EAF/61730A88" Ref="C12"  Part="1"
+AR Path="/617509F7/61730A88" Ref="C22"  Part="1"
+AR Path="/61750A2A/61730A88" Ref="C?"  Part="1"
+F 0 "C12" H 5800 3050 50  0000 L CNN
 F 1 "10 uF" H 5800 2950 50  0000 L CNN
 F 2 "" H 5750 3150 50  0001 C CNN
@@
 	5750 3000 5750 3050
 $Comp
-L Device:C_Small C3
+L Device:C_Small C13
 U 1 1 61733718
 P 6150 3150
-F 0 "C3" H 6200 3050 50  0000 L CNN
+AR Path="/61717EAF/61733718" Ref="C13"  Part="1"
+AR Path="/617509F7/61733718" Ref="C23"  Part="1"
+AR Path="/61750A2A/61733718" Ref="C?"  Part="1"
+F 0 "C13" H 6200 3050 50  0000 L CNN
 F 1 "0.1 uF" H 6200 2950 50  0000 L CNN
 F 2 "" H 6150 3150 50  0001 C CNN
@@
 U 1 1 61735A2B
 P 5950 3500
+AR Path="/61717EAF/61735A2B" Ref="#PWR?"  Part="1"
+AR Path="/617509F7/61735A2B" Ref="#PWR?"  Part="1"
+AR Path="/61750A2A/61735A2B" Ref="#PWR?"  Part="1"
 F 0 "#PWR?" H 5950 3250 50  0001 C CNN
 F 1 "GND" H 5955 3327 50  0000 C CNN
@@
 	6150 3050 6150 3000
 $Comp
-L IFE98:IFE98 J1
+L IFE98:IFE98 J?
 U 1 1 61710D71
 P 7700 4250
-F 0 "J1" H 8200 4515 50  0000 C CNN
+AR Path="/61717EAF/61710D71" Ref="J?"  Part="1"
+AR Path="/617509F7/61710D71" Ref="J?"  Part="1"
+AR Path="/61750A2A/61710D71" Ref="J?"  Part="1"
+F 0 "J?" H 8200 4515 50  0000 C CNN
 F 1 "IFE98" H 8200 4424 50  0000 C CNN
 F 2 "IFE98" H 8550 4350 50  0001 L CNN
@@
 $EndComp
 $Comp
-L 74ACT08SCX:74ACT08SCX IC1
+L 74ACT08SCX:74ACT08SCX U1
 U 1 1 61717F3E
 P 5100 4150
-F 0 "IC1" H 5600 4415 50  0000 C CNN
+AR Path="/61717EAF/61717F3E" Ref="U1"  Part="1"
+AR Path="/617509F7/61717F3E" Ref="U2"  Part="1"
+AR Path="/61750A2A/61717F3E" Ref="U3"  Part="1"
+F 0 "U1" H 5600 4415 50  0000 C CNN
 F 1 "74ACT08SCX" H 5600 4324 50  0000 C CNN
 F 2 "SOIC127P600X175-14N" H 5950 4250 50  0001 L CNN
 F 3 "http://docs-emea.rs-online.com/webdocs/0f9a/0900766b80f9a397.pdf" H 5950 4150 50  0001 L CNN
-F 4 "AND Gate Quad 2 Input CMOS SOIC14" H 5950 4050 50  0001 L CNN "Description"
-F 5 "1.75" H 5950 3950 50  0001 L CNN "Height"
-F 6 "ON Semiconductor" H 5950 3850 50  0001 L CNN "Manufacturer_Name"
-F 7 "74ACT08SCX" H 5950 3750 50  0001 L CNN "Manufacturer_Part_Number"
-F 8 "512-74ACT08SCX" H 5950 3650 50  0001 L CNN "Mouser Part Number"
-F 9 "https://www.mouser.com/Search/Refine.aspx?Keyword=512-74ACT08SCX" H 5950 3550 50  0001 L CNN "Mouser Price/Stock"
-F 10 "74ACT08SCX" H 5950 3450 50  0001 L CNN "Arrow Part Number"
-F 11 "https://www.arrow.com/en/products/74act08scx/on-semiconductor" H 5950 3350 50  0001 L CNN "Arrow Price/Stock"
 	1    5100 4150
 	1    0    0    -1
@@
 U 1 1 6173205B
 P 4700 4350
+AR Path="/61717EAF/6173205B" Ref="#PWR?"  Part="1"
+AR Path="/617509F7/6173205B" Ref="#PWR?"  Part="1"
+AR Path="/61750A2A/6173205B" Ref="#PWR?"  Part="1"
 F 0 "#PWR?" H 4700 4100 50  0001 C CNN
 F 1 "GND" H 4705 4177 50  0000 C CNN
@@
 	6400 4250 6400 5050
 $Comp
-L Device:R_Small_US R1
+L Device:R_Small_US R?
 U 1 1 617428A7
 P 6700 4450
-F 0 "R1" V 6900 4450 50  0000 L CNN
+AR Path="/61717EAF/617428A7" Ref="R?"  Part="1"
+AR Path="/617509F7/617428A7" Ref="R?"  Part="1"
+AR Path="/61750A2A/617428A7" Ref="R?"  Part="1"
+F 0 "R?" V 6900 4450 50  0000 L CNN
 F 1 "150 Ohm" V 6800 4200 50  0000 L CNN
 F 2 "" H 6700 4450 50  0001 C CNN
@@
 	6100 4450 6500 4450
 $Comp
-L Device:C_Small C4
+L Device:C_Small C14
 U 1 1 61748E58
 P 6700 4800
-F 0 "C4" V 6900 4800 50  0000 L CNN
+AR Path="/61717EAF/61748E58" Ref="C14"  Part="1"
+AR Path="/617509F7/61748E58" Ref="C24"  Part="1"
+AR Path="/61750A2A/61748E58" Ref="C?"  Part="1"
+F 0 "C14" V 6900 4800 50  0000 L CNN
 F 1 "100 pF" V 6800 4650 50  0000 L CNN
 F 2 "" H 6700 4800 50  0001 C CNN
@@
 	6950 4450 6800 4450
 $Comp
-L Device:R_Small_US R2
+L Device:R_Small_US R?
 U 1 1 6174EB5A
 P 7300 3300
-F 0 "R2" H 7400 3250 50  0000 L CNN
+AR Path="/61717EAF/6174EB5A" Ref="R?"  Part="1"
+AR Path="/617509F7/6174EB5A" Ref="R?"  Part="1"
+AR Path="/61750A2A/6174EB5A" Ref="R?"  Part="1"
+F 0 "R?" H 7400 3250 50  0000 L CNN
 F 1 "365 Ohm" H 7400 3350 50  0000 L CNN
 F 2 "" H 7300 3300 50  0001 C CNN
@@
 U 1 1 6175F75B
 P 7500 4750
+AR Path="/61717EAF/6175F75B" Ref="#PWR?"  Part="1"
+AR Path="/617509F7/6175F75B" Ref="#PWR?"  Part="1"
+AR Path="/61750A2A/6175F75B" Ref="#PWR?"  Part="1"
 F 0 "#PWR?" H 7500 4500 50  0001 C CNN
 F 1 "GND" H 7505 4577 50  0000 C CNN
@@
 Wire Wire Line
 	7300 4450 7700 4450
-Text Notes 8800 4300 0    50   ~ 0
-Unsure of MH1 pin purpose
+Text GLabel 4300 4600 0    50   Input ~ 0
+5V
+Text GLabel 2950 4600 0    50   Input ~ 0
+3V3
+Text HLabel 2050 4850 0    50   Input ~ 0
+EPWM
 $EndSCHEMATC

Commit message: Add files via upload
Parts:
- removed U?: OPA356xxD, Package_SO:SOIC-8_3.9x4.9mm_P1.27mm, symbol Amplifier_Operational:OPA356xxD
Connections:
- net labels removed: 3V3
- wire segments 53 -> 44
Other:
- note removed: "Unity Gain Buffer"
Changed lines of the file:
@@
 $Descr A4 11693 8268
 encoding utf-8
-Sheet 2 6
+Sheet 5 12
 Title ""
 Date ""
@@
 Text Notes 5350 5450 0    50   ~ 10
 Emitter CKT
-Wire Wire Line
-	3500 4950 3500 5500
-Wire Wire Line
-	3500 5500 2650 5500
-Wire Wire Line
-	2650 5500 2650 5050
-Wire Wire Line
-	2650 5050 2900 5050
-$Comp
-L power:GND #PWR?
-U 1 1 617046FE
-P 3100 5250
-AR Path="/61717EAF/617046FE" Ref="#PWR?"  Part="1"
-AR Path="/617509F7/617046FE" Ref="#PWR?"  Part="1"
-AR Path="/61750A2A/617046FE" Ref="#PWR?"  Part="1"
-F 0 "#PWR?" H 3100 5000 50  0001 C CNN
-F 1 "GND" H 3105 5077 50  0000 C CNN
-F 2 "" H 3100 5250 50  0001 C CNN
-F 3 "" H 3100 5250 50  0001 C CNN
-	1    3100 5250
-	1    0    0    -1
-$EndComp
-$Comp
-L Amplifier_Operational:OPA356xxD U?
-U 1 1 617059F7
-P 3200 4950
-AR Path="/61717EAF/617059F7" Ref="U?"  Part="1"
-AR Path="/617509F7/617059F7" Ref="U?"  Part="1"
-AR Path="/61750A2A/617059F7" Ref="U?"  Part="1"
-F 0 "U?" H 3150 5250 50  0000 L CNN
-F 1 "OPA356xxD" H 3150 5150 50  0000 L CNN
-F 2 "Package_SO:SOIC-8_3.9x4.9mm_P1.27mm" H 3100 4750 50  0001 L CNN
-F 3 "http://www.ti.com/lit/ds/symlink/opa356.pdf" H 3350 5100 50  0001 C CNN
-	1    3200 4950
-	1    0    0    -1
-$EndComp
-Wire Wire Line
-	2950 4600 3100 4600
 $Comp
 L power:GND #PWR?
@@
 AR Path="/617509F7/61717683" Ref="#PWR?"  Part="1"
 AR Path="/61750A2A/61717683" Ref="#PWR?"  Part="1"
+AR Path="/6176CA10/61717683" Ref="#PWR?"  Part="1"
+AR Path="/6176CA81/61717683" Ref="#PWR?"  Part="1"
+AR Path="/6176CAE4/61717683" Ref="#PWR?"  Part="1"
 F 0 "#PWR?" H 4950 4500 50  0001 C CNN
 F 1 "GND" H 4955 4577 50  0000 C CNN
@@
 	1    0    0    -1
 $EndComp
-Wire Wire Line
-	3500 4950 4350 4950
-Connection ~ 3500 4950
 Wire Wire Line
 	4400 4600 4400 5000
@@
 AR Path="/617509F7/6171F0C9" Ref="C21"  Part="1"
 AR Path="/61750A2A/6171F0C9" Ref="C?"  Part="1"
-F 0 "C11" H 4750 3950 50  0000 L CNN
+AR Path="/6176CA10/6171F0C9" Ref="C?"  Part="1"
+AR Path="/6176CA81/6171F0C9" Ref="C?"  Part="1"
+AR Path="/6176CAE4/6171F0C9" Ref="C?"  Part="1"
+F 0 "C?" H 4750 3950 50  0000 L CNN
 F 1 "0.1 uF" H 4750 3850 50  0000 L CNN
 F 2 "" H 4700 4050 50  0001 C CNN
@@
 Wire Wire Line
 	4700 4150 4700 4350
-Wire Wire Line
-	3100 4600 3100 4650
-Wire Notes Line
-	2250 4450 2250 5650
-Wire Notes Line
-	2250 5650 3700 5650
-Wire Notes Line
-	3700 5650 3700 4450
-Wire Notes Line
-	3700 4450 2250 4450
-Text Notes 2700 4400 0    50   ~ 0
-Unity Gain Buffer
-Wire Wire Line
-	2900 4850 2050 4850
 Wire Wire Line
 	4400 4600 4300 4600
@@
 AR Path="/617509F7/61730A88" Ref="C22"  Part="1"
 AR Path="/61750A2A/61730A88" Ref="C?"  Part="1"
-F 0 "C12" H 5800 3050 50  0000 L CNN
+AR Path="/6176CA10/61730A88" Ref="C?"  Part="1"
+AR Path="/6176CA81/61730A88" Ref="C?"  Part="1"
+AR Path="/6176CAE4/61730A88" Ref="C?"  Part="1"
+F 0 "C?" H 5800 3050 50  0000 L CNN
 F 1 "10 uF" H 5800 2950 50  0000 L CNN
 F 2 "" H 5750 3150 50  0001 C CNN
@@
 AR Path="/617509F7/61733718" Ref="C23"  Part="1"
 AR Path="/61750A2A/61733718" Ref="C?"  Part="1"
-F 0 "C13" H 6200 3050 50  0000 L CNN
+AR Path="/6176CA10/61733718" Ref="C?"  Part="1"
+AR Path="/6176CA81/61733718" Ref="C?"  Part="1"
+AR Path="/6176CAE4/61733718" Ref="C?"  Part="1"
+F 0 "C?" H 6200 3050 50  0000 L CNN
 F 1 "0.1 uF" H 6200 2950 50  0000 L CNN
 F 2 "" H 6150 3150 50  0001 C CNN
@@
 AR Path="/617509F7/61735A2B" Ref="#PWR?"  Part="1"
 AR Path="/61750A2A/61735A2B" Ref="#PWR?"  Part="1"
+AR Path="/6176CA10/61735A2B" Ref="#PWR?"  Part="1"
+AR Path="/6176CA81/61735A2B" Ref="#PWR?"  Part="1"
+AR Path="/6176CAE4/61735A2B" Ref="#PWR?"  Part="1"
 F 0 "#PWR?" H 5950 3250 50  0001 C CNN
 F 1 "GND" H 5955 3327 50  0000 C CNN
@@
 AR Path="/617509F7/61710D71" Ref="J?"  Part="1"
 AR Path="/61750A2A/61710D71" Ref="J?"  Part="1"
+AR Path="/6176CA10/61710D71" Ref="J?"  Part="1"
+AR Path="/6176CA81/61710D71" Ref="J?"  Part="1"
+AR Path="/6176CAE4/61710D71" Ref="J?"  Part="1"
 F 0 "J?" H 8200 4515 50  0000 C CNN
 F 1 "IFE98" H 8200 4424 50  0000 C CNN
@@
 AR Path="/617509F7/61717F3E" Ref="U2"  Part="1"
 AR Path="/61750A2A/61717F3E" Ref="U3"  Part="1"
-F 0 "U1" H 5600 4415 50  0000 C CNN
+AR Path="/61717F3E" Ref="U1"  Part="1"
+AR Path="/6176CA10/61717F3E" Ref="U?"  Part="1"
+AR Path="/6176CA81/61717F3E" Ref="U?"  Part="1"
+AR Path="/6176CAE4/61717F3E" Ref="U?"  Part="1"
+F 0 "U?" H 5600 4415 50  0000 C CNN
 F 1 "74ACT08SCX" H 5600 4324 50  0000 C CNN
 F 2 "SOIC127P600X175-14N" H 5950 4250 50  0001 L CNN
@@
 AR Path="/617509F7/6173205B" Ref="#PWR?"  Part="1"
 AR Path="/61750A2A/6173205B" Ref="#PWR?"  Part="1"
+AR Path="/6176CA10/6173205B" Ref="#PWR?"  Part="1"
+AR Path="/6176CA81/6173205B" Ref="#PWR?"  Part="1"
+AR Path="/6176CAE4/6173205B" Ref="#PWR?"  Part="1"
 F 0 "#PWR?" H 4700 4100 50  0001 C CNN
 F 1 "GND" H 4705 4177 50  0000 C CNN
@@
 	4950 4750 5100 4750
 Wire Wire Line
-	4400 5000 6350 5000
-Wire Wire Line
-	4350 4950 4350 5050
-Wire Wire Line
-	4350 5050 6400 5050
-Wire Wire Line
-	6350 5000 6350 4350
-Wire Wire Line
-	6350 4350 6100 4350
-Wire Wire Line
-	6400 4250 6100 4250
-Wire Wire Line
-	6400 4250 6400 5050
+	4400 5000 6200 5000
+Wire Wire Line
+	6200 5000 6200 4350
+Wire Wire Line
+	6200 4350 6100 4350
 $Comp
 L Device:R_Small_US R?
@@
 AR Path="/617509F7/617428A7" Ref="R?"  Part="1"
 AR Path="/61750A2A/617428A7" Ref="R?"  Part="1"
+AR Path="/6176CA10/617428A7" Ref="R?"  Part="1"
+AR Path="/6176CA81/617428A7" Ref="R?"  Part="1"
+AR Path="/6176CAE4/617428A7" Ref="R?"  Part="1"
 F 0 "R?" V 6900 4450 50  0000 L CNN
 F 1 "150 Ohm" V 6800 4200 50  0000 L CNN
@@
 AR Path="/617509F7/61748E58" Ref="C24"  Part="1"
 AR Path="/61750A2A/61748E58" Ref="C?"  Part="1"
-F 0 "C14" V 6900 4800 50  0000 L CNN
+AR Path="/6176CA10/61748E58" Ref="C?"  Part="1"
+AR Path="/6176CA81/61748E58" Ref="C?"  Part="1"
+AR Path="/6176CAE4/61748E58" Ref="C?"  Part="1"
+F 0 "C?" V 6900 4800 50  0000 L CNN
 F 1 "100 pF" V 6800 4650 50  0000 L CNN
 F 2 "" H 6700 4800 50  0001 C CNN
@@
 AR Path="/617509F7/6174EB5A" Ref="R?"  Part="1"
 AR Path="/61750A2A/6174EB5A" Ref="R?"  Part="1"
+AR Path="/6176CA10/6174EB5A" Ref="R?"  Part="1"
+AR Path="/6176CA81/6174EB5A" Ref="R?"  Part="1"
+AR Path="/6176CAE4/6174EB5A" Ref="R?"  Part="1"
 F 0 "R?" H 7400 3250 50  0000 L CNN
 F 1 "365 Ohm" H 7400 3350 50  0000 L CNN
@@
 AR Path="/617509F7/6175F75B" Ref="#PWR?"  Part="1"
 AR Path="/61750A2A/6175F75B" Ref="#PWR?"  Part="1"
+AR Path="/6176CA10/6175F75B" Ref="#PWR?"  Part="1"
+AR Path="/6176CA81/6175F75B" Ref="#PWR?"  Part="1"
+AR Path="/6176CAE4/6175F75B" Ref="#PWR?"  Part="1"
 F 0 "#PWR?" H 7500 4500 50  0001 C CNN
 F 1 "GND" H 7505 4577 50  0000 C CNN
@@
 Text GLabel 4300 4600 0    50   Input ~ 0
 5V
-Text GLabel 2950 4600 0    50   Input ~ 0
-3V3
-Text HLabel 2050 4850 0    50   Input ~ 0
+Text HLabel 8550 5250 2    50   Input ~ 0
 EPWM
+Wire Wire Line
+	6400 4250 6100 4250
+Wire Wire Line
+	6400 4250 6400 5250
+Wire Wire Line
+	6400 5250 8550 5250
 $EndSCHEMATC
