File: MC-FO/Emitter_Circuits.sch (KiCad schematic (older format))
At the start: 8 parts, among them U27 74ACT08SCX, U28 IFE98

Commit message: reset implementation, connector
Parts:
- added R29: 10K, Resistor_SMD:R_0603_1608Metric, symbol Device:R_Small_US
Connections:
- net 5V: no longer U27.13 (A2)
- net EPWM: now also R29.2
- net GND1: now also R29.1
- net RESET_FO: now also U27.13 (A2)
Other:
- note removed: "Was it just make it an input to one of the and gates?"
Changed lines of the file:
@@
 $Descr A4 11693 8268
 encoding utf-8
-Sheet 4 10
+Sheet 3 10
 Title ""
 Date ""
@@
 Comment4 ""
 $EndDescr
-Text Notes 4300 5450 0    50   ~ 10
+Text Notes 5450 6200 0    50   ~ 10
 Emitter CKT
 $Comp
@@
 AR Path="/6176CA81/617428A7" Ref="R101"  Part="1"
 AR Path="/6176CAE4/617428A7" Ref="R121"  Part="1"
-F 0 "R27" V 6900 4400 50  0000 L CNN
+F 0 "R121" V 6900 4400 50  0000 L CNN
 F 1 "150 Ohm" V 6800 4150 50  0000 L CNN
 F 2 "Resistor_SMD:R_0603_1608Metric" H 6700 4400 50  0001 C CNN
@@
 AR Path="/6176CA81/61748E58" Ref="C104"  Part="1"
 AR Path="/6176CAE4/61748E58" Ref="C124"  Part="1"
-F 0 "C36" V 6900 4750 50  0000 L CNN
+F 0 "C124" V 6900 4750 50  0000 L CNN
 F 1 "100 pF" V 6800 4600 50  0000 L CNN
 F 2 "Capacitor_SMD:C_0603_1608Metric" H 6700 4750 50  0001 C CNN
@@
 AR Path="/6176CA81/6178E7F7" Ref="R102"  Part="1"
 AR Path="/6176CAE4/6178E7F7" Ref="R122"  Part="1"
-F 0 "R28" H 7400 3250 50  0000 L CNN
+F 0 "R122" H 7400 3250 50  0000 L CNN
 F 1 "365 Ohm" H 7400 3350 50  0000 L CNN
 F 2 "Resistor_SMD:R_0603_1608Metric" H 7300 3300 50  0001 C CNN
@@
 AR Path="/6176CA81/6171F0C9" Ref="C101"  Part="1"
 AR Path="/6176CAE4/6171F0C9" Ref="C121"  Part="1"
-F 0 "C33" H 4950 3250 50  0000 L CNN
+F 0 "C121" H 4950 3250 50  0000 L CNN
 F 1 "0.1 uF" H 4950 3150 50  0000 L CNN
 F 2 "Capacitor_SMD:C_0603_1608Metric" H 4900 3350 50  0001 C CNN
@@
 AR Path="/6176CA81/61733718" Ref="C103"  Part="1"
 AR Path="/6176CAE4/61733718" Ref="C123"  Part="1"
-F 0 "C35" H 6200 3050 50  0000 L CNN
+F 0 "C123" H 6200 3050 50  0000 L CNN
 F 1 "0.1 uF" H 6200 2950 50  0000 L CNN
 F 2 "Capacitor_SMD:C_0603_1608Metric" H 6150 3150 50  0001 C CNN
@@
 AR Path="/6176CA81/61730A88" Ref="C102"  Part="1"
 AR Path="/6176CAE4/61730A88" Ref="C122"  Part="1"
-F 0 "C34" H 5800 3050 50  0000 L CNN
+F 0 "C122" H 5800 3050 50  0000 L CNN
 F 1 "10 uF" H 5800 2950 50  0000 L CNN
 F 2 "Capacitor_SMD:C_0603_1608Metric" H 5750 3150 50  0001 C CNN
@@
 AR Path="/6176CA81/61804FDE" Ref="U101"  Part="1"
 AR Path="/6176CAE4/61804FDE" Ref="U121"  Part="1"
-F 0 "U27" H 4650 4115 50  0000 C CNN
+F 0 "U121" H 4650 4115 50  0000 C CNN
 F 1 "74ACT08SCX" H 4650 4024 50  0000 C CNN
 F 2 "Package_SO:SOIC-14_3.9x8.7mm_P1.27mm" H 4650 4000 50  0001 C CNN
@@
 Wire Wire Line
 	5050 4150 5350 4150
-Wire Wire Line
-	5050 4250 5350 4250
-Wire Wire Line
-	5350 4250 5350 4150
-Connection ~ 5350 4150
 Wire Wire Line
 	5900 5250 5900 4350
@@
 AR Path="/6176CAE4/61778B54" Ref="U122"  Part="1"
 AR Path="/617509F7/61778B54" Ref="U42"  Part="1"
-F 0 "U28" H 8000 4215 50  0000 C CNN
+F 0 "U122" H 8000 4215 50  0000 C CNN
 F 1 "IFE98" H 8000 4124 50  0000 C CNN
 F 2 "Footprints_MC-FO:IFE98" H 8000 4100 50  0001 C CNN
@@
 	3650 4350 3650 4650
 Connection ~ 3650 4650
-Wire Notes Line
-	1800 2100 3150 2100
-Wire Notes Line
-	3150 2100 3150 1050
-Wire Notes Line
-	3150 1050 1800 1050
-Wire Notes Line
-	1800 1050 1800 2100
-Text HLabel 2400 1500 0    50   Input ~ 0
+Text HLabel 8550 5100 2    50   Input ~ 0
 RESET_FO
 Wire Wire Line
@@
 Wire Wire Line
 	4750 3650 4900 3650
-Text Notes 3550 1550 0    50   ~ 0
-Was it just make it an input to one of the and gates?
+Wire Wire Line
+	8550 5100 6050 5100
+Wire Wire Line
+	6050 5100 6050 4250
+Wire Wire Line
+	6050 4250 5050 4250
+$Comp
+L Device:R_Small_US R29
+U 1 1 617DC24B
+P 5900 5450
+AR Path="/61717EAF/617DC24B" Ref="R29"  Part="1"
+AR Path="/617509F7/617DC24B" Ref="R43"  Part="1"
+AR Path="/61750A2A/617DC24B" Ref="R63"  Part="1"
+AR Path="/6176CA10/617DC24B" Ref="R83"  Part="1"
+AR Path="/6176CA81/617DC24B" Ref="R103"  Part="1"
+AR Path="/6176CAE4/617DC24B" Ref="R123"  Part="1"
+F 0 "R123" H 6000 5400 50  0000 L CNN
+F 1 "10K" H 6000 5500 50  0000 L CNN
+F 2 "Resistor_SMD:R_0603_1608Metric" H 5900 5450 50  0001 C CNN
+F 3 "~" H 5900 5450 50  0001 C CNN
+	1    5900 5450
+	-1   0    0    1
+$EndComp
+Text HLabel 5900 5650 3    50   Input ~ 0
+GND1
+Wire Wire Line
+	5900 5250 5900 5350
+Connection ~ 5900 5250
+Wire Wire Line
+	5900 5550 5900 5650
 $EndSCHEMATC
