File: MC-FO/MC-LED.sch (KiCad schematic (older format))
At the start: 14 parts, among them U181 74LVC1G07QDCKTQ1, U182 74LVCE1G08W5-7, U183 BU4831F-TR, U184 BU4847F-TR

Commit message: Add files via upload
Parts:
- U182: symbol MC-FO:74LVCE1G08W5-7 -> Existing_IC_Models:74LVCE1G08W5-7
- U183: symbol MC-FO:BU4831F-TR -> Existing_IC_Models:BU4831F-TR
- U184: symbol MC-FO:BU4847F-TR -> Existing_IC_Models:BU4847F-TR
Changed lines of the file:
@@
 $EndComp
 $Comp
-L MC-FO:BU4847F-TR U184
+L Existing_IC_Models:BU4847F-TR U184
 U 1 1 61A5F13F
 P 7075 2775
@@
 $EndComp
 $Comp
-L MC-FO:BU4831F-TR U183
+L Existing_IC_Models:BU4831F-TR U183
 U 1 1 61A601DB
 P 5125 2775
@@
 Connection ~ 6100 3325
 $Comp
-L MC-FO:74LVCE1G08W5-7 U182
+L Existing_IC_Models:74LVCE1G08W5-7 U182
 U 1 1 6222C302
 P 4625 3925

Commit message: Voltage detector footprint correction
Parts:
- U183, U184: footprint Package_SO:SOP-4_3.8x4.1mm_P2.54mm -> Footprints_MC-FO:BU4847F-TR
Changed lines of the file:
@@
 F 0 "U184" H 7075 3345 50  0000 C CNN
 F 1 "BU4847F-TR" H 7075 3254 50  0000 C CNN
-F 2 "Package_SO:SOP-4_3.8x4.1mm_P2.54mm" H 7075 2775 50  0001 L BNN
+F 2 "Footprints_MC-FO:BU4847F-TR" H 7075 2775 50  0001 L BNN
 F 3 "https://fscdn.rohm.com/en/products/databook/datasheet/ic/power/voltage_detector/bu48xxg-e.pdf" H 7075 2775 50  0001 L BNN
 F 4 "Rohm" H 7075 2775 50  0001 L BNN "Manufacturer"
@@
 F 0 "U183" H 5125 3345 50  0000 C CNN
 F 1 "BU4831F-TR" H 5125 3254 50  0000 C CNN
-F 2 "Package_SO:SOP-4_3.8x4.1mm_P2.54mm" H 5125 2775 50  0001 L BNN
+F 2 "Footprints_MC-FO:BU4847F-TR" H 5125 2775 50  0001 L BNN
 F 3 "https://fscdn.rohm.com/en/products/databook/datasheet/ic/power/voltage_detector/bu48xxg-e.pdf" H 5125 2775 50  0001 L BNN
 F 4 "Rohm" H 5125 2775 50  0001 L BNN "Manufacturer"
