File: MC-ADC/MC-ADC.sch (KiCad schematic (older format))
At the start: 5 parts

Commit message: ADC Work
Parts:
- removed JP10, JP11: Jumper, symbol Device:Jumper
- removed R10: 1MOhm, symbol Device:R_Small_US
- removed R11: 50R, symbol Device:R_Small_US
- added J10, J11, J12, J2, J3, J4, J5, J6, J7, J8, J9: Conn_Coaxial, symbol Connector:Conn_Coaxial
- added U10, U? (x5): SZCM1213A-04SO, symbol MC-ADC:SZCM1213A-04SO
- gave numbers to parts that had none: 1
Connections:
- net labels removed: GND, RAW_INPUT
- wire segments 7 -> 0
Other:
- note removed: "all ADC card inputs go to BNC?\n"
- moved on the sheet: J1

Commit message: ADC Work
Parts:
- added C?: DNP, symbol Device:C_Small
- added R?: 100R, symbol Device:R_Small_US
- added R?: 20R, symbol Device:R_Small_US
- added R? (x2): 0R, symbol Device:R_Small_US
Connections:
- net BNC_Terminations/InputA0A1P: now reaches J1.1 (In)
- net BNC_Terminations/InputA0A1P: now also U?.1 (CH1), R?.2
- net BNC_Terminations/InputA0A1N: now reaches J1.2 (Ext)
- net BNC_Terminations/InputD4D5P: now reaches J12.1 (In)
- net BNC_Terminations/InputD4D5N: now reaches J12.2 (Ext)
- new net: R?.1, R?.2, R?.2
- new net: C?.2, R?.1
- new net ADCINA0: C?.1, R?.1
- new net GND: R?.1, R?.2
Other:
- note added: "0 Ohm DNP resistors to GND just before ADC inputs -- necessary?"
- note added: "to connector & then DSP\n"
- moved on the sheet: J1, J10, J11, J12, J2, J3, J4, J5, J6, J7, J8, J9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
Changed lines of the file:
@@
 L Connector:Conn_Coaxial J1
 U 1 1 61F07758
-P 950 2300
-F 0 "J1" H 1100 2300 50  0000 L CNN
-F 1 "Conn_Coaxial" H 700 2450 50  0000 L CNN
-F 2 "" H 950 2300 50  0001 C CNN
-F 3 " ~" H 950 2300 50  0001 C CNN
-	1    950  2300
+P 950 950
+F 0 "J1" H 1100 950 50  0000 L CNN
+F 1 "Conn_Coaxial" H 700 1100 50  0000 L CNN
+F 2 "" H 950 950 50  0001 C CNN
+F 3 " ~" H 950 950 50  0001 C CNN
+	1    950  950
 	-1   0    0    -1
 $EndComp
@@
 L MC-ADC:SZCM1213A-04SO U10
 U 1 1 61F0B91E
-P 3350 1200
-F 0 "U10" H 3350 1765 50  0000 C CNN
-F 1 "SZCM1213A-04SO" H 3350 1674 50  0000 C CNN
-F 2 "" H 3300 1800 50  0001 C CNN
-F 3 "" H 3300 1800 50  0001 C CNN
-	1    3350 1200
+P 7650 5900
+F 0 "U10" H 7650 6465 50  0000 C CNN
+F 1 "SZCM1213A-04SO" H 7650 6374 50  0000 C CNN
+F 2 "" H 7600 6500 50  0001 C CNN
+F 3 "" H 7600 6500 50  0001 C CNN
+	1    7650 5900
 	1    0    0    -1
 $EndComp
@@
 L MC-ADC:SZCM1213A-04SO U?
 U 1 1 61F0ECE3
-P 4750 1200
-F 0 "U?" H 4750 1765 50  0000 C CNN
-F 1 "SZCM1213A-04SO" H 4750 1674 50  0000 C CNN
-F 2 "" H 4700 1800 50  0001 C CNN
-F 3 "" H 4700 1800 50  0001 C CNN
-	1    4750 1200
+P 9050 5900
+F 0 "U?" H 9050 6465 50  0000 C CNN
+F 1 "SZCM1213A-04SO" H 9050 6374 50  0000 C CNN
+F 2 "" H 9000 6500 50  0001 C CNN
+F 3 "" H 9000 6500 50  0001 C CNN
+	1    9050 5900
 	1    0    0    -1
 $EndComp
@@
 L MC-ADC:SZCM1213A-04SO U?
 U 1 1 61F0F9D7
-P 6050 1200
-F 0 "U?" H 6050 1765 50  0000 C CNN
-F 1 "SZCM1213A-04SO" H 6050 1674 50  0000 C CNN
-F 2 "" H 6000 1800 50  0001 C CNN
-F 3 "" H 6000 1800 50  0001 C CNN
-	1    6050 1200
+P 10350 5900
+F 0 "U?" H 10350 6465 50  0000 C CNN
+F 1 "SZCM1213A-04SO" H 10350 6374 50  0000 C CNN
+F 2 "" H 10300 6500 50  0001 C CNN
+F 3 "" H 10300 6500 50  0001 C CNN
+	1    10350 5900
 	1    0    0    -1
 $EndComp
@@
 L MC-ADC:SZCM1213A-04SO U?
 U 1 1 61F11B57
-P 7350 1200
-F 0 "U?" H 7350 1765 50  0000 C CNN
-F 1 "SZCM1213A-04SO" H 7350 1674 50  0000 C CNN
-F 2 "" H 7300 1800 50  0001 C CNN
-F 3 "" H 7300 1800 50  0001 C CNN
-	1    7350 1200
+P 7400 1250
+F 0 "U?" H 7400 1815 50  0000 C CNN
+F 1 "SZCM1213A-04SO" H 7400 1724 50  0000 C CNN
+F 2 "" H 7350 1850 50  0001 C CNN
+F 3 "" H 7350 1850 50  0001 C CNN
+	1    7400 1250
 	1    0    0    -1
 $EndComp
@@
 	1    0    0    -1
 $EndComp
-$Sheet
-S 4800 4750 500  150
-U 61F0AAD9
-F0 "Termination_Jumper" 50
-F1 "Terminations.sch" 50
-F2 "Input" I L 4800 4800 50
-$EndSheet
 $Comp
 L Connector:Conn_Coaxial J2
 U 1 1 61F0F6A2
+P 950 1400
+F 0 "J2" H 1100 1400 50  0000 L CNN
+F 1 "Conn_Coaxial" H 700 1550 50  0000 L CNN
+F 2 "" H 950 1400 50  0001 C CNN
+F 3 " ~" H 950 1400 50  0001 C CNN
+	1    950  1400
+	-1   0    0    -1
+$EndComp
+$Comp
+L Connector:Conn_Coaxial J3
+U 1 1 61F100B8
+P 950 1850
+F 0 "J3" H 1100 1850 50  0000 L CNN
+F 1 "Conn_Coaxial" H 700 2000 50  0000 L CNN
+F 2 "" H 950 1850 50  0001 C CNN
+F 3 " ~" H 950 1850 50  0001 C CNN
+	1    950  1850
+	-1   0    0    -1
+$EndComp
+$Comp
+L Connector:Conn_Coaxial J4
+U 1 1 61F10889
+P 950 2300
+F 0 "J4" H 1100 2300 50  0000 L CNN
+F 1 "Conn_Coaxial" H 700 2450 50  0000 L CNN
+F 2 "" H 950 2300 50  0001 C CNN
+F 3 " ~" H 950 2300 50  0001 C CNN
+	1    950  2300
+	-1   0    0    -1
+$EndComp
+$Comp
+L Connector:Conn_Coaxial J5
+U 1 1 61F1BB8F
 P 950 2750
-F 0 "J2" H 1100 2750 50  0000 L CNN
+F 0 "J5" H 1100 2750 50  0000 L CNN
 F 1 "Conn_Coaxial" H 700 2900 50  0000 L CNN
 F 2 "" H 950 2750 50  0001 C CNN
@@
 $EndComp
 $Comp
-L Connector:Conn_Coaxial J3
-U 1 1 61F100B8
+L Connector:Conn_Coaxial J6
+U 1 1 61F1BB95
 P 950 3200
-F 0 "J3" H 1100 3200 50  0000 L CNN
+F 0 "J6" H 1100 3200 50  0000 L CNN
 F 1 "Conn_Coaxial" H 700 3350 50  0000 L CNN
 F 2 "" H 950 3200 50  0001 C CNN
@@
 $EndComp
 $Comp
-L Connector:Conn_Coaxial J4
-U 1 1 61F10889
+L Connector:Conn_Coaxial J7
+U 1 1 61F1BB9B
 P 950 3650
-F 0 "J4" H 1100 3650 50  0000 L CNN
+F 0 "J7" H 1100 3650 50  0000 L CNN
 F 1 "Conn_Coaxial" H 700 3800 50  0000 L CNN
 F 2 "" H 950 3650 50  0001 C CNN
@@
 $EndComp
 $Comp
-L Connector:Conn_Coaxial J5
-U 1 1 61F1BB8F
+L Connector:Conn_Coaxial J8
+U 1 1 61F1BBA1
 P 950 4100
-F 0 "J5" H 1100 4100 50  0000 L CNN
+F 0 "J8" H 1100 4100 50  0000 L CNN
 F 1 "Conn_Coaxial" H 700 4250 50  0000 L CNN
 F 2 "" H 950 4100 50  0001 C CNN
@@
 $EndComp
 $Comp
-L Connector:Conn_Coaxial J6
-U 1 1 61F1BB95
+L Connector:Conn_Coaxial J9
+U 1 1 61F20279
 P 950 4550
-F 0 "J6" H 1100 4550 50  0000 L CNN
+F 0 "J9" H 1100 4550 50  0000 L CNN
 F 1 "Conn_Coaxial" H 700 4700 50  0000 L CNN
 F 2 "" H 950 4550 50  0001 C CNN
@@
 $EndComp
 $Comp
-L Connector:Conn_Coaxial J7
-U 1 1 61F1BB9B
+L Connector:Conn_Coaxial J10
+U 1 1 61F2027F
 P 950 5000
-F 0 "J7" H 1100 5000 50  0000 L CNN
+F 0 "J10" H 1100 5000 50  0000 L CNN
 F 1 "Conn_Coaxial" H 700 5150 50  0000 L CNN
 F 2 "" H 950 5000 50  0001 C CNN
@@
 $EndComp
 $Comp
-L Connector:Conn_Coaxial J8
-U 1 1 61F1BBA1
+L Connector:Conn_Coaxial J11
+U 1 1 61F20285
 P 950 5450
-F 0 "J8" H 1100 5450 50  0000 L CNN
+F 0 "J11" H 1100 5450 50  0000 L CNN
 F 1 "Conn_Coaxial" H 700 5600 50  0000 L CNN
 F 2 "" H 950 5450 50  0001 C CNN
@@
 $EndComp
 $Comp
-L Connector:Conn_Coaxial J9
-U 1 1 61F20279
+L Connector:Conn_Coaxial J12
+U 1 1 61F2028B
 P 950 5900
-F 0 "J9" H 1100 5900 50  0000 L CNN
+F 0 "J12" H 1100 5900 50  0000 L CNN
 F 1 "Conn_Coaxial" H 700 6050 50  0000 L CNN
 F 2 "" H 950 5900 50  0001 C CNN
@@
 	-1   0    0    -1
 $EndComp
-$Comp
-L Connector:Conn_Coaxial J10
-U 1 1 61F2027F
-P 950 6350
-F 0 "J10" H 1100 6350 50  0000 L CNN
-F 1 "Conn_Coaxial" H 700 6500 50  0000 L CNN
-F 2 "" H 950 6350 50  0001 C CNN
-F 3 " ~" H 950 6350 50  0001 C CNN
-	1    950  6350
-	-1   0    0    -1
-$EndComp
-$Comp
-L Connector:Conn_Coaxial J11
-U 1 1 61F20285
-P 950 6800
-F 0 "J11" H 1100 6800 50  0000 L CNN
-F 1 "Conn_Coaxial" H 700 6950 50  0000 L CNN
-F 2 "" H 950 6800 50  0001 C CNN
-F 3 " ~" H 950 6800 50  0001 C CNN
-	1    950  6800
-	-1   0    0    -1
-$EndComp
-$Comp
-L Connector:Conn_Coaxial J12
-U 1 1 61F2028B
-P 950 7250
-F 0 "J12" H 1100 7250 50  0000 L CNN
-F 1 "Conn_Coaxial" H 700 7400 50  0000 L CNN
-F 2 "" H 950 7250 50  0001 C CNN
-F 3 " ~" H 950 7250 50  0001 C CNN
-	1    950  7250
-	-1   0    0    -1
-$EndComp
+$Sheet
+S 1100 6400 5100 950
+U 61F25080
+F0 "BNC_Terminations" 50
+F1 "Terminations.sch" 50
+F2 "InputA0A1P" I T 6100 6400 50
+F3 "GND" I B 1450 7350 50
+F4 "InputA0A1N" I T 6000 6400 50
+F5 "InputD4D5P" I T 1450 6400 50
+F6 "InputD4D5N" I T 1350 6400 50
+$EndSheet
+Wire Wire Line
+	950  6100 1350 6100
+Wire Wire Line
+	1350 6100 1350 6400
+Wire Wire Line
+	1150 5900 1450 5900
+Wire Wire Line
+	1450 5900 1450 6400
+Wire Wire Line
+	950  1150 6000 1150
+Wire Wire Line
+	6000 1150 6000 6400
+Wire Wire Line
+	1150 950  6100 950
+Wire Wire Line
+	6100 950  6100 6400
+Wire Wire Line
+	6100 950  6600 950
+Connection ~ 6100 950
+Wire Wire Line
+	6600 950  6600 2100
+Wire Wire Line
+	6600 2100 7950 2100
+Connection ~ 6600 950
+Wire Wire Line
+	6600 950  6850 950
+$Comp
+L Device:R_Small_US R?
+U 1 1 61F4E828
+P 8050 2100
+F 0 "R?" V 7845 2100 50  0000 C CNN
+F 1 "100R" V 7936 2100 50  0000 C CNN
+F 2 "" H 8050 2100 50  0001 C CNN
+F 3 "~" H 8050 2100 50  0001 C CNN
+	1    8050 2100
+	0    1    1    0
+$EndComp
+$Comp
+L Device:R_Small_US R?
+U 1 1 61F4F7F5
+P 8300 2400
+F 0 "R?" H 8232 2354 50  0000 R CNN
+F 1 "20R" H 8232 2445 50  0000 R CNN
+F 2 "" H 8300 2400 50  0001 C CNN
+F 3 "~" H 8300 2400 50  0001 C CNN
+	1    8300 2400
+	-1   0    0    1
+$EndComp
+$Comp
+L Device:R_Small_US R?
+U 1 1 61F50226
+P 8700 2100
+F 0 "R?" V 8495 2100 50  0000 C CNN
+F 1 "0R" V 8586 2100 50  0000 C CNN
+F 2 "" H 8700 2100 50  0001 C CNN
+F 3 "~" H 8700 2100 50  0001 C CNN
+	1    8700 2100
+	0    1    1    0
+$EndComp
+$Comp
+L Device:R_Small_US R?
+U 1 1 61F5092C
+P 8700 2750
+F 0 "R?" V 8495 2750 50  0000 C CNN
+F 1 "0R" V 8586 2750 50  0000 C CNN
+F 2 "" H 8700 2750 50  0001 C CNN
+F 3 "~" H 8700 2750 50  0001 C CNN
+	1    8700 2750
+	0    1    1    0
+$EndComp
+Wire Wire Line
+	8150 2100 8300 2100
+Wire Wire Line
+	8300 2100 8300 2300
+Connection ~ 8300 2100
+Wire Wire Line
+	8300 2100 8600 2100
+Wire Wire Line
+	8300 2500 8300 2750
+Wire Wire Line
+	8300 2750 8600 2750
+Wire Wire Line
+	8300 2750 8300 2900
+Connection ~ 8300 2750
+$Comp
+L power:GND #PWR?
+U 1 1 61F5292C
+P 8300 2900
+F 0 "#PWR?" H 8300 2650 50  0001 C CNN
+F 1 "GND" H 8305 2727 50  0000 C CNN
+F 2 "" H 8300 2900 50  0001 C CNN
+F 3 "" H 8300 2900 50  0001 C CNN
+	1    8300 2900
+	1    0    0    -1
+$EndComp
+$Comp
+L Device:C_Small C?
+U 1 1 61F53865
+P 9000 2400
+F 0 "C?" H 9092 2446 50  0000 L CNN
+F 1 "DNP" H 9092 2355 50  0000 L CNN
+F 2 "" H 9000 2400 50  0001 C CNN
+F 3 "~" H 9000 2400 50  0001 C CNN
+	1    9000 2400
+	1    0    0    -1
+$EndComp
+Wire Wire Line
+	8800 2100 9000 2100
+Wire Wire Line
+	9000 2100 9000 2300
+Wire Wire Line
+	9000 2500 9000 2750
+Wire Wire Line
+	9000 2750 8800 2750
+Wire Wire Line
+	9000 2100 9400 2100
+Connection ~ 9000 2100
+Text GLabel 9400 2100 2    50   Input ~ 0
+ADCINA0
+Text Notes 9450 2300 0    50   ~ 0
+to connector & then DSP\n
+Text Notes 8300 3500 0    50   ~ 0
+0 Ohm DNP resistors to GND just before ADC inputs -- necessary?
 $EndSCHEMATC

Commit message: adc WORK
Parts:
- removed J10, J11, J6, J7, J8, J9: Conn_Coaxial, symbol Connector:Conn_Coaxial
Connections:
- wire segments 23 -> 21
Other:
- moved on the sheet: J1, J2, J3, J4, J5
Changed lines of the file:
@@
 L Connector:Conn_Coaxial J1
 U 1 1 61F07758
-P 950 950
-F 0 "J1" H 1100 950 50  0000 L CNN
-F 1 "Conn_Coaxial" H 700 1100 50  0000 L CNN
-F 2 "" H 950 950 50  0001 C CNN
-F 3 " ~" H 950 950 50  0001 C CNN
-	1    950  950
+P 950 3150
+F 0 "J1" H 1100 3150 50  0000 L CNN
+F 1 "Conn_Coaxial" H 700 3300 50  0000 L CNN
+F 2 "" H 950 3150 50  0001 C CNN
+F 3 " ~" H 950 3150 50  0001 C CNN
+	1    950  3150
 	-1   0    0    -1
 $EndComp
@@
 L Connector:Conn_Coaxial J2
 U 1 1 61F0F6A2
-P 950 1400
-F 0 "J2" H 1100 1400 50  0000 L CNN
-F 1 "Conn_Coaxial" H 700 1550 50  0000 L CNN
-F 2 "" H 950 1400 50  0001 C CNN
-F 3 " ~" H 950 1400 50  0001 C CNN
-	1    950  1400
+P 950 3700
+F 0 "J2" H 1100 3700 50  0000 L CNN
+F 1 "Conn_Coaxial" H 700 3850 50  0000 L CNN
+F 2 "" H 950 3700 50  0001 C CNN
+F 3 " ~" H 950 3700 50  0001 C CNN
+	1    950  3700
 	-1   0    0    -1
 $EndComp
@@
 L Connector:Conn_Coaxial J3
 U 1 1 61F100B8
-P 950 1850
-F 0 "J3" H 1100 1850 50  0000 L CNN
-F 1 "Conn_Coaxial" H 700 2000 50  0000 L CNN
-F 2 "" H 950 1850 50  0001 C CNN
-F 3 " ~" H 950 1850 50  0001 C CNN
-	1    950  1850
+P 950 4250
+F 0 "J3" H 1100 4250 50  0000 L CNN
+F 1 "Conn_Coaxial" H 700 4400 50  0000 L CNN
+F 2 "" H 950 4250 50  0001 C CNN
+F 3 " ~" H 950 4250 50  0001 C CNN
+	1    950  4250
 	-1   0    0    -1
 $EndComp
@@
 L Connector:Conn_Coaxial J4
 U 1 1 61F10889
-P 950 2300
-F 0 "J4" H 1100 2300 50  0000 L CNN
-F 1 "Conn_Coaxial" H 700 2450 50  0000 L CNN
-F 2 "" H 950 2300 50  0001 C CNN
-F 3 " ~" H 950 2300 50  0001 C CNN
-	1    950  2300
+P 950 4750
+F 0 "J4" H 1100 4750 50  0000 L CNN
+F 1 "Conn_Coaxial" H 700 4900 50  0000 L CNN
+F 2 "" H 950 4750 50  0001 C CNN
+F 3 " ~" H 950 4750 50  0001 C CNN
+	1    950  4750
 	-1   0    0    -1
 $EndComp
@@
 L Connector:Conn_Coaxial J5
 U 1 1 61F1BB8F
-P 950 2750
-F 0 "J5" H 1100 2750 50  0000 L CNN
-F 1 "Conn_Coaxial" H 700 2900 50  0000 L CNN
-F 2 "" H 950 2750 50  0001 C CNN
-F 3 " ~" H 950 2750 50  0001 C CNN
-	1    950  2750
-	-1   0    0    -1
-$EndComp
-$Comp
-L Connector:Conn_Coaxial J6
-U 1 1 61F1BB95
-P 950 3200
-F 0 "J6" H 1100 3200 50  0000 L CNN
-F 1 "Conn_Coaxial" H 700 3350 50  0000 L CNN
-F 2 "" H 950 3200 50  0001 C CNN
-F 3 " ~" H 950 3200 50  0001 C CNN
-	1    950  3200
-	-1   0    0    -1
-$EndComp
-$Comp
-L Connector:Conn_Coaxial J7
-U 1 1 61F1BB9B
-P 950 3650
-F 0 "J7" H 1100 3650 50  0000 L CNN
-F 1 "Conn_Coaxial" H 700 3800 50  0000 L CNN
-F 2 "" H 950 3650 50  0001 C CNN
-F 3 " ~" H 950 3650 50  0001 C CNN
-	1    950  3650
-	-1   0    0    -1
-$EndComp
-$Comp
-L Connector:Conn_Coaxial J8
-U 1 1 61F1BBA1
-P 950 4100
-F 0 "J8" H 1100 4100 50  0000 L CNN
-F 1 "Conn_Coaxial" H 700 4250 50  0000 L CNN
-F 2 "" H 950 4100 50  0001 C CNN
-F 3 " ~" H 950 4100 50  0001 C CNN
-	1    950  4100
-	-1   0    0    -1
-$EndComp
-$Comp
-L Connector:Conn_Coaxial J9
-U 1 1 61F20279
-P 950 4550
-F 0 "J9" H 1100 4550 50  0000 L CNN
-F 1 "Conn_Coaxial" H 700 4700 50  0000 L CNN
-F 2 "" H 950 4550 50  0001 C CNN
-F 3 " ~" H 950 4550 50  0001 C CNN
-	1    950  4550
-	-1   0    0    -1
-$EndComp
-$Comp
-L Connector:Conn_Coaxial J10
-U 1 1 61F2027F
-P 950 5000
-F 0 "J10" H 1100 5000 50  0000 L CNN
-F 1 "Conn_Coaxial" H 700 5150 50  0000 L CNN
-F 2 "" H 950 5000 50  0001 C CNN
-F 3 " ~" H 950 5000 50  0001 C CNN
-	1    950  5000
-	-1   0    0    -1
-$EndComp
-$Comp
-L Connector:Conn_Coaxial J11
-U 1 1 61F20285
-P 950 5450
-F 0 "J11" H 1100 5450 50  0000 L CNN
-F 1 "Conn_Coaxial" H 700 5600 50  0000 L CNN
-F 2 "" H 950 5450 50  0001 C CNN
-F 3 " ~" H 950 5450 50  0001 C CNN
-	1    950  5450
+P 950 5300
+F 0 "J5" H 1100 5300 50  0000 L CNN
+F 1 "Conn_Coaxial" H 700 5450 50  0000 L CNN
+F 2 "" H 950 5300 50  0001 C CNN
+F 3 " ~" H 950 5300 50  0001 C CNN
+	1    950  5300
 	-1   0    0    -1
 $EndComp
@@
 	1450 5900 1450 6400
 Wire Wire Line
-	950  1150 6000 1150
-Wire Wire Line
 	6000 1150 6000 6400
-Wire Wire Line
-	1150 950  6100 950
 Wire Wire Line
 	6100 950  6100 6400
 Wire Wire Line
 	6100 950  6600 950
-Connection ~ 6100 950
 Wire Wire Line
 	6600 950  6600 2100

Commit message: Significant ADC Progress
Parts:
- removed J12, J4, J5: Conn_Coaxial, symbol Connector:Conn_Coaxial
- removed U10, U? (x4): SZCM1213A-04SO, symbol MC-ADC:SZCM1213A-04SO
- added C? (x5): C_Small, symbol Device:C_Small
- added D? (x3): 10V, symbol Device:D_Zener
- added DNP (x3): R, symbol Device:R_Small_US
- added J1: 86094327313755E1LF, symbol MC-ADC:86094327313755E1LF
- added JP? (x3): Jumper_3_Bridged12, symbol Jumper:Jumper_3_Bridged12
- added R? (x3): 0R, symbol Device:R_Small_US
- added R? (x3): 1MOhm, symbol Device:R_Small_US
- added R? (x3): 50R, symbol Device:R_Small_US
- added R? (x5): R_Small_US, symbol Device:R_Small_US
- added R? (x6): 100R, symbol Device:R_Small_US
- added R? (x3): 250R, symbol Device:R_Small_US
- added U? (x3): 74LVC1G32SE-7, symbol 74xGxx:74LVC1G32
- J1, J2, J3: footprint (none) -> Connector_Coaxial:BNC_Amphenol_031-6575_Horizontal
- gave numbers to parts that had none: 6
Connections:
- net labels added: 24V, ADCINA2, ADCINA4, ADCINB2
- wire segments 21 -> 216
Other:
- note added: "BW calcs to meet requirements"
- note added: "Edge Connector - Amphenol"
- note added: "Need to deal with driving SAR ADCs"
- note added: "accounting for 15mm with each \nBNC connection, total number of \nconnections = 92/15 = 6 with no \nspace in-between\n\n\n3 BNC connectors on 2 cards\n"
- note added: "post CDR\n"
- note removed: "0 Ohm DNP resistors to GND just before ADC inputs -- necessary?"
- moved on the sheet: C1, J1, J2, J3, R1, R2, R3, R4, U2

Commit message: ADC Work
Parts:
- removed C? (x2): C_Small, symbol Device:C_Small
- removed D? (x2): 10V, symbol Device:D_Zener
- removed J2, J3: Conn_Coaxial, Connector_Coaxial:BNC_Amphenol_031-6575_Horizontal, symbol Connector:Conn_Coaxial
- removed JP? (x2): Jumper_3_Bridged12, symbol Jumper:Jumper_3_Bridged12
- removed R? (x2): 0R, symbol Device:R_Small_US
- removed R? (x2): 1MOhm, symbol Device:R_Small_US
- removed R? (x2): 50R, symbol Device:R_Small_US
- removed R? (x2): R_Small_US, symbol Device:R_Small_US
- removed R? (x4): 100R, symbol Device:R_Small_US
- removed R? (x2): 250R, symbol Device:R_Small_US
- removed U? (x2): 74LVC1G32SE-7, symbol 74xGxx:74LVC1G32
- added J?: Conn_Coaxial, Connector_Coaxial:BNC_Amphenol_031-6575_Horizontal, symbol Connector:Conn_Coaxial
- added JP?: Jumper, symbol Jumper:Jumper_3_Bridged12
- added R? (x3): 0R, symbol Device:R_Small_US
- added R?: 1MOhm, symbol Device:R_Small_US
- added R?: 50R, symbol Device:R_Small_US
- JP?: value Jumper_3_Bridged12 -> Jumper
Connections:
- wire segments 216 -> 151
Other:
- moved on the sheet: DNP, J1, JP?, R?

Commit message: ADC Work
Parts:
- removed C? (x2): C_Small, symbol Device:C_Small
- removed D?: 10V, symbol Device:D_Zener
- removed J?: Conn_Coaxial, Connector_Coaxial:BNC_Amphenol_031-6575_Horizontal, symbol Connector:Conn_Coaxial
- removed JP?: Jumper, symbol Jumper:Jumper_3_Bridged12
- removed R? (x2): R_Small_US, symbol Device:R_Small_US
- removed R? (x2): 100R, symbol Device:R_Small_US
- removed R?: 1MOhm, symbol Device:R_Small_US
- removed R?: 50R, symbol Device:R_Small_US
- removed R? (x2): 0R, symbol Device:R_Small_US
- removed R?: 250R, symbol Device:R_Small_US
- removed U?: 74LVC1G32SE-7, symbol 74xGxx:74LVC1G32
- added C?: C_Small, symbol Device:C_Small
- added JP?: Jumper, symbol Jumper:Jumper_3_Bridged12
- added R?: R_Small_US, symbol Device:R_Small_US
Connections:
- wire segments 151 -> 128
Other:
- note added: "Filter -> SAR ADC"
- note added: "INA 592"
- note added: "V divider if needed"
- moved on the sheet: C?, DNP, J1, JP?, R?

Commit message: ADC work
Parts:
- removed C?: C_Small, symbol Device:C_Small
- removed JP?: Jumper, symbol Jumper:Jumper_3_Bridged12
- removed R?: R_Small_US, symbol Device:R_Small_US
Connections:
- net labels added: GND1, GND2
- wire segments 128 -> 113
Other:
- note removed: "INA 592"
- note removed: "V divider if needed"
- moved on the sheet: C?, R?

Commit message: ADC Updates!
Parts:
- removed DNP (x3): R, symbol Device:R_Small_US
- removed J1: Conn_Coaxial, Connector_Coaxial:BNC_Amphenol_031-6575_Horizontal, symbol Connector:Conn_Coaxial
- removed JP?: Jumper, symbol Jumper:Jumper_3_Bridged12
- removed R? (x2): 0R, symbol Device:R_Small_US
- removed R?: 1MOhm, symbol Device:R_Small_US
- removed R?: 50R, symbol Device:R_Small_US
- added U? (x2): LM324DTBR2G, symbol MC-ADC:LM324DTBR2G
Connections:
- net labels added: 1.5V
- wire segments 113 -> 161
Other:
- note added: "3 BNC connectors on 2 cards\n"
- note removed: "accounting for 15mm with each \nBNC connection, total number of \nconnections = 92/15 = 6 with no \nspace in-between\n\n\n3 BNC connectors on 2 cards\n"
- moved on the sheet: C?, R?, U2
