File: MC-ADC/MC-ADC.sch (KiCad schematic (older format))
At the start: 26 parts, among them J1 86094327313755E1LF, U81 LM324DTBR2G, U82 LT6238CGN#PBF

Commit message: ADC Gerbers Generated
Connections:
- net 24V: now also J1.17 (Pin_17); no longer J1.2 (Pin_2)
- net ADCIN1: now also J1.29 (Pin_29); no longer J1.31 (Pin_31)
- net ADCIN2: now also J1.27 (Pin_27); no longer J1.29 (Pin_29)
- net ADCIN3: now also J1.25 (Pin_25); no longer J1.27 (Pin_27)
- net GND1: now also J1.2 (Pin_2), J1.31 (Pin_31); no longer J1.17 (Pin_17), J1.25 (Pin_25)
- net SAFE_STATE_FLAG renamed ~SAFE_STATE_FLAG
Other:
- moved on the sheet: J1
Changed lines of the file:
@@
 L MC-ADC:86094327313755E1LF J1
 U 1 1 61FF85F3
-P 10200 1750
-F 0 "J1" H 10250 2667 50  0000 C CNN
-F 1 "86094327313755E1LF" H 10250 2576 50  0000 C CNN
-F 2 "Footprints_MC-ADC:86094327313755E1LF" H 10200 1750 50  0001 C CNN
-F 3 "https://www.mouser.com/ProductDetail/649-94327313755E1LF" H 10200 1750 50  0001 C CNN
-	1    10200 1750
-	1    0    0    -1
-$EndComp
-Text GLabel 9800 1050 0    50   Input ~ 0
+P 9950 2000
+F 0 "J1" H 10350 800 50  0000 C CNN
+F 1 "86094327313755E1LF" H 10000 900 50  0000 C CNN
+F 2 "Footprints_MC-ADC:86094327313755E1LF" H 9950 2000 50  0001 C CNN
+F 3 "https://www.mouser.com/ProductDetail/649-94327313755E1LF" H 9950 2000 50  0001 C CNN
+	1    9950 2000
+	-1   0    0    1
+$EndComp
+Text GLabel 9450 2700 0    50   Input ~ 0
 24V
 Wire Wire Line
-	9900 1050 9900 1150
-Wire Wire Line
-	9900 2450 10000 2450
-Wire Wire Line
-	9900 2450 9900 2350
-Wire Wire Line
-	9900 2350 10000 2350
-Connection ~ 9900 2450
-Wire Wire Line
-	9900 2350 9900 2250
-Wire Wire Line
-	9900 2250 10000 2250
-Connection ~ 9900 2350
-Wire Wire Line
-	9900 2250 9900 2150
-Wire Wire Line
-	9900 2150 10000 2150
-Connection ~ 9900 2250
-Wire Wire Line
-	9900 2150 9900 2050
-Wire Wire Line
-	9900 2050 10000 2050
-Connection ~ 9900 2150
-Wire Wire Line
-	9900 2050 9900 1950
-Wire Wire Line
-	9900 1950 10000 1950
-Connection ~ 9900 2050
-Wire Wire Line
-	9900 1950 9900 1850
-Wire Wire Line
-	9900 1850 10000 1850
-Connection ~ 9900 1950
-Wire Wire Line
-	9900 1850 9900 1750
-Wire Wire Line
-	9900 1750 10000 1750
-Connection ~ 9900 1850
-Wire Wire Line
-	9900 1750 9900 1650
-Wire Wire Line
-	9900 1650 10000 1650
-Connection ~ 9900 1750
-Wire Wire Line
-	9900 1650 9900 1550
-Wire Wire Line
-	9900 1550 10000 1550
-Connection ~ 9900 1650
-Wire Wire Line
-	9900 1550 9900 1450
-Wire Wire Line
-	9900 1450 10000 1450
-Connection ~ 9900 1550
-Wire Wire Line
-	9900 1450 9900 1350
-Wire Wire Line
-	9900 1350 10000 1350
-Connection ~ 9900 1450
-Wire Wire Line
-	9900 1350 9900 1250
-Wire Wire Line
-	9900 1250 10000 1250
-Connection ~ 9900 1350
-Connection ~ 9900 1050
-Wire Wire Line
-	9900 1050 9800 1050
-Wire Wire Line
-	9900 1050 10000 1050
-Wire Wire Line
-	9900 1150 10000 1150
-Wire Notes Line
-	9050 650  9050 3100
-Wire Notes Line
-	11100 3100 11100 650
+	10250 2000 10150 2000
+Wire Wire Line
+	10250 2000 10250 2100
+Wire Wire Line
+	10250 2100 10150 2100
+Wire Wire Line
+	10250 2100 10250 2200
+Wire Wire Line
+	10250 2200 10150 2200
+Connection ~ 10250 2100
+Wire Wire Line
+	10250 2200 10250 2300
+Wire Wire Line
+	10250 2300 10150 2300
+Connection ~ 10250 2200
+Wire Wire Line
+	10250 2300 10250 2400
+Wire Wire Line
+	10250 2400 10150 2400
+Connection ~ 10250 2300
+Wire Wire Line
+	10250 2400 10250 2500
+Wire Wire Line
+	10250 2500 10150 2500
+Connection ~ 10250 2400
 Text Notes 9600 600  0    50   ~ 0
 Edge Connector - Amphenol\n
@@
 Wire Wire Line
 	4100 1150 3750 1150
-Text GLabel 10700 2450 2    50   Input ~ 0
+Text GLabel 9450 1500 0    50   Input ~ 0
 ADCIN1
-Text GLabel 10700 2250 2    50   Input ~ 0
+Text GLabel 9450 1700 0    50   Input ~ 0
 ADCIN2
 Text GLabel 5350 3650 3    50   Input ~ 0
 ADCIN1
 Wire Wire Line
-	10500 1550 10600 1550
-Wire Wire Line
-	10600 1550 10600 1650
-Wire Wire Line
-	10500 1650 10600 1650
-Connection ~ 10600 1650
-Wire Wire Line
-	10600 1650 10600 1750
-Wire Wire Line
-	10500 1750 10600 1750
-Connection ~ 10600 1750
-Wire Wire Line
-	10600 1750 10600 1850
-Wire Wire Line
-	10500 1850 10600 1850
-Connection ~ 10600 1850
-Wire Wire Line
-	10600 1850 10600 1950
-Wire Wire Line
-	10500 1950 10600 1950
+	9650 2200 9550 2200
+Wire Wire Line
+	9550 2200 9550 2100
+Wire Wire Line
+	9650 2100 9550 2100
+Connection ~ 9550 2100
+Wire Wire Line
+	9550 2100 9550 2000
+Wire Wire Line
+	9650 2000 9550 2000
+Connection ~ 9550 2000
 $Comp
 L power:GND1 #PWR0101
 U 1 1 620E7EB3
-P 10250 2800
-F 0 "#PWR0101" H 10250 2550 50  0001 C CNN
-F 1 "GND1" H 10255 2627 50  0000 C CNN
-F 2 "" H 10250 2800 50  0001 C CNN
-F 3 "" H 10250 2800 50  0001 C CNN
-	1    10250 2800
+P 9900 2900
+F 0 "#PWR0101" H 9900 2650 50  0001 C CNN
+F 1 "GND1" H 9905 2727 50  0000 C CNN
+F 2 "" H 9900 2900 50  0001 C CNN
+F 3 "" H 9900 2900 50  0001 C CNN
+	1    9900 2900
 	1    0    0    -1
 $EndComp
@@
 Wire Wire Line
 	5350 4900 5350 5200
-Text GLabel 10700 2050 2    50   Input ~ 0
+Text GLabel 9450 1900 0    50   Input ~ 0
 ADCIN3
 Text GLabel 5350 5200 3    50   Input ~ 0
@@
 ADCIN3
 Wire Wire Line
-	9900 2750 10250 2750
-Wire Wire Line
-	10250 2750 10250 2800
-Connection ~ 10250 2750
-Wire Wire Line
-	10250 2750 10600 2750
-Wire Wire Line
-	9900 2450 9900 2750
-Wire Wire Line
-	10000 2550 9800 2550
-Text GLabel 9800 2550 0    50   Input ~ 0
-SAFE_STATE_FLAG
+	9900 2850 9900 2900
+Text GLabel 10350 1200 2    50   Input ~ 0
+~SAFE_STATE_FLAG
 Wire Notes Line
-	9050 3100 11100 3100
+	9050 3150 11100 3150
 Wire Notes Line
 	9050 650  11100 650
@@
 	3400 1300 3400 2950
 Text GLabel 1850 1550 2    50   Input ~ 0
-SAFE_STATE_FLAG
+~SAFE_STATE_FLAG
 Wire Wire Line
 	5100 1200 5900 1200
@@
 Wire Wire Line
 	5250 4600 5750 4600
-Wire Wire Line
-	10500 1050 10600 1050
-Wire Wire Line
-	10600 1050 10600 1150
-Connection ~ 10600 1550
-Wire Wire Line
-	10500 1450 10600 1450
-Connection ~ 10600 1450
-Wire Wire Line
-	10600 1450 10600 1550
-Wire Wire Line
-	10500 1350 10600 1350
-Connection ~ 10600 1350
-Wire Wire Line
-	10600 1350 10600 1450
-Wire Wire Line
-	10500 1250 10600 1250
-Connection ~ 10600 1250
-Wire Wire Line
-	10600 1250 10600 1350
-Wire Wire Line
-	10500 1150 10600 1150
-Connection ~ 10600 1150
-Wire Wire Line
-	10600 1150 10600 1250
-Wire Wire Line
-	10500 2450 10700 2450
-Wire Wire Line
-	10500 2250 10700 2250
-Wire Wire Line
-	10500 2050 10700 2050
-Wire Wire Line
-	10600 1950 10600 2150
-Wire Wire Line
-	10600 2150 10500 2150
-Connection ~ 10600 1950
-Wire Wire Line
-	10600 2150 10600 2350
-Wire Wire Line
-	10600 2350 10500 2350
-Connection ~ 10600 2150
-Wire Wire Line
-	10600 2350 10600 2550
-Wire Wire Line
-	10600 2550 10500 2550
-Connection ~ 10600 2350
-Wire Wire Line
-	10600 2750 10600 2550
-Connection ~ 10600 2550
+Connection ~ 9550 2200
+Wire Wire Line
+	9650 2300 9550 2300
+Connection ~ 9550 2300
+Wire Wire Line
+	9550 2300 9550 2200
+Wire Wire Line
+	9650 2400 9550 2400
+Connection ~ 9550 2400
+Wire Wire Line
+	9550 2400 9550 2300
+Wire Wire Line
+	9650 2500 9550 2500
+Connection ~ 9550 2500
+Wire Wire Line
+	9550 2500 9550 2400
+Wire Wire Line
+	9650 2600 9550 2600
+Wire Wire Line
+	9550 2600 9550 2500
+Wire Wire Line
+	9650 1900 9450 1900
+Wire Wire Line
+	9550 1200 9650 1200
 $Comp
 L power:GND1 #PWR0102
@@
 Wire Wire Line
 	5600 6400 5600 7350
+Wire Wire Line
+	9450 2700 9650 2700
+Text GLabel 10350 2700 2    50   Input ~ 0
+24V
+Wire Wire Line
+	10350 2700 10150 2700
+Wire Wire Line
+	10250 2500 10250 2600
+Wire Wire Line
+	10250 2600 10150 2600
+Connection ~ 10250 2500
+Wire Wire Line
+	10350 1200 10150 1200
+Wire Wire Line
+	9450 1500 9650 1500
+Wire Wire Line
+	9450 1700 9650 1700
+Wire Wire Line
+	9550 1200 9550 1300
+Wire Wire Line
+	9550 1300 9650 1300
+Connection ~ 9550 1300
+Wire Wire Line
+	9550 1300 9550 1400
+Wire Wire Line
+	9550 1400 9650 1400
+Connection ~ 9550 1400
+Wire Wire Line
+	9550 1400 9550 1600
+Wire Wire Line
+	10150 1300 10250 1300
+Wire Wire Line
+	10250 1300 10250 1400
+Wire Wire Line
+	10250 2000 10250 1900
+Connection ~ 10250 2000
+Connection ~ 10250 1400
+Wire Wire Line
+	10250 1400 10150 1400
+Wire Wire Line
+	9550 1600 9650 1600
+Connection ~ 9550 1600
+Wire Wire Line
+	9550 1600 9550 1800
+Wire Wire Line
+	9550 1800 9650 1800
+Connection ~ 9550 1800
+Wire Wire Line
+	9550 1800 9550 2000
+Wire Wire Line
+	10150 1900 10250 1900
+Connection ~ 10250 1900
+Wire Wire Line
+	10250 1900 10250 1800
+Wire Wire Line
+	10150 1800 10250 1800
+Connection ~ 10250 1800
+Wire Wire Line
+	10250 1800 10250 1700
+Wire Wire Line
+	10150 1700 10250 1700
+Connection ~ 10250 1700
+Wire Wire Line
+	10250 1700 10250 1600
+Wire Wire Line
+	10150 1600 10250 1600
+Connection ~ 10250 1600
+Wire Wire Line
+	10250 1600 10250 1500
+Wire Wire Line
+	10150 1500 10250 1500
+Connection ~ 10250 1500
+Wire Wire Line
+	10250 1500 10250 1400
+Wire Wire Line
+	9900 2850 9550 2850
+Wire Wire Line
+	9550 2850 9550 2600
+Connection ~ 9550 2600
+Wire Wire Line
+	9900 2850 10250 2850
+Wire Wire Line
+	10250 2850 10250 2600
+Connection ~ 9900 2850
+Connection ~ 10250 2600
+Wire Notes Line
+	11100 650  11100 3150
+Wire Notes Line
+	9050 650  9050 3150
 $EndSCHEMATC
