File: MC-ADC/Voltage_Regulation.sch (KiCad schematic (older format))
At the start: 8 parts

Commit message: ADC work
Parts:
- added C?: 2.2 uF, Capacitor_SMD:C_1210_3225Metric, symbol Device:C_Small
- added C? (x2): unpopulated, Capacitor_SMD:C_1210_3225Metric, symbol Device:C_Small
- added L?: 10uH, Inductor_SMD:L_1812_4532Metric_Pad1.30x3.40mm_HandSolder, symbol Device:L_Small
- added U?: NMK2412SC, symbol MC-ADC:NMK2412SC
Connections:
- net labels added: -12V, 0V, 12V
- wire segments 33 -> 59
Other:
- note added: "24V -> +/-12V Circuit"
- moved on the sheet: C?, L?, U?

Commit message: ADC Updates!
Parts:
- removed C?: unpopulated, Capacitor_SMD:C_1210_3225Metric, symbol Device:C_Small
- removed C?: 4.7 uF, Capacitor_SMD:C_1210_3225Metric, symbol Device:C_Small
- removed L?: 3.9uH, Inductor_SMD:L_1812_4532Metric_Pad1.30x3.40mm_HandSolder, symbol Device:L_Small
- removed U?: R-78E3.3-0.5, symbol MC-ADC:R-78E3.3-0.5
- added R?: 750R, symbol Device:R_Small_US
- added R?: 2.5KOhm, symbol Device:R_Small_US
Connections:
- net labels added: +12V, 1.5V
- net labels removed: 12V, 3V3
- wire segments 59 -> 52
Other:
- note added: "5V -> 1.5V Circuit"
- note removed: "24V -> 3.3V Circuit"
- moved on the sheet: C?, L?, U?

Commit message: ADC
Parts:
- added C?: unpopulated, Capacitor_SMD:C_1210_3225Metric, symbol Device:C_Small
- added C?: 4.7 uF, Capacitor_SMD:C_1210_3225Metric, symbol Device:C_Small
- added L?: 3.9uH, Inductor_SMD:L_1812_4532Metric_Pad1.30x3.40mm_HandSolder, symbol Device:L_Small
- added U?: R-78E3.3-0.5, symbol MC-ADC:R-78E3.3-0.5
- R?: value 750R -> 900R
- R?: value 2.5KOhm -> 2KOhm
Connections:
- net labels added: 3V3
- wire segments 52 -> 67
Other:
- note added: "24V -> 3.3V Circuit"
- note added: "3.3V -> 1.5V Circuit ( High precision resistors )\ntolerance = 0.25%"
- note removed: "5V -> 1.5V Circuit"
- moved on the sheet: C?, L?, R?, U?

Commit message: ADC Work
Parts:
- removed C?: unpopulated, Capacitor_SMD:C_1210_3225Metric, symbol Device:C_Small
- removed C?: 4.7 uF, Capacitor_SMD:C_1210_3225Metric, symbol Device:C_Small
- removed L?: 3.9uH, Inductor_SMD:L_1812_4532Metric_Pad1.30x3.40mm_HandSolder, symbol Device:L_Small
- removed R?: 900R, symbol Device:R_Small_US
- removed R?: 2KOhm, symbol Device:R_Small_US
- removed U?: R-78E5.0-0.5, symbol MC-ADC:R-78E5.0-0.5
- removed U?: R-78E3.3-0.5, symbol MC-ADC:R-78E3.3-0.5
- added C?: 4.7 uF, Capacitor_SMD:C_1210_3225Metric, symbol Device:C_Small
- added C?: unpopulated, Capacitor_SMD:C_1210_3225Metric, symbol Device:C_Small
- added L?: 3.9uH, Inductor_SMD:L_1812_4532Metric_Pad1.30x3.40mm_HandSolder, symbol Device:L_Small
- added U? (x2): NMK2405SAC, symbol MC-ADC:NMK2405SAC
Connections:
- net labels added: -5V, 3VREF
- net labels removed: 1.5V, 3V3
- wire segments 67 -> 66
Other:
- note added: "24V -> +5V Circuit"
- note added: "24V -> -5V Circuit"
- note added: "Waiting for 3V reference selection"
- note removed: "24V -> 3.3V Circuit"
- note removed: "24V -> 5V Circuit"
- note removed: "3.3V -> 1.5V Circuit ( High precision resistors )\ntolerance = 0.25%"
- moved on the sheet: C?
Changed lines of the file:
@@
 $EndDescr
 Text Notes 5500 1450 0    50   ~ 0
-24V -> 5V Circuit
+24V -> +5V Circuit
 Wire Wire Line
 	3500 1950 3500 2150
-Text HLabel 4600 2250 0    50   Output ~ 0
+Text HLabel 5250 2450 0    50   Output ~ 0
 5V
 Connection ~ 3750 1950
@@
 L Device:C_Small C?
 U 1 1 617C79EA
-P 5450 2450
-F 0 "C?" H 5542 2496 50  0000 L CNN
-F 1 "unpopulated" H 5542 2405 50  0000 L CNN
-F 2 "Capacitor_SMD:C_1210_3225Metric" H 5450 2450 50  0001 C CNN
-F 3 "~" H 5450 2450 50  0001 C CNN
-	1    5450 2450
-	1    0    0    -1
-$EndComp
-Wire Wire Line
-	5450 2550 5450 2900
-Wire Wire Line
-	5450 2900 5650 2900
+P 5550 2600
+F 0 "C?" H 5642 2646 50  0000 L CNN
+F 1 "unpopulated" H 5642 2555 50  0000 L CNN
+F 2 "Capacitor_SMD:C_1210_3225Metric" H 5550 2600 50  0001 C CNN
+F 3 "~" H 5550 2600 50  0001 C CNN
+	1    5550 2600
+	1    0    0    -1
+$EndComp
+Wire Wire Line
+	5550 2700 5550 3050
+Wire Wire Line
+	5550 3050 5750 3050
 Text HLabel 1250 1650 0    50   Input ~ 0
 Vdd
-Text Notes 7000 4000 0    50   ~ 0
-3.3V -> 1.5V Circuit ( High precision resistors )\ntolerance = 0.25%
-Wire Wire Line
-	1700 1650 3750 1650
-Wire Wire Line
-	1250 1650 1700 1650
-Wire Wire Line
-	5450 2250 5450 2350
 $Comp
 L Device:L_Small L?
@@
 $EndComp
 Wire Wire Line
-	4350 1650 5450 1650
-Wire Wire Line
 	3750 1950 5300 1950
-$Comp
-L MC-ADC:R-78E5.0-0.5 U?
-U 1 1 61FA343C
-P 5800 1500
-F 0 "U?" H 6128 1246 50  0000 L CNN
-F 1 "R-78E5.0-0.5" H 6128 1155 50  0000 L CNN
-F 2 "" H 5800 1500 50  0001 C CNN
-F 3 "" H 5800 1500 50  0001 C CNN
-	1    5800 1500
-	1    0    0    -1
-$EndComp
 Wire Wire Line
 	5300 1950 5300 1800
-Wire Wire Line
-	5300 1800 5450 1800
-Connection ~ 5450 2250
-Wire Wire Line
-	5450 1950 5450 2250
-Connection ~ 1700 1650
 $Comp
 L MC-ADC:NMK2412SC U?
@@
 Text Notes 5500 5300 0    50   ~ 0
 24V -> +/-12V Circuit
-Text HLabel 5650 2900 2    50   Input ~ 0
+Text HLabel 5750 3050 2    50   Input ~ 0
 0V
+Text HLabel 4450 2250 0    50   Input ~ 0
+0V
+Wire Wire Line
+	1250 1650 1700 1650
+Wire Wire Line
+	1700 1650 3750 1650
+Connection ~ 1700 1650
+Wire Wire Line
+	1700 1650 1700 4050
+$Comp
+L MC-ADC:NMK2405SAC U?
+U 1 1 62216D88
+P 5900 1400
+F 0 "U?" H 6228 971 50  0000 L CNN
+F 1 "NMK2405SAC" H 6228 880 50  0000 L CNN
+F 2 "" H 5900 1400 50  0001 C CNN
+F 3 "" H 5900 1400 50  0001 C CNN
+	1    5900 1400
+	1    0    0    -1
+$EndComp
+$Comp
+L MC-ADC:NMK2405SAC U?
+U 1 1 62218407
+P 5950 3400
+F 0 "U?" H 6278 2971 50  0000 L CNN
+F 1 "NMK2405SAC" H 6278 2880 50  0000 L CNN
+F 2 "" H 5950 3400 50  0001 C CNN
+F 3 "" H 5950 3400 50  0001 C CNN
+	1    5950 3400
+	1    0    0    -1
+$EndComp
+Wire Wire Line
+	4350 1650 5550 1650
 Text HLabel 3500 2150 0    50   Input ~ 0
+GND
+Wire Wire Line
+	5300 1800 5550 1800
+Wire Wire Line
+	4450 2250 5400 2250
+Wire Wire Line
+	5400 2250 5400 1950
+Wire Wire Line
+	5400 1950 5550 1950
+Wire Wire Line
+	5550 2100 5550 2450
+Wire Wire Line
+	5550 2450 5250 2450
+Connection ~ 5550 2450
+Wire Wire Line
+	5550 2450 5550 2500
+$Comp
+L Device:L_Small L?
+U 1 1 622238BD
+P 4250 4050
+F 0 "L?" V 4450 4050 50  0000 L CNN
+F 1 "3.9uH" V 4350 3950 50  0000 L CNN
+F 2 "Inductor_SMD:L_1812_4532Metric_Pad1.30x3.40mm_HandSolder" H 4250 4050 50  0001 C CNN
+F 3 "https://www.digikey.com/en/products/detail/recom-power/RLS-126/9920565" H 4250 4050 50  0001 C CNN
+	1    4250 4050
+	0    -1   -1   0
+$EndComp
+$Comp
+L Device:C_Small C?
+U 1 1 622238C4
+P 3750 3850
+F 0 "C?" H 3842 3896 50  0000 L CNN
+F 1 "4.7 uF" H 3842 3805 50  0000 L CNN
+F 2 "Capacitor_SMD:C_1210_3225Metric" H 3750 3850 50  0001 C CNN
+F 3 "~" H 3750 3850 50  0001 C CNN
+	1    3750 3850
+	1    0    0    -1
+$EndComp
+Wire Wire Line
+	1700 4050 3750 4050
+Wire Wire Line
+	3500 3650 3750 3650
+Wire Wire Line
+	3750 3750 3750 3650
+Connection ~ 3750 3650
+Wire Wire Line
+	3750 3950 3750 4050
+Connection ~ 3750 4050
+Wire Wire Line
+	3750 4050 4150 4050
+Wire Wire Line
+	3500 3650 3500 3450
+Text HLabel 3500 3450 0    50   Input ~ 0
+GND
+Connection ~ 1700 4050
+Wire Wire Line
+	1700 4050 1700 5500
+Wire Wire Line
+	3750 3650 5600 3650
+Wire Wire Line
+	4350 4050 4650 4050
+Wire Wire Line
+	4650 4050 4650 3800
+Wire Wire Line
+	4650 3800 5600 3800
+Wire Wire Line
+	5600 3950 4800 3950
+Wire Wire Line
+	4800 3950 4800 4400
+Wire Wire Line
+	4800 4400 4500 4400
+Text HLabel 4500 4400 0    50   Input ~ 0
 0V
-Text HLabel 7350 5000 2    50   Input ~ 0
-0V
-$Comp
-L Device:R_Small_US R?
-U 1 1 622D70A9
-P 6800 4200
-F 0 "R?" H 6868 4246 50  0000 L CNN
-F 1 "900R" H 6868 4155 50  0000 L CNN
-F 2 "" H 6800 4200 50  0001 C CNN
-F 3 "~" H 6800 4200 50  0001 C CNN
-	1    6800 4200
-	1    0    0    -1
-$EndComp
-$Comp
-L Device:R_Small_US R?
-U 1 1 622D7F6F
-P 6800 4650
-F 0 "R?" H 6868 4696 50  0000 L CNN
-F 1 "2KOhm" H 6868 4605 50  0000 L CNN
-F 2 "" H 6800 4650 50  0001 C CNN
-F 3 "~" H 6800 4650 50  0001 C CNN
-	1    6800 4650
-	1    0    0    -1
-$EndComp
-Wire Wire Line
-	6800 4100 6800 4000
-Wire Wire Line
-	6800 4750 6800 5000
-Wire Wire Line
-	6800 5000 7350 5000
-Wire Wire Line
-	6800 4300 6800 4400
-Text HLabel 7350 4400 2    50   Input ~ 0
-1.5V
-Wire Wire Line
-	6800 4400 7350 4400
-Connection ~ 6800 4400
-Wire Wire Line
-	6800 4400 6800 4550
-$Comp
-L MC-ADC:R-78E3.3-0.5 U?
-U 1 1 62156CA7
-P 5850 3300
-F 0 "U?" H 6178 3046 50  0000 L CNN
-F 1 "R-78E3.3-0.5" H 6178 2955 50  0000 L CNN
-F 2 "" H 5850 3300 50  0001 C CNN
-F 3 "" H 5850 3300 50  0001 C CNN
-	1    5850 3300
-	1    0    0    -1
-$EndComp
-Wire Wire Line
-	1700 1650 1700 3450
-Wire Wire Line
-	4600 2250 5450 2250
-$Comp
-L Device:C_Small C?
-U 1 1 62166F66
-P 5450 4250
-F 0 "C?" H 5542 4296 50  0000 L CNN
-F 1 "unpopulated" H 5542 4205 50  0000 L CNN
-F 2 "Capacitor_SMD:C_1210_3225Metric" H 5450 4250 50  0001 C CNN
-F 3 "~" H 5450 4250 50  0001 C CNN
-	1    5450 4250
-	1    0    0    -1
-$EndComp
-Wire Wire Line
-	5450 4350 5450 4700
-Wire Wire Line
-	5450 4700 5650 4700
-Text HLabel 5650 4700 2    50   Input ~ 0
-0V
-Wire Wire Line
-	5450 3750 5500 3750
-Text Notes 5500 3250 0    50   ~ 0
-24V -> 3.3V Circuit
-$Comp
-L Device:L_Small L?
-U 1 1 6216D879
-P 4200 3450
-F 0 "L?" V 4400 3450 50  0000 L CNN
-F 1 "3.9uH" V 4300 3350 50  0000 L CNN
-F 2 "Inductor_SMD:L_1812_4532Metric_Pad1.30x3.40mm_HandSolder" H 4200 3450 50  0001 C CNN
-F 3 "https://www.digikey.com/en/products/detail/recom-power/RLS-126/9920565" H 4200 3450 50  0001 C CNN
-	1    4200 3450
-	0    -1   -1   0
-$EndComp
-$Comp
-L Device:C_Small C?
-U 1 1 6216D87F
-P 3750 3600
-F 0 "C?" H 3842 3646 50  0000 L CNN
-F 1 "4.7 uF" H 3842 3555 50  0000 L CNN
-F 2 "Capacitor_SMD:C_1210_3225Metric" H 3750 3600 50  0001 C CNN
-F 3 "~" H 3750 3600 50  0001 C CNN
-	1    3750 3600
-	1    0    0    -1
-$EndComp
-Wire Wire Line
-	3750 3500 3750 3450
-Wire Wire Line
-	3750 3450 4100 3450
-Wire Wire Line
-	3750 3700 3750 3750
-Wire Wire Line
-	3500 3750 3500 3950
-Text HLabel 3500 3950 0    50   Input ~ 0
-0V
-Wire Wire Line
-	3500 3750 3750 3750
-Wire Wire Line
-	4300 3450 5500 3450
-Wire Wire Line
-	4250 3750 4250 3600
-Wire Wire Line
-	3750 3750 4250 3750
-Connection ~ 3750 3750
-Wire Wire Line
-	4250 3600 5500 3600
-Wire Wire Line
-	3750 3450 1700 3450
-Connection ~ 3750 3450
-Connection ~ 1700 3450
-Wire Wire Line
-	1700 3450 1700 5500
-Wire Wire Line
-	5450 3750 5450 4000
-Connection ~ 5450 4000
-Wire Wire Line
-	5450 4000 5450 4150
-Wire Wire Line
-	5450 4000 6800 4000
-Wire Wire Line
-	5450 4000 5150 4000
-Text HLabel 5150 4000 0    50   Input ~ 0
-3V3
+$Comp
+L Device:C_Small C?
+U 1 1 62239962
+P 5600 4600
+F 0 "C?" H 5692 4646 50  0000 L CNN
+F 1 "unpopulated" H 5692 4555 50  0000 L CNN
+F 2 "Capacitor_SMD:C_1210_3225Metric" H 5600 4600 50  0001 C CNN
+F 3 "~" H 5600 4600 50  0001 C CNN
+	1    5600 4600
+	1    0    0    -1
+$EndComp
+Wire Wire Line
+	5600 4700 5600 4850
+Wire Wire Line
+	5600 4100 5600 4450
+Wire Wire Line
+	5600 4450 5300 4450
+Connection ~ 5600 4450
+Wire Wire Line
+	5600 4450 5600 4500
+Wire Wire Line
+	4800 4400 4800 4850
+Wire Wire Line
+	4800 4850 5600 4850
+Connection ~ 4800 4400
+Text HLabel 5300 4450 0    50   Input ~ 0
+-5V
+Text Notes 5600 3400 0    50   ~ 0
+24V -> -5V Circuit
+Text Notes 7300 4350 0    50   ~ 0
+Waiting for 3V reference selection
+Text HLabel 7950 4500 0    50   Input ~ 0
+3VREF
 $EndSCHEMATC

Commit message: ADC Work
Parts:
- removed C? (x2): unpopulated, Capacitor_SMD:C_1210_3225Metric, symbol Device:C_Small
- removed C? (x2): 4.7 uF, Capacitor_SMD:C_1210_3225Metric, symbol Device:C_Small
- removed L? (x2): 3.9uH, Inductor_SMD:L_1812_4532Metric_Pad1.30x3.40mm_HandSolder, symbol Device:L_Small
- removed U? (x2): NMK2405SAC, symbol MC-ADC:NMK2405SAC
- added C10: 4.7 uF, Capacitor_SMD:C_1210_3225Metric, symbol Device:C_Small
- added C14, C15, C17: 0.1 uF, Capacitor_SMD:C_1210_3225Metric, symbol Device:C_Small
- added C16: 10 uF, Capacitor_SMD:C_1210_3225Metric, symbol Device:C_Small
- added C18: unpopulated, Capacitor_SMD:C_1210_3225Metric, symbol Device:C_Small
- added L10: 3.9 uH, Inductor_SMD:L_1812_4532Metric_Pad1.30x3.40mm_HandSolder, symbol Device:L_Small
- added R10: 1.87K, Resistor_SMD:R_0603_1608Metric, symbol Device:R_Small_US
- added R11: 1.43K, Resistor_SMD:R_0603_1608Metric, symbol Device:R_Small_US
- added R12: 30.9K, Resistor_SMD:R_1206_3216Metric, symbol Device:R_Small_US
- added R13: 1.07K, Resistor_SMD:R_1206_3216Metric, symbol Device:R_Small_US
- added U10: MAX6216, symbol MC-ADC:MAX6216
- added U11: R-78E3.3-0.5, symbol MC-ADC:R-78E3.3-0.5
- L11: renamed from L?; footprint Inductor_SMD:L_1812_4532Metric_Pad1.30x3.40mm_HandSolder -> (none)
- gave numbers to parts that had none: 4
Connections:
- net labels added: VREF, VSE+, VSE-
- net labels removed: -5V, 0V, 3VREF, 5V
- wire segments 66 -> 84
Other:
- note added: "+/- 11.64 to 12.6V"
- note added: "-0.421V to -0.389V"
- note added: "1.3V"
- note added: "24V -> 3.3V Circuit"
- note added: "Approx. -0.4V"
- note added: "Approx. 3.3V"
- note removed: "24V -> +5V Circuit"
- note removed: "24V -> -5V Circuit"
- note removed: "Waiting for 3V reference selection"

Commit message: ADC Work + Start Layout
Parts:
- removed U12: NMK2412SC, symbol MC-ADC:NMK2412SC
- added U12: RD-2412D_P, Footprints_MC-ADC:RD-2412D, symbol MC-ADC:RD-2412D_P
- L11: footprint (none) -> Footprints_MC-ADC:INDPM4040X190N
- U10: value MAX6216 -> MAX6126AASA30+; footprint (none) -> Package_SO:SOIC-8_3.9x4.9mm_P1.27mm
- U11: footprint (none) -> Package_SIP:SIP3_11.6x8.5mm
Connections:
- net +12V: now also U12.6 (+Vout)
- net -12V: now also U12.4 (-Vout)
- net GND: now also U12.2 (-Vin), U12.5 (0V)
- net at L11.2: now also U12.1 (+Vin)
Other:
- note added: "3.99V to 3.201V"
Changed lines of the file:
@@
 Vdd
-$Comp
-L MC-ADC:NMK2412SC U12
-U 1 1 621121F5
-P 5850 5250
-F 0 "U12" H 6178 4746 50  0000 L CNN
-F 1 "NMK2412SC" H 6178 4655 50  0000 L CNN
-F 2 "" H 5850 5250 50  0001 C CNN
-F 3 "" H 5850 5250 50  0001 C CNN
-	1    5850 5250
-	1    0    0    -1
-$EndComp
 $Comp
 L Device:L_Small L11
@@
 F 0 "L11" V 4400 5500 50  0000 L CNN
 F 1 "10uH" V 4300 5400 50  0000 L CNN
-F 2 "" H 4200 5500 50  0001 C CNN
-F 3 "" H 4200 5500 50  0001 C CNN
+F 2 "Footprints_MC-ADC:INDPM4040X190N" H 4200 5500 50  0001 C CNN
+F 3 "https://www.digikey.com/en/products/detail/vishay-dale/IFSC1515AHER100M01/2744232" H 4200 5500 50  0001 C CNN
 	1    4200 5500
 	0    -1   -1   0
@@
 F 1 "2.2 uF" H 3842 5605 50  0000 L CNN
 F 2 "Capacitor_SMD:C_1210_3225Metric" H 3750 5650 50  0001 C CNN
-F 3 "~" H 3750 5650 50  0001 C CNN
+F 3 "https://www.digikey.com/en/products/detail/taiyo-yuden/GMK325BJ225KN-T/930725" H 3750 5650 50  0001 C CNN
 	1    3750 5650
 	1    0    0    -1
@@
 F 0 "U11" H 6178 3446 50  0000 L CNN
 F 1 "R-78E3.3-0.5" H 6178 3355 50  0000 L CNN
-F 2 "" H 5850 3700 50  0001 C CNN
-F 3 "" H 5850 3700 50  0001 C CNN
+F 2 "Package_SIP:SIP3_11.6x8.5mm" H 5850 3700 50  0001 C CNN
+F 3 "https://www.mouser.com/ProductDetail/RECOM-Power/R-78E33-05?qs=sGAEpiMZZMuyVE%2FzJ6Hm15MDYDf%252Bvm5TgPIMDw4suvM%3D" H 5850 3700 50  0001 C CNN
 	1    5850 3700
 	1    0    0    -1
@@
 F 1 "3.9 uH" V 4300 3750 50  0000 L CNN
 F 2 "Inductor_SMD:L_1812_4532Metric_Pad1.30x3.40mm_HandSolder" H 4200 3850 50  0001 C CNN
-F 3 "https://www.digikey.com/en/products/detail/recom-power/RLS-126/9920565" H 4200 3850 50  0001 C CNN
+F 3 "https://www.digikey.com/en/products/detail/recom-power/RLS-397/9920568" H 4200 3850 50  0001 C CNN
 	1    4200 3850
 	0    -1   -1   0
@@
 F 1 "4.7 uF" H 3842 3955 50  0000 L CNN
 F 2 "Capacitor_SMD:C_1210_3225Metric" H 3750 4000 50  0001 C CNN
-F 3 "~" H 3750 4000 50  0001 C CNN
+F 3 "https://www.digikey.com/en/products/detail/kyocera-avx/12105C475K4Z2A/2512117" H 3750 4000 50  0001 C CNN
 	1    3750 4000
 	1    0    0    -1
@@
 U 1 1 6236B85D
 P 5800 1650
+AR Path="/6236B85D" Ref="U10"  Part="1"
+AR Path="/61F9F3BA/6236B85D" Ref="U10"  Part="1"
 F 0 "U10" H 5900 1665 50  0000 C CNN
-F 1 "MAX6216" H 5900 1574 50  0000 C CNN
-F 2 "" H 5800 1650 50  0001 C CNN
-F 3 "" H 5800 1650 50  0001 C CNN
+F 1 "MAX6126AASA30+" H 5900 1574 50  0000 C CNN
+F 2 "Package_SO:SOIC-8_3.9x4.9mm_P1.27mm" H 5800 1650 50  0001 C CNN
+F 3 "https://www.digikey.com/en/products/detail/analog-devices-inc-maxim-integrated/MAX6126AASA30/1867184?s=N4IgjCBcpg7LBOKoDGUBmBDANgZwKYA0IA9lANogBMADFQGxWwgC6xADgC5QgDKnAJwCWAOwDmIAL7EAtFWQg0kQQFcipCiACsIYkhbSQMpNEVRV6spEoQDh%2BdZABZAIIANemAYuXvF60kgA" H 5800 1650 50  0001 C CNN
 	1    5800 1650
 	1    0    0    -1
@@
 F 1 "0.1 uF" H 4142 2405 50  0000 L CNN
 F 2 "Capacitor_SMD:C_1210_3225Metric" H 4050 2450 50  0001 C CNN
-F 3 "~" H 4050 2450 50  0001 C CNN
+F 3 "https://www.digikey.com/en/products/detail/kyocera-avx/12105C104KAT2A/563725" H 4050 2450 50  0001 C CNN
 	1    4050 2450
 	1    0    0    -1
@@
 F 1 "0.1 uF" H 4692 2405 50  0000 L CNN
 F 2 "Capacitor_SMD:C_1210_3225Metric" H 4600 2450 50  0001 C CNN
-F 3 "~" H 4600 2450 50  0001 C CNN
+F 3 "https://www.digikey.com/en/products/detail/kyocera-avx/12105C104KAT2A/563725" H 4600 2450 50  0001 C CNN
 	1    4600 2450
 	1    0    0    -1
@@
 F 1 "10 uF" H 6892 2255 50  0000 L CNN
 F 2 "Capacitor_SMD:C_1210_3225Metric" H 6800 2300 50  0001 C CNN
-F 3 "~" H 6800 2300 50  0001 C CNN
+F 3 "https://www.digikey.com/en/products/detail/samsung-electro-mechanics/CL32A106KLULNNE/3888965" H 6800 2300 50  0001 C CNN
 	1    6800 2300
 	1    0    0    -1
@@
 F 1 "0.1 uF" H 7392 2255 50  0000 L CNN
 F 2 "Capacitor_SMD:C_1210_3225Metric" H 7300 2300 50  0001 C CNN
-F 3 "~" H 7300 2300 50  0001 C CNN
+F 3 "https://www.digikey.com/en/products/detail/kyocera-avx/12105C104KAT2A/563725" H 7300 2300 50  0001 C CNN
 	1    7300 2300
 	1    0    0    -1
@@
 Text Notes 8650 5500 0    50   ~ 0
 -0.421V to -0.389V
+$Comp
+L MC-ADC:RD-2412D_P U12
+U 1 1 622B3159
+P 5850 5250
+F 0 "U12" H 6178 4746 50  0000 L CNN
+F 1 "RD-2412D_P" H 6178 4655 50  0000 L CNN
+F 2 "Footprints_MC-ADC:RD-2412D" H 5850 5250 50  0001 C CNN
+F 3 "https://www.digikey.com/en/products/detail/recom-power/RD-2412D-P/2303678?s=N4IgTCBcDaIEoBEC0YAsBGMCD0AFEAugL5A" H 5850 5250 50  0001 C CNN
+	1    5850 5250
+	1    0    0    -1
+$EndComp
+Text Notes 4600 4750 0    50   ~ 0
+3.99V to 3.201V
 $EndSCHEMATC

Commit message: ADC Work + Layout
Parts:
- removed U10: MAX6126AASA30+, Package_SO:SOIC-8_3.9x4.9mm_P1.27mm, symbol MC-ADC:MAX6216
- added U10: MAX6126AASA30+, Package_SO:SOIC-8_3.9x4.9mm_P1.27mm, symbol MC-ADC:MAX6126AASA30+
Connections:
- net GND: now also U10.3 (GND), U10.4 (GNDS)
- net Vdd: now also U10.2 (IN)
- net at C14.1: now also U10.1 (NR)
- net at C16.1, C17.1, R10.1: now also U10.6 (OUTS), U10.7 (OUTF)
Changed lines of the file:
@@
 Wire Wire Line
 	5500 4750 5500 5000
-$Comp
-L MC-ADC:MAX6216 U10
-U 1 1 6236B85D
-P 5800 1650
-AR Path="/6236B85D" Ref="U10"  Part="1"
-AR Path="/61F9F3BA/6236B85D" Ref="U10"  Part="1"
-F 0 "U10" H 5900 1665 50  0000 C CNN
-F 1 "MAX6126AASA30+" H 5900 1574 50  0000 C CNN
-F 2 "Package_SO:SOIC-8_3.9x4.9mm_P1.27mm" H 5800 1650 50  0001 C CNN
-F 3 "https://www.digikey.com/en/products/detail/analog-devices-inc-maxim-integrated/MAX6126AASA30/1867184?s=N4IgjCBcpg7LBOKoDGUBmBDANgZwKYA0IA9lANogBMADFQGxWwgC6xADgC5QgDKnAJwCWAOwDmIAL7EAtFWQg0kQQFcipCiACsIYkhbSQMpNEVRV6spEoQDh%2BdZABZAIIANemAYuXvF60kgA" H 5800 1650 50  0001 C CNN
-	1    5800 1650
-	1    0    0    -1
-$EndComp
 Wire Wire Line
 	5500 2050 4600 2050
@@
 Text Notes 4600 4750 0    50   ~ 0
 3.99V to 3.201V
+$Comp
+L MC-ADC:MAX6126AASA30+ U10
+U 1 1 62296BB3
+P 5800 1650
+F 0 "U10" H 5900 1665 50  0000 C CNN
+F 1 "MAX6126AASA30+" H 5900 1574 50  0000 C CNN
+F 2 "Package_SO:SOIC-8_3.9x4.9mm_P1.27mm" H 5800 1650 50  0001 C CNN
+F 3 "https://www.digikey.com/en/products/detail/analog-devices-inc-maxim-integrated/MAX6126AASA30/1867184?s=N4IgjCBcpg7LBOKoDGUBmBDANgZwKYA0IA9lANogBMADFQGxWwgC6xADgC5QgDKnAJwCWAOwDmIAL7EAtFWQg0kQQFcipCiACsIYkhbSQMpNEVRV6spEoQDh%2BdZABZAIIANemAYuXvF60kgA" H 5800 1650 50  0001 C CNN
+	1    5800 1650
+	1    0    0    -1
+$EndComp
 $EndSCHEMATC
