File: MC-Backplane/Backplane.kicad_pcb (KiCad board)
At the start: 2 copper layers, 17 parts, among them J1 1730010, J21 86094328314755V1LF, J22 86094328314755V1LF, J40 374472, J41 86094328314755V1LF, J42 86094328314755V1LF, J43 86094328314755V1LF, U11 86094328314755V1LF, U12 86094328314755V1LF, U13 86094328314755V1LF, U16 86094328314755V1LF, U17 86094328314755V1LF, U18 86094328314755V1LF, U51 64600001223, U52 SISS05DN-T1-GE3

Commit message: schematic reorg and layout begins
Parts:
- removed D51: BZX84C9V1-7-F, Package_TO_SOT_SMD:SOT-23_Handsoldering
- removed J21, J22, J41, J42, J43: 86094328314755V1LF, 86094328314755V1LF
- removed J40: 374472, Footprints_MC-Backplane:374472
- removed R51: 3k, Resistor_SMD:R_1206_3216Metric
- removed U16, U17, U18: 86094328314755V1LF, Footprints_MC-Backplane:86094328314755V1LF
- removed U51: 64600001223, Footprints_MC-Backplane:64600001223
- removed U52: SISS05DN-T1-GE3, Footprints_MC-Backplane:Vishay_PowerPAK_1212-8_Single
- added D1: BZX84C9V1-7-F, Package_TO_SOT_SMD:SOT-23_Handsoldering, F.Cu at (226.4, 11.7)
- added H1: 86094327313755E1LF, Footprints_MC-FO:86094327313755E1LF, F.Cu at (20.2, 95.9)
- added R1: 3k, Resistor_SMD:R_1206_3216Metric, F.Cu at (232.5, 11.0)
- added REF**: MountingHole_3.2mm_M3, MountingHole:MountingHole_3.2mm_M3, F.Cu at (449.2, 34.6)
- added REF**: MountingHole_3.2mm_M3, MountingHole:MountingHole_3.2mm_M3, F.Cu at (78.4, 34.4)
- added REF**: MountingHole_3.2mm_M3, MountingHole:MountingHole_3.2mm_M3, F.Cu at (357.8, 157.1)
- added REF**: MountingHole_3.2mm_M3, MountingHole:MountingHole_3.2mm_M3, F.Cu at (362.9, 157.1)
- added REF**: MountingHole_3.2mm_M3, MountingHole:MountingHole_3.2mm_M3, F.Cu at (368.0, 157.1)
- added REF**: MountingHole_3.2mm_M3, MountingHole:MountingHole_3.2mm_M3, F.Cu at (408.6, 157.1)
- added REF**: MountingHole_3.2mm_M3, MountingHole:MountingHole_3.2mm_M3, F.Cu at (403.6, 157.1)
- added REF**: MountingHole_3.2mm_M3, MountingHole:MountingHole_3.2mm_M3, F.Cu at (286.7, 157.1)
- added REF**: MountingHole_3.2mm_M3, MountingHole:MountingHole_3.2mm_M3, F.Cu at (291.8, 157.1)
- added REF**: MountingHole_3.2mm_M3, MountingHole:MountingHole_3.2mm_M3, F.Cu at (261.3, 157.1)
- added REF**: MountingHole_3.2mm_M3, MountingHole:MountingHole_3.2mm_M3, F.Cu at (296.9, 157.1)
- added REF**: MountingHole_3.2mm_M3, MountingHole:MountingHole_3.2mm_M3, F.Cu at (246.1, 157.0)
- added REF**: MountingHole_3.2mm_M3, MountingHole:MountingHole_3.2mm_M3, F.Cu at (98.7, 34.4)
- added REF**: MountingHole_3.2mm_M3, MountingHole:MountingHole_3.2mm_M3, F.Cu at (251.2, 157.0)
- added REF**: MountingHole_3.2mm_M3, MountingHole:MountingHole_3.2mm_M3, F.Cu at (281.6, 157.1)
- added REF**: MountingHole_3.2mm_M3, MountingHole:MountingHole_3.2mm_M3, F.Cu at (256.2, 157.1)
- added REF**: MountingHole_3.2mm_M3, MountingHole:MountingHole_3.2mm_M3, F.Cu at (276.6, 157.1)
- added REF**: MountingHole_3.2mm_M3, MountingHole:MountingHole_3.2mm_M3, F.Cu at (271.5, 157.1)
- added REF**: MountingHole_3.2mm_M3, MountingHole:MountingHole_3.2mm_M3, F.Cu at (266.4, 157.1)
- added REF**: MountingHole_3.2mm_M3, MountingHole:MountingHole_3.2mm_M3, F.Cu at (230.8, 157.0)
- added REF**: MountingHole_3.2mm_M3, MountingHole:MountingHole_3.2mm_M3, F.Cu at (220.7, 157.0)
- added REF**: MountingHole_3.2mm_M3, MountingHole:MountingHole_3.2mm_M3, F.Cu at (225.8, 157.0)
- added REF**: MountingHole_3.2mm_M3, MountingHole:MountingHole_3.2mm_M3, F.Cu at (215.6, 157.0)
- added REF**: MountingHole_3.2mm_M3, MountingHole:MountingHole_3.2mm_M3, F.Cu at (93.6, 34.4)
- added REF**: MountingHole_3.2mm_M3, MountingHole:MountingHole_3.2mm_M3, F.Cu at (210.5, 157.0)
- added REF**: MountingHole_3.2mm_M3, MountingHole:MountingHole_3.2mm_M3, F.Cu at (205.4, 157.0)
- added REF**: MountingHole_3.2mm_M3, MountingHole:MountingHole_3.2mm_M3, F.Cu at (190.2, 157.0)
- added REF**: MountingHole_3.2mm_M3, MountingHole:MountingHole_3.2mm_M3, F.Cu at (195.3, 157.0)
- added REF**: MountingHole_3.2mm_M3, MountingHole:MountingHole_3.2mm_M3, F.Cu at (200.4, 157.0)
- added REF**: MountingHole_3.2mm_M3, MountingHole:MountingHole_3.2mm_M3, F.Cu at (302.0, 157.1)
- added REF**: MountingHole_3.2mm_M3, MountingHole:MountingHole_3.2mm_M3, F.Cu at (327.4, 157.1)
- added REF**: MountingHole_3.2mm_M3, MountingHole:MountingHole_3.2mm_M3, F.Cu at (241.0, 157.0)
- added REF**: MountingHole_3.2mm_M3, MountingHole:MountingHole_3.2mm_M3, F.Cu at (317.2, 157.1)
- added REF**: MountingHole_3.2mm_M3, MountingHole:MountingHole_3.2mm_M3, F.Cu at (347.7, 157.1)
- added REF**: MountingHole_3.2mm_M3, MountingHole:MountingHole_3.2mm_M3, F.Cu at (88.5, 34.4)
- added REF**: MountingHole_3.2mm_M3, MountingHole:MountingHole_3.2mm_M3, F.Cu at (352.8, 157.1)
- added REF**: MountingHole_3.2mm_M3, MountingHole:MountingHole_3.2mm_M3, F.Cu at (337.5, 157.1)
- added REF**: MountingHole_3.2mm_M3, MountingHole:MountingHole_3.2mm_M3, F.Cu at (235.9, 157.0)
- added REF**: MountingHole_3.2mm_M3, MountingHole:MountingHole_3.2mm_M3, F.Cu at (307.0, 157.1)
- added REF**: MountingHole_3.2mm_M3, MountingHole:MountingHole_3.2mm_M3, F.Cu at (312.1, 157.1)
- added REF**: MountingHole_3.2mm_M3, MountingHole:MountingHole_3.2mm_M3, F.Cu at (332.4, 157.1)
- added REF**: MountingHole_3.2mm_M3, MountingHole:MountingHole_3.2mm_M3, F.Cu at (322.3, 157.1)
- added REF**: MountingHole_3.2mm_M3, MountingHole:MountingHole_3.2mm_M3, F.Cu at (342.6, 157.1)
- added REF**: MountingHole_3.2mm_M3, MountingHole:MountingHole_3.2mm_M3, F.Cu at (175.0, 157.0)
- added REF**: MountingHole_3.2mm_M3, MountingHole:MountingHole_3.2mm_M3, F.Cu at (164.8, 157.0)
- added REF**: MountingHole_3.2mm_M3, MountingHole:MountingHole_3.2mm_M3, F.Cu at (388.2, 34.6)
- added REF**: MountingHole_3.2mm_M3, MountingHole:MountingHole_3.2mm_M3, F.Cu at (169.9, 157.0)
- added REF**: MountingHole_3.2mm_M3, MountingHole:MountingHole_3.2mm_M3, F.Cu at (159.7, 157.0)
- added REF**: MountingHole_3.2mm_M3, MountingHole:MountingHole_3.2mm_M3, F.Cu at (154.6, 157.0)
- added REF**: MountingHole_3.2mm_M3, MountingHole:MountingHole_3.2mm_M3, F.Cu at (149.6, 157.0)
- added REF**: MountingHole_3.2mm_M3, MountingHole:MountingHole_3.2mm_M3, F.Cu at (134.3, 157.0)
- added REF**: MountingHole_3.2mm_M3, MountingHole:MountingHole_3.2mm_M3, F.Cu at (139.4, 157.0)
- added REF**: MountingHole_3.2mm_M3, MountingHole:MountingHole_3.2mm_M3, F.Cu at (144.5, 157.0)
- added REF**: MountingHole_3.2mm_M3, MountingHole:MountingHole_3.2mm_M3, F.Cu at (185.1, 157.0)
- added REF**: MountingHole_3.2mm_M3, MountingHole:MountingHole_3.2mm_M3, F.Cu at (180.0, 157.0)
- added REF**: MountingHole_3.2mm_M3, MountingHole:MountingHole_3.2mm_M3, F.Cu at (119.1, 157.0)
- added REF**: MountingHole_3.2mm_M3, MountingHole:MountingHole_3.2mm_M3, F.Cu at (403.5, 34.6)
- added REF**: MountingHole_3.2mm_M3, MountingHole:MountingHole_3.2mm_M3, F.Cu at (108.9, 157.0)
- added REF**: MountingHole_3.2mm_M3, MountingHole:MountingHole_3.2mm_M3, F.Cu at (114.0, 157.0)
- added REF**: MountingHole_3.2mm_M3, MountingHole:MountingHole_3.2mm_M3, F.Cu at (103.8, 157.0)
- added REF**: MountingHole_3.2mm_M3, MountingHole:MountingHole_3.2mm_M3, F.Cu at (98.8, 157.0)
- added REF**: MountingHole_3.2mm_M3, MountingHole:MountingHole_3.2mm_M3, F.Cu at (93.7, 157.0)
- added REF**: MountingHole_3.2mm_M3, MountingHole:MountingHole_3.2mm_M3, F.Cu at (78.4, 157.0)
- added REF**: MountingHole_3.2mm_M3, MountingHole:MountingHole_3.2mm_M3, F.Cu at (83.5, 157.0)
- added REF**: MountingHole_3.2mm_M3, MountingHole:MountingHole_3.2mm_M3, F.Cu at (88.6, 157.0)
- added REF**: MountingHole_3.2mm_M3, MountingHole:MountingHole_3.2mm_M3, F.Cu at (129.2, 157.0)
- added REF**: MountingHole_3.2mm_M3, MountingHole:MountingHole_3.2mm_M3, F.Cu at (124.2, 157.0)
- added REF**: MountingHole_3.2mm_M3, MountingHole:MountingHole_3.2mm_M3, F.Cu at (408.6, 34.6)
- added REF**: MountingHole_3.2mm_M3, MountingHole:MountingHole_3.2mm_M3, F.Cu at (73.4, 157.0)
- added REF**: MountingHole_3.2mm_M3, MountingHole:MountingHole_3.2mm_M3, F.Cu at (68.3, 157.0)
- added REF**: MountingHole_3.2mm_M3, MountingHole:MountingHole_3.2mm_M3, F.Cu at (63.2, 157.0)
- added REF**: MountingHole_3.2mm_M3, MountingHole:MountingHole_3.2mm_M3, F.Cu at (58.1, 157.0)
- added REF**: MountingHole_3.2mm_M3, MountingHole:MountingHole_3.2mm_M3, F.Cu at (48.0, 157.0)
- added REF**: MountingHole_3.2mm_M3, MountingHole:MountingHole_3.2mm_M3, F.Cu at (53.0, 157.0)
- added REF**: MountingHole_3.2mm_M3, MountingHole:MountingHole_3.2mm_M3, F.Cu at (42.9, 157.0)
- added REF**: MountingHole_3.2mm_M3, MountingHole:MountingHole_3.2mm_M3, F.Cu at (37.8, 157.0)
- added REF**: MountingHole_3.2mm_M3, MountingHole:MountingHole_3.2mm_M3, F.Cu at (27.6, 156.9)
- added REF**: MountingHole_3.2mm_M3, MountingHole:MountingHole_3.2mm_M3, F.Cu at (22.6, 156.9)
- added REF**: MountingHole_3.2mm_M3, MountingHole:MountingHole_3.2mm_M3, F.Cu at (428.9, 34.6)
- added REF**: MountingHole_3.2mm_M3, MountingHole:MountingHole_3.2mm_M3, F.Cu at (32.7, 157.0)
- added REF**: MountingHole_3.2mm_M3, MountingHole:MountingHole_3.2mm_M3, F.Cu at (413.6, 34.6)
- added REF**: MountingHole_3.2mm_M3, MountingHole:MountingHole_3.2mm_M3, F.Cu at (423.8, 34.6)
- added REF**: MountingHole_3.2mm_M3, MountingHole:MountingHole_3.2mm_M3, F.Cu at (444.1, 34.6)
- added REF**: MountingHole_3.2mm_M3, MountingHole:MountingHole_3.2mm_M3, F.Cu at (434.0, 34.6)
- added REF**: MountingHole_3.2mm_M3, MountingHole:MountingHole_3.2mm_M3, F.Cu at (439.0, 34.6)
- added REF**: MountingHole_3.2mm_M3, MountingHole:MountingHole_3.2mm_M3, F.Cu at (378.1, 34.6)
- added REF**: MountingHole_3.2mm_M3, MountingHole:MountingHole_3.2mm_M3, F.Cu at (362.8, 34.6)
- added REF**: MountingHole_3.2mm_M3, MountingHole:MountingHole_3.2mm_M3, F.Cu at (383.2, 34.6)
- added REF**: MountingHole_3.2mm_M3, MountingHole:MountingHole_3.2mm_M3, F.Cu at (373.0, 34.6)
- added REF**: MountingHole_3.2mm_M3, MountingHole:MountingHole_3.2mm_M3, F.Cu at (347.6, 34.5)
- added REF**: MountingHole_3.2mm_M3, MountingHole:MountingHole_3.2mm_M3, F.Cu at (352.7, 34.5)
- added REF**: MountingHole_3.2mm_M3, MountingHole:MountingHole_3.2mm_M3, F.Cu at (398.4, 34.6)
- added REF**: MountingHole_3.2mm_M3, MountingHole:MountingHole_3.2mm_M3, F.Cu at (367.9, 34.6)
- added REF**: MountingHole_3.2mm_M3, MountingHole:MountingHole_3.2mm_M3, F.Cu at (108.8, 34.4)
- added REF**: MountingHole_3.2mm_M3, MountingHole:MountingHole_3.2mm_M3, F.Cu at (357.8, 34.6)
- added REF**: MountingHole_3.2mm_M3, MountingHole:MountingHole_3.2mm_M3, F.Cu at (393.3, 34.6)
- added REF**: MountingHole_3.2mm_M3, MountingHole:MountingHole_3.2mm_M3, F.Cu at (53.0, 34.4)
- added REF**: MountingHole_3.2mm_M3, MountingHole:MountingHole_3.2mm_M3, F.Cu at (42.8, 34.4)
- added REF**: MountingHole_3.2mm_M3, MountingHole:MountingHole_3.2mm_M3, F.Cu at (47.9, 34.4)
- added REF**: MountingHole_3.2mm_M3, MountingHole:MountingHole_3.2mm_M3, F.Cu at (37.7, 34.4)
- added REF**: MountingHole_3.2mm_M3, MountingHole:MountingHole_3.2mm_M3, F.Cu at (32.6, 34.4)
- added REF**: MountingHole_3.2mm_M3, MountingHole:MountingHole_3.2mm_M3, F.Cu at (27.6, 34.4)
- added REF**: MountingHole_3.2mm_M3, MountingHole:MountingHole_3.2mm_M3, F.Cu at (22.5, 34.4)
- added REF**: MountingHole_3.2mm_M3, MountingHole:MountingHole_3.2mm_M3, F.Cu at (418.7, 34.6)
- added REF**: MountingHole_3.2mm_M3, MountingHole:MountingHole_3.2mm_M3, F.Cu at (113.9, 34.4)
- added REF**: MountingHole_3.2mm_M3, MountingHole:MountingHole_3.2mm_M3, F.Cu at (235.8, 34.5)
- added REF**: MountingHole_3.2mm_M3, MountingHole:MountingHole_3.2mm_M3, F.Cu at (276.5, 34.5)
- added REF**: MountingHole_3.2mm_M3, MountingHole:MountingHole_3.2mm_M3, F.Cu at (271.4, 34.5)
- added REF**: MountingHole_3.2mm_M3, MountingHole:MountingHole_3.2mm_M3, F.Cu at (281.6, 34.5)
- added REF**: MountingHole_3.2mm_M3, MountingHole:MountingHole_3.2mm_M3, F.Cu at (286.6, 34.5)
- added REF**: MountingHole_3.2mm_M3, MountingHole:MountingHole_3.2mm_M3, F.Cu at (240.9, 34.5)
- added REF**: MountingHole_3.2mm_M3, MountingHole:MountingHole_3.2mm_M3, F.Cu at (251.1, 34.5)
- added REF**: MountingHole_3.2mm_M3, MountingHole:MountingHole_3.2mm_M3, F.Cu at (246.0, 34.5)
- added REF**: MountingHole_3.2mm_M3, MountingHole:MountingHole_3.2mm_M3, F.Cu at (266.3, 34.5)
- added REF**: MountingHole_3.2mm_M3, MountingHole:MountingHole_3.2mm_M3, F.Cu at (261.2, 34.5)
- added REF**: MountingHole_3.2mm_M3, MountingHole:MountingHole_3.2mm_M3, F.Cu at (83.4, 34.4)
- added REF**: MountingHole_3.2mm_M3, MountingHole:MountingHole_3.2mm_M3, F.Cu at (256.2, 34.5)
- added REF**: MountingHole_3.2mm_M3, MountingHole:MountingHole_3.2mm_M3, F.Cu at (317.1, 34.5)
- added REF**: MountingHole_3.2mm_M3, MountingHole:MountingHole_3.2mm_M3, F.Cu at (220.6, 34.5)
- added REF**: MountingHole_3.2mm_M3, MountingHole:MountingHole_3.2mm_M3, F.Cu at (210.4, 34.5)
- added REF**: MountingHole_3.2mm_M3, MountingHole:MountingHole_3.2mm_M3, F.Cu at (215.5, 34.5)
- added REF**: MountingHole_3.2mm_M3, MountingHole:MountingHole_3.2mm_M3, F.Cu at (195.2, 34.5)
- added REF**: MountingHole_3.2mm_M3, MountingHole:MountingHole_3.2mm_M3, F.Cu at (230.8, 34.5)
- added REF**: MountingHole_3.2mm_M3, MountingHole:MountingHole_3.2mm_M3, F.Cu at (205.4, 34.5)
- added REF**: MountingHole_3.2mm_M3, MountingHole:MountingHole_3.2mm_M3, F.Cu at (200.3, 34.5)
- added REF**: MountingHole_3.2mm_M3, MountingHole:MountingHole_3.2mm_M3, F.Cu at (180.0, 34.5)
- added REF**: MountingHole_3.2mm_M3, MountingHole:MountingHole_3.2mm_M3, F.Cu at (119.0, 34.4)
- added REF**: MountingHole_3.2mm_M3, MountingHole:MountingHole_3.2mm_M3, F.Cu at (185.0, 34.5)
- added REF**: MountingHole_3.2mm_M3, MountingHole:MountingHole_3.2mm_M3, F.Cu at (190.1, 34.5)
- added REF**: MountingHole_3.2mm_M3, MountingHole:MountingHole_3.2mm_M3, F.Cu at (291.7, 34.5)
- added REF**: MountingHole_3.2mm_M3, MountingHole:MountingHole_3.2mm_M3, F.Cu at (307.0, 34.5)
- added REF**: MountingHole_3.2mm_M3, MountingHole:MountingHole_3.2mm_M3, F.Cu at (337.4, 34.5)
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Connections:
- J1 pad 1: GND -> /GND
- U11 pad A1: 24V -> /24V
- U11 pad A10: GND -> /DSP/ADC_15
- U11 pad A11: /DSPSlot/GD_GPIO14_RESET -> /GND
- U11 pad A12: GND -> /Analog3/ADC_3
- U11 pad A13: GPIO12_EMITTER_ENABLE -> /GND
- U11 pad A14: GND -> /GND
- U11 pad A15: ~GPIO13_SAFE_STATE_FLAG~ -> /GND
- U11 pad A16: GND -> /~SAFE_STATE_FLAG~
- U11 pad A2: 24V -> /24V
- U11 pad A3: GND -> /GND
- U11 pad A4: GND -> /GND
- U11 pad A5: GND -> /GND
- U11 pad A6: GND -> /GND
- U11 pad A7: GND -> /GND
- U11 pad A8: GND -> /Analog3/ADC_1
- U11 pad A9: GND -> /GND
- U11 pad B1: GND -> /GND
- U11 pad B10: Net-(U11-PadB10) -> /GND
- U11 pad B11: Net-(U11-PadB10) -> /GND
- U11 pad B12: Net-(U11-PadB10) -> /GND
- U11 pad B13: Net-(U11-PadB10) -> /GND
- U11 pad B14: Net-(U11-PadB10) -> /GND
- U11 pad B15: Net-(U11-PadB10) -> /GND
- U11 pad B16: Net-(U11-PadB10) -> /GND
- U11 pad B2: GND -> /GND
- U11 pad B3: GND -> /GND
- U11 pad B4: GND -> /GND
- U11 pad B5: GND -> /GND
- U11 pad B6: GND -> /GND
- U11 pad B7: GND -> /GND
- U11 pad B8: GND -> /GND
- U11 pad B9: GND -> /GND
- U11 pad C1: Net-(U11-PadB10) -> /GND
- U11 pad C10: /DSPSlot/GD1_EPWM_11B -> /GND
- U11 pad C11: Net-(U11-PadB10) -> /Analog3/ADC_4
- U11 pad C12: /DSPSlot/GD1_GPIO52_STATUS_2 -> /GND
- U11 pad C13: Net-(U11-PadB10) -> /Analog3/ADC_5
- U11 pad C14: Net-(U11-PadB10) -> /GND
- U11 pad C15: Net-(U11-PadB10) -> /Analog3/ADC_6
- U11 pad C16: CLOCK -> /GND
- U11 pad C2: /DSPSlot/GD1_EPWM_12A -> /GND
- U11 pad C3: Net-(U11-PadB10) -> /GND
- U11 pad C4: /DSPSlot/GD1_EPWM_12B -> /GND
- U11 pad C5: Net-(U11-PadB10) -> /GND
- U11 pad C6: /DSPSlot/GD1_GPIO53_STATUS_1 -> /GND
- U11 pad C7: Net-(U11-PadB10) -> /GND
- U11 pad C8: /DSPSlot/GD1_EPWM_11A -> /GND
- U11 pad C9: Net-(U11-PadB10) -> /GND
- U12 pad A1: 24V -> /Analog1/ADC_6
- U12 pad A10: GND -> /GND
- U12 pad A11: /DSPSlot/GD_GPIO14_RESET -> /24V
- U12 pad A12: GND -> /GND
- U12 pad A13: GPIO12_EMITTER_ENABLE -> /DSP/SD1_D2
- U12 pad A14: GND -> /GND
- U12 pad A15: ~GPIO13_SAFE_STATE_FLAG~ -> /DSP/SD2_D1
- U12 pad A16: GND -> /GND
- U12 pad A2: 24V -> /GND
- U12 pad A3: GND -> /Analog1/ADC_1
- U12 pad A4: GND -> /GND
- U12 pad A5: GND -> /Analog2/ADC_2
- U12 pad A6: GND -> /GND
- U12 pad A7: GND -> /Analog3/ADC_3
- U12 pad A8: GND -> /GND
- U12 pad A9: GND -> /GND
- U12 pad B1: GND -> /GND
- U12 pad B10: GND -> /GND
- U12 pad B11: GND -> /GND
- U12 pad B12: GND -> /24V
- U12 pad B13: GND -> /GND
- U12 pad B14: GND -> /SD1/PWMA_CLK_OUT
- U12 pad B15: GND -> /GND
- U12 pad B16: GND -> /DSP/SD2_D4
- U12 pad B2: GND -> /Analog1/ADC_3
- U12 pad B3: GND -> /GND
- U12 pad B4: GND -> /Analog2/ADC_4
- U12 pad B5: GND -> /GND
- U12 pad B6: GND -> /Analog3/ADC_5
- U12 pad B7: GND -> /GND
- U12 pad B8: GND -> /GND
- U12 pad B9: GND -> /GND
- U12 pad C1: GND -> /Analog1/ADC_5
- U12 pad C10: /GateDriveSlots/GD2_EPWM_9B -> /GND
- U12 pad C11: GND -> /24V
- U12 pad C12: /DSPSlot/GD2_GPIO44_STATUS_2 -> /GND
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Routing:
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Other:
- board outline added: 431.8 x 132.6 mm
- copper layers 2 -> 4

Commit message: placement done- tracks started
Parts:
- removed H1: 86094327313755E1LF, Footprints_MC-FO:86094327313755E1LF
- removed the REF** at (449.2, 34.6)
- removed the REF** at (78.4, 34.4)
- removed the REF** at (357.8, 157.1)
- removed the REF** at (362.9, 157.1)
- removed the REF** at (368.0, 157.1)
- removed the REF** at (408.6, 157.1)
- removed the REF** at (403.6, 157.1)
- removed the REF** at (98.7, 34.4)
- removed the REF** at (93.6, 34.4)
- removed the REF** at (327.4, 157.1)
- removed the REF** at (317.2, 157.1)
- removed the REF** at (347.7, 157.1)
- removed the REF** at (88.5, 34.4)
- removed the REF** at (352.8, 157.1)
- removed the REF** at (337.5, 157.1)
- removed the REF** at (332.4, 157.1)
- removed the REF** at (322.3, 157.1)
- removed the REF** at (342.6, 157.1)
- removed the REF** at (388.2, 34.6)
- removed the REF** at (403.5, 34.6)
- removed the REF** at (408.6, 34.6)
- removed the REF** at (428.9, 34.6)
- removed the REF** at (413.6, 34.6)
- removed the REF** at (423.8, 34.6)
- removed the REF** at (444.1, 34.6)
- removed the REF** at (434.0, 34.6)
- removed the REF** at (439.0, 34.6)
- removed the REF** at (378.1, 34.6)
- removed the REF** at (362.8, 34.6)
- removed the REF** at (383.2, 34.6)
- removed the REF** at (373.0, 34.6)
- removed the REF** at (347.6, 34.5)
- removed the REF** at (352.7, 34.5)
- removed the REF** at (398.4, 34.6)
- removed the REF** at (367.9, 34.6)
- removed the REF** at (108.8, 34.4)
- removed the REF** at (357.8, 34.6)
- removed the REF** at (393.3, 34.6)
- removed the REF** at (53.0, 34.4)
- removed the REF** at (42.8, 34.4)
- removed the REF** at (47.9, 34.4)
- removed the REF** at (37.7, 34.4)
- removed the REF** at (32.6, 34.4)
- removed the REF** at (27.6, 34.4)
- removed the REF** at (22.5, 34.4)
- removed the REF** at (418.7, 34.6)
- removed the REF** at (113.9, 34.4)
- removed the REF** at (235.8, 34.5)
- removed the REF** at (276.5, 34.5)
- removed the REF** at (271.4, 34.5)
- removed the REF** at (281.6, 34.5)
- removed the REF** at (286.6, 34.5)
- removed the REF** at (240.9, 34.5)
- removed the REF** at (251.1, 34.5)
- removed the REF** at (246.0, 34.5)
- removed the REF** at (266.3, 34.5)
- removed the REF** at (261.2, 34.5)
- removed the REF** at (83.4, 34.4)
- removed the REF** at (256.2, 34.5)
- removed the REF** at (317.1, 34.5)
- removed the REF** at (220.6, 34.5)
- removed the REF** at (210.4, 34.5)
- removed the REF** at (215.5, 34.5)
- removed the REF** at (195.2, 34.5)
- removed the REF** at (230.8, 34.5)
- removed the REF** at (205.4, 34.5)
- removed the REF** at (200.3, 34.5)
- removed the REF** at (180.0, 34.5)
- removed the REF** at (119.0, 34.4)
- removed the REF** at (185.0, 34.5)
- removed the REF** at (190.1, 34.5)
- removed the REF** at (291.7, 34.5)
- removed the REF** at (307.0, 34.5)
- removed the REF** at (337.4, 34.5)
- removed the REF** at (342.5, 34.5)
- removed the REF** at (327.3, 34.5)
- removed the REF** at (296.8, 34.5)
- removed the REF** at (301.9, 34.5)
- removed the REF** at (312.0, 34.5)
- removed the REF** at (68.2, 34.4)
- removed the REF** at (124.1, 34.4)
- removed the REF** at (149.5, 34.5)
- removed the REF** at (63.1, 34.4)
- removed the REF** at (139.3, 34.5)
- removed the REF** at (169.8, 34.5)
- removed the REF** at (174.9, 34.5)
- removed the REF** at (322.2, 34.5)
- removed the REF** at (159.6, 34.5)
- removed the REF** at (58.0, 34.4)
- removed the REF** at (332.4, 34.5)
- removed the REF** at (73.3, 34.4)
- removed the REF** at (129.2, 34.4)
- removed the REF** at (134.2, 34.5)
- removed the REF** at (154.6, 34.5)
- removed the REF** at (225.7, 34.5)
- removed the REF** at (144.4, 34.5)
- removed the REF** at (164.7, 34.5)
- removed the REF** at (429.0, 157.1)
- removed the REF** at (449.3, 157.1)
- removed the REF** at (444.2, 157.1)
- removed the REF** at (434.0, 157.1)
- removed the REF** at (103.8, 34.4)
- removed the REF** at (439.1, 157.1)
- removed the REF** at (423.9, 157.1)
- removed the REF** at (413.7, 157.1)
- removed the REF** at (418.8, 157.1)
- removed the REF** at (398.5, 157.1)
- removed the REF** at (388.3, 157.1)
- removed the REF** at (393.4, 157.1)
- removed the REF** at (383.2, 157.1)
- removed the REF** at (378.2, 157.1)
- removed the REF** at (373.1, 157.1)
- J1: moved to B.Cu
- moved J1 404.1 mm to (40.3, 46.8), turned to 270 degrees
- moved U2 220.5 mm to (28.1, 79.2), turned to 270 degrees
- moved R1 218.1 mm to (29.0, 89.5), turned to 270 degrees
- moved D1 211.4 mm to (28.0, 84.5), turned to 90 degrees
- moved U1 203.8 mm to (28.4, 51.8), turned to 270 degrees
- moved U11 108.8 mm to (307.7, 108.9)
- moved U5 98.1 mm to (287.4, 108.9)
- moved U10 85.6 mm to (267.1, 108.9)
- moved U12 74.4 mm to (226.2, 135.1)
- moved U4 42.6 mm to (196.0, 127.5)
- moved U3 34.6 mm to (175.6, 127.5)
- moved U8 27.2 mm to (155.3, 114.8)
- moved U9 25.5 mm to (135.0, 114.8)
- moved U7 23.2 mm to (114.7, 114.8)
- moved U14 17.3 mm to (94.3, 114.8)
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Connections:
- U12 pad A10: /GND -> /24V
- U12 pad A13: /DSP/SD1_D2 -> /GND
- U12 pad A15: /DSP/SD2_D1 -> /DSP/SD2_D2
- U12 pad A17: /SD2/PWMA_CLK_OUT -> /GND
- U12 pad A31: /DSP/GD1_EPWM_11A -> /DSP/GD1_EPWM_12B
- U12 pad B10: /GND -> /24V
- U12 pad B12: /24V -> /DSP/SD1_D4
- U12 pad B14: /SD1/PWMA_CLK_OUT -> /GND
- U12 pad B16: /DSP/SD2_D4 -> /SD2/PWMA_CLK_OUT
- U12 pad B32: /DSP/GD1_GPIO52_STATUS_2 -> /DSP/GD1_GPIO53_STATUS_1
- U12 pad B9: /GND -> /24V
- U12 pad C11: /24V -> /DSP/SD1_D2
- U12 pad C13: /DSP/SD1_D3 -> /SD1/PWMA_CLK_OUT
- U12 pad C15: /DSP/SD2_D2 -> /DSP/SD2_D4
- U12 pad C31: /DSP/GD1_EPWM_12B -> /DSP/GD1_EPWM_11A
- U12 pad D12: /DSP/SD1_D1 -> /DSP/SD1_D3
- U12 pad D14: /SD1/PWMB_CLK_OUT -> /DSP/SD2_D1
- U12 pad D32: /DSP/GD1_GPIO53_STATUS_1 -> /DSP/GD1_GPIO52_STATUS_2
- U12 pad E11: /GND -> /DSP/SD1_D1
- U12 pad E13: /DSP/SD1_D4 -> /SD1/PWMB_CLK_OUT
- U3 pad A1: /24V -> /GND
- U3 pad A10: /GND -> /SD1/PWMA_CLK_OUT
- U3 pad A4: /GND -> /DSP/SD1_D2
- U3 pad A6: /GND -> /DSP/SD1_D1
- U3 pad C1: /GND -> /24V
- U3 pad C10: /GND -> /SD1/PWMB_CLK_OUT
- U3 pad C11: /DSP/SD1_D3 -> /GND
- U3 pad C13: /DSP/SD1_D4 -> /GND
- U3 pad C2: /GND -> /24V
- U3 pad C3: /SD1/PWMA_CLK_OUT -> /GND
- U3 pad C5: /SD1/PWMB_CLK_OUT -> /GND
- U3 pad C6: /GND -> /DSP/SD1_D4
- U3 pad C7: /DSP/SD1_D1 -> /GND
- U3 pad C8: /GND -> /DSP/SD1_D3
- U3 pad C9: /DSP/SD1_D2 -> /GND
- U4 pad A1: /24V -> /GND
- U4 pad A10: /GND -> /SD2/PWMA_CLK_OUT
- U4 pad A4: /GND -> /DSP/SD2_D2
- U4 pad A6: /GND -> /DSP/SD2_D1
- U4 pad C1: /GND -> /24V
- U4 pad C10: /GND -> /SD2/PWMB_CLK_OUT
- U4 pad C11: /DSP/SD2_D3 -> /GND
- U4 pad C13: /DSP/SD2_D4 -> /GND
- U4 pad C2: /GND -> /24V
- U4 pad C3: /SD2/PWMA_CLK_OUT -> /GND
- U4 pad C5: /SD2/PWMB_CLK_OUT -> /GND
- U4 pad C6: /GND -> /DSP/SD2_D4
- U4 pad C7: /DSP/SD2_D1 -> /GND
- U4 pad C8: /GND -> /DSP/SD2_D3
- U4 pad C9: /DSP/SD2_D2 -> /GND
Routing:
- net /24V: track 0.00 -> 270.3 mm, vias 0 -> 1
- net /DSP/GD1_EPWM_12B: track 0.00 -> 240.0 mm
- net /DSP/GD1_GPIO53_STATUS_1: track 0.00 -> 224.9 mm
- net /DSP/GD1_EPWM_12A: track 0.00 -> 211.5 mm
- net /DSP/GD1_GPIO52_STATUS_2: track 0.00 -> 202.9 mm
- net /DSP/SD1_D4: track 0.00 -> 56.2 mm
- net /DSP/SD1_D3: track 0.00 -> 49.9 mm
- net /DSP/SD1_D2: track 0.00 -> 49.7 mm
- net /SD1/PWMA_CLK_OUT: track 0.00 -> 46.4 mm
- net /DSP/SD1_D1: track 0.00 -> 42.5 mm
- net /DSP/SD2_D2: track 0.00 -> 40.0 mm
- net /DSP/SD2_D4: track 0.00 -> 36.5 mm
- net /DSP/GD1_EPWM_11A: track 0.00 -> 34.6 mm
- net /SD2/PWMB_CLK_OUT: track 0.00 -> 31.7 mm
- net /SD2/PWMA_CLK_OUT: track 0.00 -> 30.8 mm
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- added copper zone on In1.Cu, net /GND
- added copper zone on In2.Cu, net /GND
Other:
- board size 431.8 x 132.6 mm -> 294.6 x 132.6 mm

Commit message: layout done: cleaning up and checking MH
Parts:
- added REF**: MountingHole_3.2mm_M3, MountingHole:MountingHole_3.2mm_M3, F.Cu at (296.8, 34.4)
- added REF**: MountingHole_3.2mm_M3, MountingHole:MountingHole_3.2mm_M3, F.Cu at (261.3, 34.4)
- added REF**: MountingHole_3.2mm_M3, MountingHole:MountingHole_3.2mm_M3, F.Cu at (215.6, 34.4)
- added REF**: MountingHole_3.2mm_M3, MountingHole:MountingHole_3.2mm_M3, F.Cu at (307.0, 34.4)
- added REF**: MountingHole_3.2mm_M3, MountingHole:MountingHole_3.2mm_M3, F.Cu at (195.2, 34.4)
- added REF**: MountingHole_3.2mm_M3, MountingHole:MountingHole_3.2mm_M3, F.Cu at (230.8, 34.4)
- added REF**: MountingHole_3.2mm_M3, MountingHole:MountingHole_3.2mm_M3, F.Cu at (169.8, 34.4)
- added REF**: MountingHole_3.2mm_M3, MountingHole:MountingHole_3.2mm_M3, F.Cu at (241.0, 34.4)
- added REF**: MountingHole_3.2mm_M3, MountingHole:MountingHole_3.2mm_M3, F.Cu at (164.8, 34.4)
- added REF**: MountingHole_3.2mm_M3, MountingHole:MountingHole_3.2mm_M3, F.Cu at (210.5, 34.4)
- added REF**: MountingHole_3.2mm_M3, MountingHole:MountingHole_3.2mm_M3, F.Cu at (205.4, 34.4)
- added REF**: MountingHole_3.2mm_M3, MountingHole:MountingHole_3.2mm_M3, F.Cu at (271.4, 34.4)
- added REF**: MountingHole_3.2mm_M3, MountingHole:MountingHole_3.2mm_M3, F.Cu at (174.9, 34.4)
- added REF**: MountingHole_3.2mm_M3, MountingHole:MountingHole_3.2mm_M3, F.Cu at (312.1, 34.5)
- added REF**: MountingHole_3.2mm_M3, MountingHole:MountingHole_3.2mm_M3, F.Cu at (235.9, 34.4)
- added REF**: MountingHole_3.2mm_M3, MountingHole:MountingHole_3.2mm_M3, F.Cu at (200.3, 34.4)
- added REF**: MountingHole_3.2mm_M3, MountingHole:MountingHole_3.2mm_M3, F.Cu at (190.2, 34.4)
- added REF**: MountingHole_3.2mm_M3, MountingHole:MountingHole_3.2mm_M3, F.Cu at (225.7, 34.4)
- added REF**: MountingHole_3.2mm_M3, MountingHole:MountingHole_3.2mm_M3, F.Cu at (266.4, 34.4)
- added REF**: MountingHole_3.2mm_M3, MountingHole:MountingHole_3.2mm_M3, F.Cu at (220.6, 34.4)
- added REF**: MountingHole_3.2mm_M3, MountingHole:MountingHole_3.2mm_M3, F.Cu at (301.9, 34.4)
- added REF**: MountingHole_3.2mm_M3, MountingHole:MountingHole_3.2mm_M3, F.Cu at (32.7, 34.3)
- added REF**: MountingHole_3.2mm_M3, MountingHole:MountingHole_3.2mm_M3, F.Cu at (281.6, 34.4)
- added REF**: MountingHole_3.2mm_M3, MountingHole:MountingHole_3.2mm_M3, F.Cu at (22.5, 34.3)
- added REF**: MountingHole_3.2mm_M3, MountingHole:MountingHole_3.2mm_M3, F.Cu at (27.6, 34.3)
- added REF**: MountingHole_3.2mm_M3, MountingHole:MountingHole_3.2mm_M3, F.Cu at (42.8, 34.3)
- added REF**: MountingHole_3.2mm_M3, MountingHole:MountingHole_3.2mm_M3, F.Cu at (53.0, 34.3)
- added REF**: MountingHole_3.2mm_M3, MountingHole:MountingHole_3.2mm_M3, F.Cu at (47.9, 34.3)
- added REF**: MountingHole_3.2mm_M3, MountingHole:MountingHole_3.2mm_M3, F.Cu at (68.2, 34.3)
- added REF**: MountingHole_3.2mm_M3, MountingHole:MountingHole_3.2mm_M3, F.Cu at (58.1, 34.3)
- added REF**: MountingHole_3.2mm_M3, MountingHole:MountingHole_3.2mm_M3, F.Cu at (124.1, 34.4)
- added REF**: MountingHole_3.2mm_M3, MountingHole:MountingHole_3.2mm_M3, F.Cu at (73.3, 34.3)
- added REF**: MountingHole_3.2mm_M3, MountingHole:MountingHole_3.2mm_M3, F.Cu at (63.2, 34.3)
- added REF**: MountingHole_3.2mm_M3, MountingHole:MountingHole_3.2mm_M3, F.Cu at (246.0, 34.4)
- added REF**: MountingHole_3.2mm_M3, MountingHole:MountingHole_3.2mm_M3, F.Cu at (37.8, 34.3)
- added REF**: MountingHole_3.2mm_M3, MountingHole:MountingHole_3.2mm_M3, F.Cu at (108.9, 34.4)
- added REF**: MountingHole_3.2mm_M3, MountingHole:MountingHole_3.2mm_M3, F.Cu at (78.4, 34.3)
- added REF**: MountingHole_3.2mm_M3, MountingHole:MountingHole_3.2mm_M3, F.Cu at (93.6, 34.4)
- added REF**: MountingHole_3.2mm_M3, MountingHole:MountingHole_3.2mm_M3, F.Cu at (103.8, 34.4)
- added REF**: MountingHole_3.2mm_M3, MountingHole:MountingHole_3.2mm_M3, F.Cu at (119.0, 34.4)
- added REF**: MountingHole_3.2mm_M3, MountingHole:MountingHole_3.2mm_M3, F.Cu at (98.7, 34.4)
- added REF**: MountingHole_3.2mm_M3, MountingHole:MountingHole_3.2mm_M3, F.Cu at (185.1, 34.4)
- added REF**: MountingHole_3.2mm_M3, MountingHole:MountingHole_3.2mm_M3, F.Cu at (139.4, 34.4)
- added REF**: MountingHole_3.2mm_M3, MountingHole:MountingHole_3.2mm_M3, F.Cu at (149.5, 34.4)
- added REF**: MountingHole_3.2mm_M3, MountingHole:MountingHole_3.2mm_M3, F.Cu at (291.8, 34.4)
- added REF**: MountingHole_3.2mm_M3, MountingHole:MountingHole_3.2mm_M3, F.Cu at (159.7, 34.4)
- added REF**: MountingHole_3.2mm_M3, MountingHole:MountingHole_3.2mm_M3, F.Cu at (154.6, 34.4)
- added REF**: MountingHole_3.2mm_M3, MountingHole:MountingHole_3.2mm_M3, F.Cu at (134.3, 34.4)
- added REF**: MountingHole_3.2mm_M3, MountingHole:MountingHole_3.2mm_M3, F.Cu at (144.4, 34.4)
- added REF**: MountingHole_3.2mm_M3, MountingHole:MountingHole_3.2mm_M3, F.Cu at (129.2, 34.4)
- added REF**: MountingHole_3.2mm_M3, MountingHole:MountingHole_3.2mm_M3, F.Cu at (88.6, 34.4)
- added REF**: MountingHole_3.2mm_M3, MountingHole:MountingHole_3.2mm_M3, F.Cu at (114.0, 34.4)
- added REF**: MountingHole_3.2mm_M3, MountingHole:MountingHole_3.2mm_M3, F.Cu at (180.0, 34.4)
- added REF**: MountingHole_3.2mm_M3, MountingHole:MountingHole_3.2mm_M3, F.Cu at (83.5, 34.3)
- added REF**: MountingHole_3.2mm_M3, MountingHole:MountingHole_3.2mm_M3, F.Cu at (286.7, 34.4)
- added REF**: MountingHole_3.2mm_M3, MountingHole:MountingHole_3.2mm_M3, F.Cu at (276.5, 34.4)
- added REF**: MountingHole_3.2mm_M3, MountingHole:MountingHole_3.2mm_M3, F.Cu at (256.2, 34.4)
- added REF**: MountingHole_3.2mm_M3, MountingHole:MountingHole_3.2mm_M3, F.Cu at (251.1, 34.4)
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Connections:
- U10 pad A10: /Analog1/ADC_2 -> /GND
- U10 pad A11: /GND -> /DSP/ADC1_B5
- U10 pad A12: /Analog1/ADC_3 -> /GND
- U10 pad A13: /GND -> /DSP/ADC1_15
- U10 pad A2: /24V -> /GND
- U10 pad A8: /Analog1/ADC_1 -> /GND
- U10 pad A9: /GND -> /DSP/ADC1_D3
- U10 pad C1: /GND -> /24V
- U10 pad C11: /Analog1/ADC_4 -> /DSP/ADC1_B4
- U10 pad C13: /Analog1/ADC_5 -> /DSP/ADC1_14
- U10 pad C15: /Analog1/ADC_6 -> /GND
- U10 pad C9: /GND -> /DSP/ADC1_D2
- U11 pad A10: /DSP/ADC_15 -> /GND
- U11 pad A11: /GND -> /DSP/ADC3_B3
- U11 pad A12: /Analog3/ADC_3 -> /GND
- U11 pad A13: /GND -> /DSP/ADC3_A3
- U11 pad A2: /24V -> /GND
- U11 pad A8: /Analog3/ADC_1 -> /GND
- U11 pad A9: /GND -> /DSP/ADC3_C3
- U11 pad C1: /GND -> /24V
- U11 pad C11: /Analog3/ADC_4 -> /DSP/ADC3_B2
- U11 pad C13: /Analog3/ADC_5 -> /DSP/ADC3_A2
- U11 pad C15: /Analog3/ADC_6 -> /GND
- U11 pad C9: /GND -> /DSP/ADC3_C2
- U12 pad A1: /Analog1/ADC_6 -> /24V
- U12 pad A10: /24V -> /GND
- U12 pad A11: /24V -> /GND
- U12 pad A17: /GND -> /GD_GPIO14_RESET
- U12 pad A19: /DSP/GD6_EPWM_1A -> /DSP/GD6_GPIO16_STATUS_1
- U12 pad A21: /DSP/GD5_EPWM_3B -> /DSP/GD5_EPWM_3A
- U12 pad A23: /DSP/GD5_GPIO19_STATUS_1 -> /DSP/GD_EPWM_5B
- U12 pad A25: /DSP/GD4_GPIO22_STATUS_2 -> /DSP/GD3_GPIO24_STATUS_2
- U12 pad A3: /Analog1/ADC_1 -> /DSP/ADC3_C3
- U12 pad A31: /DSP/GD1_EPWM_12B -> /DSP/GD1_EPWM_12A
- U12 pad A5: /Analog2/ADC_2 -> /DSP/ADC3_A2
- U12 pad A7: /Analog3/ADC_3 -> /DSP/ADC2_A5
- U12 pad A9: /GND -> /DSP/ADC1_B4
- U12 pad B1: /GND -> /24V
- U12 pad B10: /24V -> /GND
- U12 pad B18: /GD_GPIO14_RESET -> /DSP/GD6_GPIO15_STATUS_2
- U12 pad B2: /Analog1/ADC_3 -> /GND
- U12 pad B20: /DSP/GD6_GPIO15_STATUS_2 -> /DSP/GD6_EPWM_2A
- U12 pad B22: /DSP/GD5_EPWM_4A -> /DSP/GD5_EPWM_4B
- U12 pad B24: /DSP/GD_EPWM_6B -> /DSP/GD4_GPIO23_STATUS_1
- U12 pad B30: /DSP/GD2_GPIO45_STATUS_1 -> /DSP/GD1_GPIO52_STATUS_2
- U12 pad B32: /DSP/GD1_GPIO53_STATUS_1 -> /DSP/GD1_EPWM_12B
- U12 pad B4: /Analog2/ADC_4 -> /DSP/ADC3_B2
- U12 pad B6: /Analog3/ADC_5 -> /DSP/ADC2_C5
- U12 pad B8: /GND -> /DSP/ADC1_D2
- U12 pad B9: /24V -> /GND
- U12 pad C1: /Analog1/ADC_5 -> /GND
- U12 pad C19: /DSP/GD6_EPWM_2B -> /DSP/GD6_EPWM_1A
- U12 pad C21: /DSP/GD5_EPWM_3A -> /DSP/GD5_EPWM_3B
- U12 pad C23: /DSP/GD_EPWM_5B -> /DSP/GD4_GPIO22_STATUS_2
- U12 pad C25: /DSP/GD4_GPIO23_STATUS_1 -> /DSP/GD_EPWM_6A
- U12 pad C27: /DSP/GD3_GPIO24_STATUS_2 -> /DSP/GD3_EPWM_8B
- U12 pad C29: /DSP/GD2_EPWM_10A -> /DSP/GD2_GPIO45_STATUS_1
- U12 pad C3: /Analog2/ADC_6 -> /DSP/ADC3_C2
- U12 pad C5: /Analog2/ADC_1 -> /DSP/ADC2_D1
- U12 pad C7: /DSP/ADC_15 -> /DSP/ADC2_A4
- U12 pad C9: /GND -> /DSP/ADC1_15
- U12 pad D18: /DSP/GD6_EPWM_1B -> /GND
- U12 pad D2: /Analog1/ADC_2 -> /GND
- U12 pad D20: /DSP/GD6_GPIO16_STATUS_1 -> /DSP/GD6_EPWM_2B
- U12 pad D22: /DSP/GD5_GPIO18_STATUS_2 -> /DSP/GD5_GPIO19_STATUS_1
- U12 pad D24: /DSP/GD_EPWM_6A -> /DSP/GD_EPWM_5A
- U12 pad D26: /DSP/GD3_EPWM_8B -> /DSP/GD3_EPWM_7B
- U12 pad D28: /DSP/GD2_EPWM_9A -> /DSP/GD2_GPIO44_STATUS_2
- U12 pad D30: /DSP/GD1_EPWM_11B -> /DSP/GD2_EPWM_10A
- U12 pad D32: /DSP/GD1_GPIO52_STATUS_2 -> /DSP/GD1_GPIO53_STATUS_1
- U12 pad D4: /Analog2/ADC_3 -> /DSP/ADC3_A3
- U12 pad D6: /Analog3/ADC_4 -> /DSP/ADC2_C4
- U12 pad D8: /GND -> /DSP/ADC1_B5
- U12 pad E1: /Analog1/ADC_4 -> /GND
- U12 pad E19: /DSP/GD6_EPWM_2A -> /DSP/GD6_EPWM_1B
- U12 pad E21: /DSP/GD5_EPWM_4B -> /DSP/GD5_GPIO18_STATUS_2
- U12 pad E23: /DSP/GD_EPWM_5A -> /DSP/GD5_EPWM_4A
- U12 pad E25: /DSP/GD3_EPWM_7B -> /DSP/GD_EPWM_6B
- U12 pad E29: /DSP/GD2_GPIO44_STATUS_2 -> /DSP/GD2_EPWM_9A
- U12 pad E3: /Analog2/ADC_5 -> /DSP/ADC3_B3
- U12 pad E31: /DSP/GD1_EPWM_12A -> /DSP/GD1_EPWM_11B
- U12 pad E5: /Analog3/ADC_6 -> /DSP/ADC2_D0
- U12 pad E7: /Analog3/ADC_1 -> /DSP/ADC1_D3
- U12 pad E9: /GND -> /DSP/ADC1_14
- U13 pad A1: /24V -> /GND
- U13 pad A11: /GD_GPIO14_RESET -> /DSP/GD2_GPIO44_STATUS_2
- U13 pad A13: /GPIO12_EMITTER_ENABLE -> /DSP/GD2_EPWM_9A
- U13 pad A15: /~SAFE_STATE_FLAG~ -> /DSP/GD2_EPWM_10B
- U13 pad A2: /24V -> /GND
- U13 pad A5: /GND -> /~SAFE_STATE_FLAG~
- U13 pad A7: /GND -> /GPIO12_EMITTER_ENABLE
- U13 pad A9: /GND -> /GD_GPIO14_RESET
- U13 pad B10: Net-(U13-PadB10) -> /GND
- U13 pad B11: Net-(U13-PadB10) -> /GND
- U13 pad B12: Net-(U13-PadB10) -> /GND
- U13 pad B13: Net-(U13-PadB10) -> /GND
- U13 pad B14: Net-(U13-PadB10) -> /GND
- U13 pad B15: Net-(U13-PadB10) -> /GND
- U13 pad B16: Net-(U13-PadB10) -> /GND
- U13 pad C1: Net-(U13-PadB10) -> /24V
- U13 pad C10: /DSP/GD2_EPWM_9B -> /GND
- U13 pad C11: Net-(U13-PadB10) -> /DSP/GD2_EPWM_9B
- U13 pad C12: /DSP/GD2_GPIO44_STATUS_2 -> /GND
- U13 pad C13: Net-(U13-PadB10) -> /DSP/GD2_GPIO45_STATUS_1
- U13 pad C14: Net-(U13-PadB10) -> /GND
- U13 pad C15: Net-(U13-PadB10) -> /DSP/GD2_EPWM_10A
- U13 pad C16: Net-(U13-PadB10) -> /GND
- U13 pad C2: /DSP/GD2_EPWM_10A -> /24V
- U13 pad C3: Net-(U13-PadB10) -> /GND
- U13 pad C4: /DSP/GD2_EPWM_10B -> /GND
- U13 pad C5: Net-(U13-PadB10) -> /GND
- U13 pad C6: /DSP/GD2_GPIO45_STATUS_1 -> /GND
- U13 pad C7: Net-(U13-PadB10) -> /GND
- U13 pad C8: /DSP/GD2_EPWM_9A -> /GND
- U13 pad C9: Net-(U13-PadB10) -> /GND
- U14 pad A1: /24V -> /GND
- U14 pad A11: /GD_GPIO14_RESET -> /DSP/GD3_GPIO24_STATUS_2
- U14 pad A13: /GPIO12_EMITTER_ENABLE -> /DSP/GD3_EPWM_7A
- U14 pad A15: /~SAFE_STATE_FLAG~ -> /DSP/GD3_EPWM_8B
- U14 pad A2: /24V -> /GND
- U14 pad A5: /GND -> /~SAFE_STATE_FLAG~
- U14 pad A7: /GND -> /GPIO12_EMITTER_ENABLE
- U14 pad A9: /GND -> /GD_GPIO14_RESET
- U14 pad B10: Net-(U14-PadB10) -> /GND
- U14 pad B11: Net-(U14-PadB10) -> /GND
- U14 pad B12: Net-(U14-PadB10) -> /GND
- U14 pad B13: Net-(U14-PadB10) -> /GND
- U14 pad B14: Net-(U14-PadB10) -> /GND
- U14 pad B15: Net-(U14-PadB10) -> /GND
- U14 pad B16: Net-(U14-PadB10) -> /GND
- U14 pad C1: Net-(U14-PadB10) -> /24V
- U14 pad C10: /DSP/GD3_EPWM_7B -> /GND
- U14 pad C11: Net-(U14-PadB10) -> /DSP/GD3_EPWM_7B
- U14 pad C12: /DSP/GD3_GPIO24_STATUS_2 -> /GND
- U14 pad C13: Net-(U14-PadB10) -> /DSP/GD3_GPIO25_STATUS_1
- U14 pad C14: Net-(U14-PadB10) -> /GND
- U14 pad C15: Net-(U14-PadB10) -> /DSP/GD3_EPWM_8A
- U14 pad C16: Net-(U14-PadB10) -> /GND
- U14 pad C2: /DSP/GD3_EPWM_8A -> /24V
- U14 pad C3: Net-(U14-PadB10) -> /GND
- U14 pad C4: /DSP/GD3_EPWM_8B -> /GND
- U14 pad C5: Net-(U14-PadB10) -> /GND
- U14 pad C6: /DSP/GD3_GPIO25_STATUS_1 -> /GND
- U14 pad C7: Net-(U14-PadB10) -> /GND
- U14 pad C8: /DSP/GD3_EPWM_7A -> /GND
- U14 pad C9: Net-(U14-PadB10) -> /GND
- U3 pad A1: /GND -> /24V
- U3 pad A16: /~SAFE_STATE_FLAG~ -> /GND
- U3 pad C12: /GND -> /~SAFE_STATE_FLAG~
- U3 pad C2: /24V -> /GND
- U4 pad A1: /GND -> /24V
- U4 pad A16: /~SAFE_STATE_FLAG~ -> /GND
- U4 pad C12: /GND -> /~SAFE_STATE_FLAG~
- U4 pad C2: /24V -> /GND
- U5 pad A10: /Analog2/ADC_2 -> /GND
- U5 pad A11: /GND -> /DSP/ADC2_C5
- U5 pad A12: /Analog2/ADC_3 -> /GND
- U5 pad A13: /GND -> /DSP/ADC2_A5
- U5 pad A2: /24V -> /GND
- U5 pad A8: /Analog2/ADC_1 -> /GND
- U5 pad A9: /GND -> /DSP/ADC2_D1
- U5 pad C1: /GND -> /24V
- U5 pad C11: /Analog2/ADC_4 -> /DSP/ADC2_C4
- U5 pad C13: /Analog2/ADC_5 -> /DSP/ADC2_A4
- U5 pad C15: /Analog2/ADC_6 -> /GND
- U5 pad C9: /GND -> /DSP/ADC2_D0
- U6 pad A1: /24V -> /GND
- U6 pad A11: /GD_GPIO14_RESET -> /DSP/GD1_GPIO52_STATUS_2
- U6 pad A13: /GPIO12_EMITTER_ENABLE -> /DSP/GD1_EPWM_11A
- U6 pad A15: /~SAFE_STATE_FLAG~ -> /DSP/GD1_EPWM_12B
- U6 pad A2: /24V -> /GND
- U6 pad A5: /GND -> /~SAFE_STATE_FLAG~
- U6 pad A7: /GND -> /GPIO12_EMITTER_ENABLE
- U6 pad A9: /GND -> /GD_GPIO14_RESET
- U6 pad B10: Net-(U6-PadB10) -> /GND
- U6 pad B11: Net-(U6-PadB10) -> /GND
- U6 pad B12: Net-(U6-PadB10) -> /GND
- U6 pad B13: Net-(U6-PadB10) -> /GND
- U6 pad B14: Net-(U6-PadB10) -> /GND
- U6 pad B15: Net-(U6-PadB10) -> /GND
- U6 pad B16: Net-(U6-PadB10) -> /GND
- U6 pad C1: Net-(U6-PadB10) -> /24V
- U6 pad C10: /DSP/GD1_EPWM_11B -> /GND
- U6 pad C11: Net-(U6-PadB10) -> /DSP/GD1_EPWM_11B
- U6 pad C12: /DSP/GD1_GPIO52_STATUS_2 -> /GND
- U6 pad C13: Net-(U6-PadB10) -> /DSP/GD1_GPIO53_STATUS_1
- U6 pad C14: Net-(U6-PadB10) -> /GND
- U6 pad C15: Net-(U6-PadB10) -> /DSP/GD1_EPWM_12A
- U6 pad C16: Net-(U6-PadB10) -> /GND
- U6 pad C2: /DSP/GD1_EPWM_12A -> /24V
- U6 pad C3: Net-(U6-PadB10) -> /GND
- U6 pad C4: /DSP/GD1_EPWM_12B -> /GND
- U6 pad C5: Net-(U6-PadB10) -> /GND
- U6 pad C6: /DSP/GD1_GPIO53_STATUS_1 -> /GND
- U6 pad C7: Net-(U6-PadB10) -> /GND
- U6 pad C8: /DSP/GD1_EPWM_11A -> /GND
- U6 pad C9: Net-(U6-PadB10) -> /GND
- U7 pad A1: /24V -> /GND
- U7 pad A11: /GD_GPIO14_RESET -> /DSP/GD4_GPIO22_STATUS_2
- U7 pad A13: /GPIO12_EMITTER_ENABLE -> /DSP/GD_EPWM_5A
- U7 pad A15: /~SAFE_STATE_FLAG~ -> /DSP/GD_EPWM_6B
- U7 pad A2: /24V -> /GND
- U7 pad A5: /GND -> /~SAFE_STATE_FLAG~
- U7 pad A7: /GND -> /GPIO12_EMITTER_ENABLE
- U7 pad A9: /GND -> /GD_GPIO14_RESET
- U7 pad B10: Net-(U7-PadB10) -> /GND
- U7 pad B11: Net-(U7-PadB10) -> /GND
- U7 pad B12: Net-(U7-PadB10) -> /GND
- U7 pad B13: Net-(U7-PadB10) -> /GND
- U7 pad B14: Net-(U7-PadB10) -> /GND
- U7 pad B15: Net-(U7-PadB10) -> /GND
- U7 pad B16: Net-(U7-PadB10) -> /GND
- U7 pad C1: Net-(U7-PadB10) -> /24V
- U7 pad C10: /DSP/GD_EPWM_5B -> /GND
- U7 pad C11: Net-(U7-PadB10) -> /DSP/GD_EPWM_5B
- U7 pad C12: /DSP/GD4_GPIO22_STATUS_2 -> /GND
- U7 pad C13: Net-(U7-PadB10) -> /DSP/GD4_GPIO23_STATUS_1
- U7 pad C14: Net-(U7-PadB10) -> /GND
- U7 pad C15: Net-(U7-PadB10) -> /DSP/GD_EPWM_6A
- U7 pad C16: Net-(U7-PadB10) -> /GND
- U7 pad C2: /DSP/GD_EPWM_6A -> /24V
- U7 pad C3: Net-(U7-PadB10) -> /GND
- U7 pad C4: /DSP/GD_EPWM_6B -> /GND
- U7 pad C5: Net-(U7-PadB10) -> /GND
- U7 pad C6: /DSP/GD4_GPIO23_STATUS_1 -> /GND
- U7 pad C7: Net-(U7-PadB10) -> /GND
- U7 pad C8: /DSP/GD_EPWM_5A -> /GND
- U7 pad C9: Net-(U7-PadB10) -> /GND
- U8 pad A1: /24V -> /GND
- U8 pad A11: /GD_GPIO14_RESET -> /DSP/GD6_GPIO15_STATUS_2
- U8 pad A13: /GPIO12_EMITTER_ENABLE -> /DSP/GD6_EPWM_1A
- U8 pad A15: /~SAFE_STATE_FLAG~ -> /DSP/GD6_EPWM_2B
- U8 pad A2: /24V -> /GND
- U8 pad A5: /GND -> /~SAFE_STATE_FLAG~
- U8 pad A7: /GND -> /GPIO12_EMITTER_ENABLE
- U8 pad A9: /GND -> /GD_GPIO14_RESET
- U8 pad B10: Net-(U8-PadB10) -> /GND
- U8 pad B11: Net-(U8-PadB10) -> /GND
- U8 pad B12: Net-(U8-PadB10) -> /GND
- U8 pad B13: Net-(U8-PadB10) -> /GND
- U8 pad B14: Net-(U8-PadB10) -> /GND
- U8 pad B15: Net-(U8-PadB10) -> /GND
- U8 pad B16: Net-(U8-PadB10) -> /GND
- U8 pad C1: Net-(U8-PadB10) -> /24V
- U8 pad C10: /DSP/GD6_EPWM_1B -> /GND
- U8 pad C11: Net-(U8-PadB10) -> /DSP/GD6_EPWM_1B
- U8 pad C12: /DSP/GD6_GPIO15_STATUS_2 -> /GND
- U8 pad C13: Net-(U8-PadB10) -> /DSP/GD6_GPIO16_STATUS_1
- U8 pad C14: Net-(U8-PadB10) -> /GND
- U8 pad C15: Net-(U8-PadB10) -> /DSP/GD6_EPWM_2A
- U8 pad C16: Net-(U8-PadB10) -> /GND
- U8 pad C2: /DSP/GD6_EPWM_2A -> /24V
- U8 pad C3: Net-(U8-PadB10) -> /GND
- U8 pad C4: /DSP/GD6_EPWM_2B -> /GND
- U8 pad C5: Net-(U8-PadB10) -> /GND
- U8 pad C6: /DSP/GD6_GPIO16_STATUS_1 -> /GND
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Routing:
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- added copper zone on B.Cu, net /24V
