File: MC-Backplane/Backplane.kicad_pcb (KiCad board)
At the start: 4 copper layers, 294.6 x 132.6 mm, 133 parts, among them J1 1730010, U1 64600001223, U10 86094328314755V1LF, U11 86094328314755V1LF, U12 374472, U13 86094328314755V1LF, U14 86094328314755V1LF, U2 SISS05DN-T1-GE3, U3 86094328314755V1LF, U4 86094328314755V1LF, U5 86094328314755V1LF, U6 86094328314755V1LF, U7 86094328314755V1LF, U8 86094328314755V1LF, U9 86094328314755V1LF

Commit message: Layout done: ready for revisions
- double check measurements and connector placement
-passes DRC schematic and layout
Parts:
- removed the REF** at (296.8, 34.4)
- removed the REF** at (261.3, 34.4)
- removed the REF** at (93.7, 157.0)
- removed the REF** at (78.4, 157.0)
- removed the REF** at (83.5, 157.0)
- removed the REF** at (88.6, 157.0)
- removed the REF** at (129.2, 157.0)
- removed the REF** at (124.2, 157.0)
- removed the REF** at (73.4, 157.0)
- removed the REF** at (68.3, 157.0)
- removed the REF** at (63.2, 157.0)
- removed the REF** at (58.1, 157.0)
- removed the REF** at (215.6, 34.4)
- removed the REF** at (48.0, 157.0)
- removed the REF** at (53.0, 157.0)
- removed the REF** at (42.9, 157.0)
- removed the REF** at (37.8, 157.0)
- removed the REF** at (27.6, 156.9)
- removed the REF** at (22.6, 156.9)
- removed the REF** at (32.7, 157.0)
- removed the REF** at (307.0, 34.4)
- removed the REF** at (195.2, 34.4)
- removed the REF** at (230.8, 34.4)
- removed the REF** at (169.8, 34.4)
- removed the REF** at (241.0, 34.4)
- removed the REF** at (164.8, 34.4)
- removed the REF** at (210.5, 34.4)
- removed the REF** at (205.4, 34.4)
- removed the REF** at (271.4, 34.4)
- removed the REF** at (174.9, 34.4)
- removed the REF** at (312.1, 34.5)
- removed the REF** at (235.9, 34.4)
- removed the REF** at (200.3, 34.4)
- removed the REF** at (190.2, 34.4)
- removed the REF** at (225.7, 34.4)
- removed the REF** at (266.4, 34.4)
- removed the REF** at (220.6, 34.4)
- removed the REF** at (301.9, 34.4)
- removed the REF** at (32.7, 34.3)
- removed the REF** at (281.6, 34.4)
- removed the REF** at (22.5, 34.3)
- removed the REF** at (27.6, 34.3)
- removed the REF** at (42.8, 34.3)
- removed the REF** at (53.0, 34.3)
- removed the REF** at (47.9, 34.3)
- removed the REF** at (68.2, 34.3)
- removed the REF** at (58.1, 34.3)
- removed the REF** at (124.1, 34.4)
- removed the REF** at (73.3, 34.3)
- removed the REF** at (63.2, 34.3)
- removed the REF** at (246.0, 34.4)
- removed the REF** at (37.8, 34.3)
- removed the REF** at (108.9, 34.4)
- removed the REF** at (78.4, 34.3)
- removed the REF** at (93.6, 34.4)
- removed the REF** at (103.8, 34.4)
- removed the REF** at (119.0, 34.4)
- removed the REF** at (98.7, 34.4)
- removed the REF** at (185.1, 34.4)
- removed the REF** at (139.4, 34.4)
- removed the REF** at (149.5, 34.4)
- removed the REF** at (291.8, 34.4)
- removed the REF** at (159.7, 34.4)
- removed the REF** at (154.6, 34.4)
- removed the REF** at (134.3, 34.4)
- removed the REF** at (144.4, 34.4)
- removed the REF** at (129.2, 34.4)
- removed the REF** at (88.6, 34.4)
- removed the REF** at (114.0, 34.4)
- removed the REF** at (180.0, 34.4)
- removed the REF** at (83.5, 34.3)
- removed the REF** at (286.7, 157.1)
- removed the REF** at (286.7, 34.4)
- removed the REF** at (291.8, 157.1)
- removed the REF** at (261.3, 157.1)
- removed the REF** at (296.9, 157.1)
- removed the REF** at (246.1, 157.0)
- removed the REF** at (251.2, 157.0)
- removed the REF** at (281.6, 157.1)
- removed the REF** at (256.2, 157.1)
- removed the REF** at (276.6, 157.1)
- removed the REF** at (271.5, 157.1)
- removed the REF** at (266.4, 157.1)
- removed the REF** at (276.5, 34.4)
- removed the REF** at (230.8, 157.0)
- removed the REF** at (220.7, 157.0)
- removed the REF** at (225.8, 157.0)
- removed the REF** at (215.6, 157.0)
- removed the REF** at (210.5, 157.0)
- removed the REF** at (205.4, 157.0)
- removed the REF** at (190.2, 157.0)
- removed the REF** at (195.3, 157.0)
- removed the REF** at (200.4, 157.0)
- removed the REF** at (302.0, 157.1)
- removed the REF** at (256.2, 34.4)
- removed the REF** at (241.0, 157.0)
- removed the REF** at (235.9, 157.0)
- removed the REF** at (307.0, 157.1)
- removed the REF** at (312.1, 157.1)
- removed the REF** at (175.0, 157.0)
- removed the REF** at (164.8, 157.0)
- removed the REF** at (169.9, 157.0)
- removed the REF** at (159.7, 157.0)
- removed the REF** at (154.6, 157.0)
- removed the REF** at (149.6, 157.0)
- removed the REF** at (251.1, 34.4)
- removed the REF** at (134.3, 157.0)
- removed the REF** at (139.4, 157.0)
- removed the REF** at (144.5, 157.0)
- removed the REF** at (185.1, 157.0)
- removed the REF** at (180.0, 157.0)
- removed the REF** at (119.1, 157.0)
- removed the REF** at (108.9, 157.0)
- removed the REF** at (114.0, 157.0)
- removed the REF** at (103.8, 157.0)
- removed the REF** at (98.8, 157.0)
- added REF**: MountingHole_3.2mm_M3, MountingHole:MountingHole_3.2mm_M3, F.Cu at (159.7, 157.0)
- added REF**: MountingHole_3.2mm_M3, MountingHole:MountingHole_3.2mm_M3, F.Cu at (180.0, 157.0)
- added REF**: MountingHole_3.2mm_M3, MountingHole:MountingHole_3.2mm_M3, F.Cu at (88.6, 34.5)
- added REF**: MountingHole_3.2mm_M3, MountingHole:MountingHole_3.2mm_M3, F.Cu at (296.9, 34.6)
- added REF**: MountingHole_3.2mm_M3, MountingHole:MountingHole_3.2mm_M3, F.Cu at (119.1, 34.5)
- added REF**: MountingHole_3.2mm_M3, MountingHole:MountingHole_3.2mm_M3, F.Cu at (73.3, 34.5)
- added REF**: MountingHole_3.2mm_M3, MountingHole:MountingHole_3.2mm_M3, F.Cu at (169.9, 34.5)
- added REF**: MountingHole_3.2mm_M3, MountingHole:MountingHole_3.2mm_M3, F.Cu at (266.4, 34.6)
- added REF**: MountingHole_3.2mm_M3, MountingHole:MountingHole_3.2mm_M3, F.Cu at (301.9, 34.6)
- added REF**: MountingHole_3.2mm_M3, MountingHole:MountingHole_3.2mm_M3, F.Cu at (312.1, 34.6)
- added REF**: MountingHole_3.2mm_M3, MountingHole:MountingHole_3.2mm_M3, F.Cu at (205.4, 34.6)
- added REF**: MountingHole_3.2mm_M3, MountingHole:MountingHole_3.2mm_M3, F.Cu at (164.8, 34.5)
- added REF**: MountingHole_3.2mm_M3, MountingHole:MountingHole_3.2mm_M3, F.Cu at (93.7, 157.0)
- added REF**: MountingHole_3.2mm_M3, MountingHole:MountingHole_3.2mm_M3, F.Cu at (190.2, 34.5)
- added REF**: MountingHole_3.2mm_M3, MountingHole:MountingHole_3.2mm_M3, F.Cu at (210.5, 34.6)
- added REF**: MountingHole_3.2mm_M3, MountingHole:MountingHole_3.2mm_M3, F.Cu at (22.5, 34.5)
- added REF**: MountingHole_3.2mm_M3, MountingHole:MountingHole_3.2mm_M3, F.Cu at (27.6, 34.5)
- added REF**: MountingHole_3.2mm_M3, MountingHole:MountingHole_3.2mm_M3, F.Cu at (32.7, 34.5)
- added REF**: MountingHole_3.2mm_M3, MountingHole:MountingHole_3.2mm_M3, F.Cu at (220.7, 34.6)
- added REF**: MountingHole_3.2mm_M3, MountingHole:MountingHole_3.2mm_M3, F.Cu at (235.9, 34.6)
- added REF**: MountingHole_3.2mm_M3, MountingHole:MountingHole_3.2mm_M3, F.Cu at (88.6, 157.0)
- added REF**: MountingHole_3.2mm_M3, MountingHole:MountingHole_3.2mm_M3, F.Cu at (98.7, 157.0)
- added REF**: MountingHole_3.2mm_M3, MountingHole:MountingHole_3.2mm_M3, F.Cu at (114.0, 157.0)
- added REF**: MountingHole_3.2mm_M3, MountingHole:MountingHole_3.2mm_M3, F.Cu at (119.1, 157.0)
- added REF**: MountingHole_3.2mm_M3, MountingHole:MountingHole_3.2mm_M3, F.Cu at (144.5, 157.0)
- added REF**: MountingHole_3.2mm_M3, MountingHole:MountingHole_3.2mm_M3, F.Cu at (154.6, 157.0)
- added REF**: MountingHole_3.2mm_M3, MountingHole:MountingHole_3.2mm_M3, F.Cu at (169.9, 157.0)
- added REF**: MountingHole_3.2mm_M3, MountingHole:MountingHole_3.2mm_M3, F.Cu at (301.9, 157.1)
- added REF**: MountingHole_3.2mm_M3, MountingHole:MountingHole_3.2mm_M3, F.Cu at (134.3, 157.0)
- added REF**: MountingHole_3.2mm_M3, MountingHole:MountingHole_3.2mm_M3, F.Cu at (266.4, 157.1)
- added REF**: MountingHole_3.2mm_M3, MountingHole:MountingHole_3.2mm_M3, F.Cu at (241.0, 157.1)
- added REF**: MountingHole_3.2mm_M3, MountingHole:MountingHole_3.2mm_M3, F.Cu at (190.2, 157.0)
- added REF**: MountingHole_3.2mm_M3, MountingHole:MountingHole_3.2mm_M3, F.Cu at (271.5, 157.1)
- added REF**: MountingHole_3.2mm_M3, MountingHole:MountingHole_3.2mm_M3, F.Cu at (220.7, 157.1)
- added REF**: MountingHole_3.2mm_M3, MountingHole:MountingHole_3.2mm_M3, F.Cu at (230.8, 157.1)
- added REF**: MountingHole_3.2mm_M3, MountingHole:MountingHole_3.2mm_M3, F.Cu at (210.5, 157.1)
- added REF**: MountingHole_3.2mm_M3, MountingHole:MountingHole_3.2mm_M3, F.Cu at (215.6, 157.1)
- added REF**: MountingHole_3.2mm_M3, MountingHole:MountingHole_3.2mm_M3, F.Cu at (200.3, 157.1)
- added REF**: MountingHole_3.2mm_M3, MountingHole:MountingHole_3.2mm_M3, F.Cu at (225.7, 157.1)
- added REF**: MountingHole_3.2mm_M3, MountingHole:MountingHole_3.2mm_M3, F.Cu at (149.5, 157.0)
- added REF**: MountingHole_3.2mm_M3, MountingHole:MountingHole_3.2mm_M3, F.Cu at (205.4, 157.1)
- added REF**: MountingHole_3.2mm_M3, MountingHole:MountingHole_3.2mm_M3, F.Cu at (164.8, 157.0)
- added REF**: MountingHole_3.2mm_M3, MountingHole:MountingHole_3.2mm_M3, F.Cu at (174.9, 157.0)
- added REF**: MountingHole_3.2mm_M3, MountingHole:MountingHole_3.2mm_M3, F.Cu at (312.1, 157.1)
- added REF**: MountingHole_3.2mm_M3, MountingHole:MountingHole_3.2mm_M3, F.Cu at (195.3, 157.0)
- added REF**: MountingHole_3.2mm_M3, MountingHole:MountingHole_3.2mm_M3, F.Cu at (307.0, 157.1)
- added REF**: MountingHole_3.2mm_M3, MountingHole:MountingHole_3.2mm_M3, F.Cu at (235.9, 157.1)
- added REF**: MountingHole_3.2mm_M3, MountingHole:MountingHole_3.2mm_M3, F.Cu at (37.8, 157.0)
- added REF**: MountingHole_3.2mm_M3, MountingHole:MountingHole_3.2mm_M3, F.Cu at (22.5, 157.0)
- added REF**: MountingHole_3.2mm_M3, MountingHole:MountingHole_3.2mm_M3, F.Cu at (53.0, 157.0)
- added REF**: MountingHole_3.2mm_M3, MountingHole:MountingHole_3.2mm_M3, F.Cu at (83.5, 157.0)
- added REF**: MountingHole_3.2mm_M3, MountingHole:MountingHole_3.2mm_M3, F.Cu at (73.3, 157.0)
- added REF**: MountingHole_3.2mm_M3, MountingHole:MountingHole_3.2mm_M3, F.Cu at (129.2, 157.0)
- added REF**: MountingHole_3.2mm_M3, MountingHole:MountingHole_3.2mm_M3, F.Cu at (58.1, 157.0)
- added REF**: MountingHole_3.2mm_M3, MountingHole:MountingHole_3.2mm_M3, F.Cu at (32.7, 157.0)
- added REF**: MountingHole_3.2mm_M3, MountingHole:MountingHole_3.2mm_M3, F.Cu at (68.3, 157.0)
- added REF**: MountingHole_3.2mm_M3, MountingHole:MountingHole_3.2mm_M3, F.Cu at (63.2, 157.0)
- added REF**: MountingHole_3.2mm_M3, MountingHole:MountingHole_3.2mm_M3, F.Cu at (27.6, 157.0)
- added REF**: MountingHole_3.2mm_M3, MountingHole:MountingHole_3.2mm_M3, F.Cu at (124.1, 157.0)
- added REF**: MountingHole_3.2mm_M3, MountingHole:MountingHole_3.2mm_M3, F.Cu at (47.9, 157.0)
- added REF**: MountingHole_3.2mm_M3, MountingHole:MountingHole_3.2mm_M3, F.Cu at (42.9, 157.0)
- added REF**: MountingHole_3.2mm_M3, MountingHole:MountingHole_3.2mm_M3, F.Cu at (78.4, 157.0)
- added REF**: MountingHole_3.2mm_M3, MountingHole:MountingHole_3.2mm_M3, F.Cu at (261.3, 157.1)
- added REF**: MountingHole_3.2mm_M3, MountingHole:MountingHole_3.2mm_M3, F.Cu at (291.8, 157.1)
- added REF**: MountingHole_3.2mm_M3, MountingHole:MountingHole_3.2mm_M3, F.Cu at (246.1, 157.1)
- added REF**: MountingHole_3.2mm_M3, MountingHole:MountingHole_3.2mm_M3, F.Cu at (276.5, 157.1)
- added REF**: MountingHole_3.2mm_M3, MountingHole:MountingHole_3.2mm_M3, F.Cu at (256.2, 157.1)
- added REF**: MountingHole_3.2mm_M3, MountingHole:MountingHole_3.2mm_M3, F.Cu at (281.6, 157.1)
- added REF**: MountingHole_3.2mm_M3, MountingHole:MountingHole_3.2mm_M3, F.Cu at (286.7, 157.1)
- added REF**: MountingHole_3.2mm_M3, MountingHole:MountingHole_3.2mm_M3, F.Cu at (296.9, 157.1)
- added REF**: MountingHole_3.2mm_M3, MountingHole:MountingHole_3.2mm_M3, F.Cu at (251.1, 157.1)
- added REF**: MountingHole_3.2mm_M3, MountingHole:MountingHole_3.2mm_M3, F.Cu at (37.8, 34.5)
- added REF**: MountingHole_3.2mm_M3, MountingHole:MountingHole_3.2mm_M3, F.Cu at (139.4, 157.0)
- added REF**: MountingHole_3.2mm_M3, MountingHole:MountingHole_3.2mm_M3, F.Cu at (68.3, 34.5)
- added REF**: MountingHole_3.2mm_M3, MountingHole:MountingHole_3.2mm_M3, F.Cu at (63.2, 34.5)
- added REF**: MountingHole_3.2mm_M3, MountingHole:MountingHole_3.2mm_M3, F.Cu at (225.7, 34.6)
- added REF**: MountingHole_3.2mm_M3, MountingHole:MountingHole_3.2mm_M3, F.Cu at (58.1, 34.5)
- added REF**: MountingHole_3.2mm_M3, MountingHole:MountingHole_3.2mm_M3, F.Cu at (139.4, 34.5)
- added REF**: MountingHole_3.2mm_M3, MountingHole:MountingHole_3.2mm_M3, F.Cu at (42.9, 34.5)
- added REF**: MountingHole_3.2mm_M3, MountingHole:MountingHole_3.2mm_M3, F.Cu at (108.9, 34.5)
- added REF**: MountingHole_3.2mm_M3, MountingHole:MountingHole_3.2mm_M3, F.Cu at (93.7, 34.5)
- added REF**: MountingHole_3.2mm_M3, MountingHole:MountingHole_3.2mm_M3, F.Cu at (241.0, 34.6)
- added REF**: MountingHole_3.2mm_M3, MountingHole:MountingHole_3.2mm_M3, F.Cu at (78.4, 34.5)
- added REF**: MountingHole_3.2mm_M3, MountingHole:MountingHole_3.2mm_M3, F.Cu at (108.9, 157.0)
- added REF**: MountingHole_3.2mm_M3, MountingHole:MountingHole_3.2mm_M3, F.Cu at (98.7, 34.5)
- added REF**: MountingHole_3.2mm_M3, MountingHole:MountingHole_3.2mm_M3, F.Cu at (149.5, 34.5)
- added REF**: MountingHole_3.2mm_M3, MountingHole:MountingHole_3.2mm_M3, F.Cu at (47.9, 34.5)
- added REF**: MountingHole_3.2mm_M3, MountingHole:MountingHole_3.2mm_M3, F.Cu at (230.8, 34.6)
- added REF**: MountingHole_3.2mm_M3, MountingHole:MountingHole_3.2mm_M3, F.Cu at (200.3, 34.6)
- added REF**: MountingHole_3.2mm_M3, MountingHole:MountingHole_3.2mm_M3, F.Cu at (103.8, 34.5)
- added REF**: MountingHole_3.2mm_M3, MountingHole:MountingHole_3.2mm_M3, F.Cu at (174.9, 34.5)
- added REF**: MountingHole_3.2mm_M3, MountingHole:MountingHole_3.2mm_M3, F.Cu at (307.0, 34.6)
- added REF**: MountingHole_3.2mm_M3, MountingHole:MountingHole_3.2mm_M3, F.Cu at (281.6, 34.6)
- added REF**: MountingHole_3.2mm_M3, MountingHole:MountingHole_3.2mm_M3, F.Cu at (286.7, 34.6)
- added REF**: MountingHole_3.2mm_M3, MountingHole:MountingHole_3.2mm_M3, F.Cu at (185.1, 157.0)
- added REF**: MountingHole_3.2mm_M3, MountingHole:MountingHole_3.2mm_M3, F.Cu at (261.3, 34.6)
- added REF**: MountingHole_3.2mm_M3, MountingHole:MountingHole_3.2mm_M3, F.Cu at (246.1, 34.6)
- added REF**: MountingHole_3.2mm_M3, MountingHole:MountingHole_3.2mm_M3, F.Cu at (256.2, 34.6)
- added REF**: MountingHole_3.2mm_M3, MountingHole:MountingHole_3.2mm_M3, F.Cu at (195.3, 34.5)
- added REF**: MountingHole_3.2mm_M3, MountingHole:MountingHole_3.2mm_M3, F.Cu at (251.1, 34.6)
- added REF**: MountingHole_3.2mm_M3, MountingHole:MountingHole_3.2mm_M3, F.Cu at (271.5, 34.6)
- added REF**: MountingHole_3.2mm_M3, MountingHole:MountingHole_3.2mm_M3, F.Cu at (276.5, 34.6)
- added REF**: MountingHole_3.2mm_M3, MountingHole:MountingHole_3.2mm_M3, F.Cu at (291.8, 34.6)
- added REF**: MountingHole_3.2mm_M3, MountingHole:MountingHole_3.2mm_M3, F.Cu at (144.5, 34.5)
- added REF**: MountingHole_3.2mm_M3, MountingHole:MountingHole_3.2mm_M3, F.Cu at (129.2, 34.5)
- added REF**: MountingHole_3.2mm_M3, MountingHole:MountingHole_3.2mm_M3, F.Cu at (103.8, 157.0)
- added REF**: MountingHole_3.2mm_M3, MountingHole:MountingHole_3.2mm_M3, F.Cu at (159.7, 34.5)
- added REF**: MountingHole_3.2mm_M3, MountingHole:MountingHole_3.2mm_M3, F.Cu at (185.1, 34.5)
- added REF**: MountingHole_3.2mm_M3, MountingHole:MountingHole_3.2mm_M3, F.Cu at (154.6, 34.5)
- added REF**: MountingHole_3.2mm_M3, MountingHole:MountingHole_3.2mm_M3, F.Cu at (180.0, 34.5)
- added REF**: MountingHole_3.2mm_M3, MountingHole:MountingHole_3.2mm_M3, F.Cu at (134.3, 34.5)
- added REF**: MountingHole_3.2mm_M3, MountingHole:MountingHole_3.2mm_M3, F.Cu at (114.0, 34.5)
- added REF**: MountingHole_3.2mm_M3, MountingHole:MountingHole_3.2mm_M3, F.Cu at (83.5, 34.5)
- added REF**: MountingHole_3.2mm_M3, MountingHole:MountingHole_3.2mm_M3, F.Cu at (53.0, 34.5)
- added REF**: MountingHole_3.2mm_M3, MountingHole:MountingHole_3.2mm_M3, F.Cu at (124.1, 34.5)
- added REF**: MountingHole_3.2mm_M3, MountingHole:MountingHole_3.2mm_M3, F.Cu at (215.6, 34.6)
Routing:
- net Net-(U1-Pad2): track 14.5 -> 9.89 mm
- net /DSP/GD5_GPIO18_STATUS_2: track 106.0 -> 103.7 mm
- net /DSP/GD5_EPWM_3B: track 116.3 -> 114.3 mm
- net /DSP/GD5_GPIO19_STATUS_1: track 109.7 -> 108.0 mm
- net /DSP/GD5_EPWM_3A: track 112.7 -> 111.0 mm
- net /DSP/GD2_GPIO44_STATUS_2: track 173.4 -> 171.7 mm
- net /DSP/GD2_EPWM_10B: track 171.6 -> 170.2 mm
- net /DSP/GD5_EPWM_4B: track 105.7 -> 104.6 mm
- net /DSP/GD5_EPWM_4A: track 102.8 -> 101.7 mm
- net /DSP/GD1_GPIO52_STATUS_2: track 199.3 -> 198.5 mm
- net /DSP/GD2_EPWM_10A: track 169.2 -> 168.4 mm
- net /DSP/GD2_GPIO45_STATUS_1: track 178.3 -> 179.0 mm
Other:
- board text added: "Top/bottom of card distance to edge of backplane (Sh-Hg)/2 = 16.1925mm"
- board text added: "center of mounting hole distance from top/bottom of board (Sh-Nc)/2 = 5.0419mm"

Commit message: Layout ready for review
- double check measurements and connector placement
Routing:
- net /DSP/GD2_EPWM_10A: track 168.4 -> 167.4 mm
Other:
- board text added: "pin 1 of the FO card"
- board text added: "where pcb meets card guide CG3-160e"

Commit message: spread tracks across available space
could still add some test points
Parts:
- removed the REF** at (22.5, 34.5)
- removed the REF** at (27.6, 34.5)
- removed the REF** at (32.7, 34.5)
- removed the REF** at (37.8, 157.0)
- removed the REF** at (22.5, 157.0)
- removed the REF** at (32.7, 157.0)
- removed the REF** at (27.6, 157.0)
- removed the REF** at (37.8, 34.5)
- U1: moved to B.Cu
- moved U1 120.5 mm to (113.4, 137.2), turned to 180 degrees
- moved J1 119.5 mm to (126.1, 137.2)
- moved D1 79.3 mm to (85.4, 136.3), turned to 0 degrees
- moved R1 76.2 mm to (80.2, 138.7), turned to 180 degrees
- moved U2 71.7 mm to (80.3, 135.8), turned to 180 degrees
Connections:
- U12 pad D16: /SD2/PWMB_CLK_OUT -> /GND
- U12 pad E13: /SD1/PWMB_CLK_OUT -> /GND
- U3 pad C10: /SD1/PWMB_CLK_OUT -> /GND
- U4 pad C10: /SD2/PWMB_CLK_OUT -> /GND
Routing:
- net /GND: track 3.86 -> 80.2 mm, vias 2 -> 1
- net /SD1/PWMB_CLK_OUT: track 46.4 -> 0.00 mm
- net /SD2/PWMB_CLK_OUT: track 31.7 -> 0.00 mm
- net /DSP/GD4_GPIO22_STATUS_2: track 137.5 -> 116.0 mm
- net /DSP/GD_EPWM_5A: track 130.1 -> 114.2 mm
- net /DSP/GD_EPWM_5B: track 147.0 -> 131.3 mm
- net /DSP/GD5_EPWM_3B: track 114.3 -> 98.7 mm
- net /DSP/GD5_GPIO18_STATUS_2: track 103.7 -> 88.4 mm
- net /DSP/GD3_EPWM_7B: track 158.2 -> 143.9 mm
- net /DSP/GD3_GPIO24_STATUS_2: track 163.4 -> 149.3 mm
- net /DSP/GD6_EPWM_1B: track 80.7 -> 66.9 mm
- net /DSP/GD6_GPIO15_STATUS_2: track 83.2 -> 69.4 mm
- net /DSP/GD4_GPIO23_STATUS_1: track 139.8 -> 127.1 mm
- net /DSP/GD5_GPIO19_STATUS_1: track 108.0 -> 95.4 mm
- net /DSP/GD5_EPWM_3A: track 111.0 -> 98.5 mm
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Other:
- board size 294.6 x 132.6 mm -> 274.3 x 132.6 mm

Commit message: added testpoints
Parts:
- added TP1: TestPoint, TestPoint:TestPoint_Plated_Hole_D2.0mm, F.Cu at (102.2, 125.8)
- added TP2: TestPoint, TestPoint:TestPoint_Plated_Hole_D2.0mm, F.Cu at (122.3, 93.2)
- added TP3: TestPoint, TestPoint:TestPoint_Plated_Hole_D2.0mm, F.Cu at (62.3, 130.6)
- added TP4: TestPoint, TestPoint:TestPoint_Plated_Hole_D2.0mm, F.Cu at (81.4, 89.2)
- added TP5: TestPoint, TestPoint:TestPoint_Plated_Hole_D2.0mm, F.Cu at (117.9, 137.1)
- added TP6: TestPoint, TestPoint:TestPoint_Plated_Hole_D2.0mm, F.Cu at (239.3, 138.1)
- added TP7: TestPoint, TestPoint:TestPoint_Plated_Hole_D2.0mm, F.Cu at (161.9, 104.6)
- added TP8: TestPoint, TestPoint:TestPoint_Plated_Hole_D2.0mm, F.Cu at (142.0, 100.6)
- added TP9: TestPoint, TestPoint:TestPoint_Plated_Hole_D2.0mm, F.Cu at (243.8, 122.9)
- moved J1 1.97 mm to (128.1, 137.1)
Connections:
- net /GD_GPIO14_RESET renamed /GD_GPIO14_OUTPUT_RESET
Routing:
- net /ReversePolarityPrrotection/24V_unprotected: track 7.71 -> 18.2 mm
Other:
- board text added: "24V"
- board text added: "24V unprotected"
- board text added: "ADC1"
- board text added: "ADC2"
- board text added: "ADC3"
- board text added: "Backplane Senior Design Project 20: Modular Computer Julia Germano, Jacob Williams, Zach Murray 2021-2022"
- board text added: "EMITTER_ENABLE"
- board text added: "GD1"
- board text added: "GD2"
- board text added: "GD3"
- board text added: "GD4"
- board text added: "GD5"
- board text added: "GD6"
- board text added: "GD_OUTPUT_RESET"
- board text added: "GND"
- board text added: "SAFE_STATE_FLAG"
- board text added: "SD1"
- board text added: "SD2"

Commit message: removed some MHs and attempted to fix library
Parts:
- removed the REF** at (159.7, 157.0)
- removed the REF** at (180.0, 157.0)
- removed the REF** at (266.4, 34.6)
- removed the REF** at (301.9, 34.6)
- removed the REF** at (205.4, 34.6)
- removed the REF** at (164.8, 34.5)
- removed the REF** at (220.7, 34.6)
- removed the REF** at (235.9, 34.6)
- removed the REF** at (93.7, 157.0)
- removed the REF** at (98.7, 157.0)
- removed the REF** at (114.0, 157.0)
- removed the REF** at (119.1, 157.0)
- removed the REF** at (144.5, 157.0)
- removed the REF** at (154.6, 157.0)
- removed the REF** at (301.9, 157.1)
- removed the REF** at (134.3, 157.0)
- removed the REF** at (266.4, 157.1)
- removed the REF** at (241.0, 157.1)
- removed the REF** at (220.7, 157.1)
- removed the REF** at (215.6, 157.1)
- removed the REF** at (200.3, 157.1)
- removed the REF** at (225.7, 157.1)
- removed the REF** at (205.4, 157.1)
- removed the REF** at (164.8, 157.0)
- removed the REF** at (174.9, 157.0)
- removed the REF** at (195.3, 157.0)
- removed the REF** at (307.0, 157.1)
- removed the REF** at (235.9, 157.1)
- removed the REF** at (53.0, 157.0)
- removed the REF** at (73.3, 157.0)
- removed the REF** at (83.5, 157.0)
- removed the REF** at (58.1, 157.0)
- removed the REF** at (63.2, 157.0)
- removed the REF** at (124.1, 157.0)
- removed the REF** at (42.9, 157.0)
- removed the REF** at (261.3, 157.1)
- removed the REF** at (246.1, 157.1)
- removed the REF** at (276.5, 157.1)
- removed the REF** at (78.4, 157.0)
- removed the REF** at (256.2, 157.1)
- removed the REF** at (281.6, 157.1)
- removed the REF** at (286.7, 157.1)
- removed the REF** at (296.9, 157.1)
- removed the REF** at (63.2, 34.5)
- removed the REF** at (225.7, 34.6)
- removed the REF** at (58.1, 34.5)
- removed the REF** at (139.4, 34.5)
- removed the REF** at (139.4, 157.0)
- removed the REF** at (42.9, 34.5)
- removed the REF** at (93.7, 34.5)
- removed the REF** at (241.0, 34.6)
- removed the REF** at (78.4, 34.5)
- removed the REF** at (98.7, 34.5)
- removed the REF** at (200.3, 34.6)
- removed the REF** at (103.8, 34.5)
- removed the REF** at (174.9, 34.5)
- removed the REF** at (307.0, 34.6)
- removed the REF** at (281.6, 34.6)
- removed the REF** at (286.7, 34.6)
- removed the REF** at (261.3, 34.6)
- removed the REF** at (246.1, 34.6)
- removed the REF** at (256.2, 34.6)
- removed the REF** at (195.3, 34.5)
- removed the REF** at (185.1, 157.0)
- removed the REF** at (276.5, 34.6)
- removed the REF** at (144.5, 34.5)
- removed the REF** at (159.7, 34.5)
- removed the REF** at (185.1, 34.5)
- removed the REF** at (154.6, 34.5)
- removed the REF** at (180.0, 34.5)
- removed the REF** at (134.3, 34.5)
- removed the REF** at (103.8, 157.0)
- removed the REF** at (114.0, 34.5)
- removed the REF** at (83.5, 34.5)
- removed the REF** at (53.0, 34.5)
- removed the REF** at (124.1, 34.5)
- removed the REF** at (215.6, 34.6)
- removed the REF** at (296.9, 34.6)
- removed the REF** at (119.1, 34.5)
- removed the REF** at (73.3, 34.5)
