File: MC-DSP/MC-DSP.sch (KiCad schematic (older format))
At the start: 2 parts, among them U1 TMS320F28388DZWT, U2 AMC3306M05

Commit message: updated top level of schematic with "to test" and "to do" notes
Parts:
- removed U2: AMC3306M05, symbol DSP_symbols:AMC3306M05
- added C? (x25): 0.1uF, symbol Device:C
- added R?: 56R, symbol Device:R
Connections:
- net labels added: +1V2, +3V3, GND
- wire segments 0 -> 223
Other:
- note added: "ADD JTAG connector between DSP and FTDI chip\nDSP pg 110\n"
- note added: "Add Vreg to FTDI circuit"
- note added: "Add isolated regulator\nto FTDI isolated section?"
- note added: "How to Buffer DAC outputs?\n"
- note added: "Move all power flags to be isolated"
- note added: "Place near U1"
- note added: "Seperate 5V,3V3,1V8,1V2,VDD_3V3,VDDA_3V3,VDD_1V2"
- note added: "TODO:\nADC vrefs\nADC ESD protection\nedge connecter\nFO_Enable switch\nDSP GPIO Routing"
- note added: "add pads for these for all v levels?"
- note added: "look at min loads"
- moved on the sheet: U1A, U1B, U1C, U1D, U1E, U1F, U1G, U1H

Commit message: ADC refs, FTDI changes, and more
Parts:
- added JP?: Jumper_3_Bridged12, symbol Jumper:Jumper_3_Bridged12
- added R?: 100R, symbol Device:R
- added R? (x2): 4K7, symbol Device:R
- added R? (x4): 2K2, symbol Device:R
- added R? (x3): R, symbol Device:R
- added R?: 39R, symbol Device:R
- added R?: 10K, symbol Device:R
- added R?: DNP, symbol Device:R
- added SW?: SW_SPDT, symbol Switch:SW_SPDT
- added TP1: ERRORSTS, symbol Connector:TestPoint
- added U?: conn_JTAG_14Pin, symbol DSP_symbols:conn_JTAG_14Pin
- R?: value 56R -> R
Connections:
- net labels added: +5V, -5V, ADC_14, ADC_15, ADC_A2, ADC_A3, ADC_A4, ADC_A5, ADC_B2, ADC_B3, ADC_B4, ADC_B5, ADC_C2, ADC_C3, ADC_C4, ADC_C5, ADC_D0, ADC_D1, ADC_D2, ADC_D3, CLK_Backplane, CLK_DSP, CLK_Ethernet, DPS_SCI-RX, DPS_SCI-TX, DSP_Emitter_Enable, DSP_GPIOLED1, DSP_GPIOLED2, EPWM10A, EPWM10B, EPWM11A, EPWM11B, EPWM12A, EPWM12B, EPWM1A, EPWM1B, EPWM2A, EPWM2B, EPWM3A, EPWM3B, EPWM4A, EPWM4B, EPWM5A, EPWM5B, EPWM6A, EPWM6B, EPWM7A, EPWM7B, EPWM8A, EPWM8B, EPWM9A, EPWM9B, GlobalReset, SD1_C1, SD1_C2, SD1_C3, SD1_C4, SD1_D1, SD1_D2, SD1_D3, SD1_D4, SD2_C1, SD2_C2, SD2_C3, SD2_C4, SD2_D1, SD2_D2, SD2_D3, SD2_D4, SEARAY_Emitter_Enable, VDAC
- wire segments 223 -> 365
- no-connect marks 0 -> 6
Other:
- note added: "Lines to break out to Back plane:\nAll ADC cards - 3 cards - 6 l/c - 18 lines\nAll PWM lines - \nSafe_State line\nFO_Enable line\n"
- note added: "Seperate 5V,3V3,1V8,1V2,VDD_3V3,VDDA_3V3,VDD_1V2, -5V"
- note added: "TODO HIGH-PRIORITY:\nADC vrefs\nDAC regs\nDrop ethercats, switch MMCX to BNC, breakout purple stuff to duponts (maybe GPIOs?)\nReset button\n\nTODO LOW-PRIO:\nedge connecter\nDSP GPIO Routing"
- note added: "actually calculate pulldowns to match DSP current limit\n"
- note removed: "ADD JTAG connector between DSP and FTDI chip\nDSP pg 110\n"
- note removed: "Add Vreg to FTDI circuit"
- note removed: "Add isolated regulator\nto FTDI isolated section?"
- note removed: "How to Buffer DAC outputs?\n"
- note removed: "Move all power flags to be isolated"
- note removed: "Seperate 5V,3V3,1V8,1V2,VDD_3V3,VDDA_3V3,VDD_1V2"
- note removed: "TODO:\nADC vrefs\nADC ESD protection\nedge connecter\nFO_Enable switch\nDSP GPIO Routing"
- note removed: "add pads for these for all v levels?"
- note removed: "look at min loads"
- moved on the sheet: U1A, U1B, U1F

Commit message: fixed some dsp pin routing
Connections:
- net labels added: CLK_25M_DSP, CLK_25M_Ethernet, EPWM13A, EPWM13B, EPWM14A, EPWM14B, ToBackplane
- net labels removed: CLK_Backplane, CLK_DSP, CLK_Ethernet
- wire segments 365 -> 368
Changed lines of the file:
@@
 $EndSheet
 $Sheet
-S 9500 1850 1000 1075
+S 9350 1850 1000 1075
 U 61A512C8
 F0 "25MHz Clock" 50
 F1 "MC-DSP-CLK.sch" 50
-F2 "Y0" I R 10500 2050 50
-F3 "Y1" I R 10500 2200 50
-F4 "Y2" I R 10500 2350 50
-F5 "Y3" I R 10500 2500 50
+F2 "Y0" I R 10350 2050 50
+F3 "Y1" I R 10350 2200 50
+F4 "Y2" I R 10350 2350 50
+F5 "Y3" I R 10350 2500 50
 $EndSheet
 $Sheet
@@
 NoConn ~ -2150 -1050
 Text GLabel -1900 -1150 2    50   Input ~ 0
-CLK_DSP
-Text GLabel 10500 2500 2    50   Input ~ 0
-CLK_DSP
+CLK_25M_DSP
+Text GLabel 10350 2500 2    50   Input ~ 0
+CLK_25M_DSP
 NoConn ~ -3950 -1100
 NoConn ~ -3950 -700
@@
 Text Label 16300 8550 0    50   ~ 0
 EPWM12B
-Text Label 14200 7700 2    50   ~ 0
+Text Label 16600 -300 2    50   ~ 0
 SD1_D1
-Text Label 14200 7800 2    50   ~ 0
+Text Label 16600 -400 2    50   ~ 0
 SD1_C1
-Text Label 14200 7900 2    50   ~ 0
+Text Label 14200 2550 2    50   ~ 0
 SD1_D2
-Text Label 16300 7900 0    50   ~ 0
+Text Label 14200 2650 2    50   ~ 0
 SD1_C2
 Text Label 16300 7800 0    50   ~ 0
@@
 Text Label 16300 6900 0    50   ~ 0
 SD2_C3
-Text Label 16300 6800 0    50   ~ 0
+Text Label 16300 4750 0    50   ~ 0
 SD2_D4
-Text Label 16300 6700 0    50   ~ 0
+Text Label 16300 4650 0    50   ~ 0
 SD2_C4
 Text Label -1500 200  0    50   ~ 0
@@
 Wire Wire Line
 	-2000 2300 -1150 2300
-Text GLabel 10500 2350 2    50   Input ~ 0
-CLK_Backplane
-Text GLabel 10500 2200 2    50   Input ~ 0
-CLK_Ethernet
+Text GLabel 10350 2350 2    50   Input ~ 0
+CLK_25M_Ethernet
 Wire Wire Line
 	-2000 0    -750 0
@@
 	14250 8450 13850 8450
 Wire Wire Line
-	14250 7900 13850 7900
+	13850 2550 14250 2550
 Wire Wire Line
-	14250 7800 13850 7800
+	16650 -400 16250 -400
 Wire Wire Line
-	14250 7700 13850 7700
+	16650 -300 16250 -300
 Wire Wire Line
 	16650 9350 16250 9350
@@
 	16650 8550 16250 8550
 Wire Wire Line
-	16650 7900 16250 7900
+	13850 2650 14250 2650
 Wire Wire Line
 	16650 7800 16250 7800
@@
 	16650 6900 16250 6900
 Wire Wire Line
-	16650 6800 16250 6800
-Wire Wire Line
-	16650 6700 16250 6700
+	16650 4750 16250 4750
 Wire Wire Line
-	16650 6600 16250 6600
+	16650 4650 16250 4650
 Wire Wire Line
 	16650 5900 16250 5900
@@
 	16650 6700 16750 6800
 Entry Wire Line
-	16650 6800 16750 6900
-Entry Wire Line
 	16650 6900 16750 7000
 Entry Wire Line
@@
 	16650 7800 16750 7900
 Entry Wire Line
-	16650 7900 16750 8000
-Entry Wire Line
 	16650 8550 16750 8650
 Entry Wire Line
@@
 Entry Wire Line
 	13750 8550 13850 8450
-Entry Wire Line
-	13750 8000 13850 7900
-Entry Wire Line
-	13750 7900 13850 7800
-Entry Wire Line
-	13750 7800 13850 7700
 Wire Bus Line
 	-1050 9900 13750 9900
@@
 Wire Bus Line
 	13750 9900 16750 9900
+Connection ~ 16750 9900
+Text Label 16950 9900 0    50   ~ 0
+ToBackplane
+Wire Bus Line
+	16750 9900 17500 9900
+Text Label 16300 6700 0    50   ~ 0
+EPWM13A
+Text Label 16300 6600 0    50   ~ 0
+EPWM13B
+Text Label 16300 6500 0    50   ~ 0
+EPWM14A
+Text Label 16300 6400 0    50   ~ 0
+EPWM14B
+Entry Wire Line
+	16650 6400 16750 6500
+Entry Wire Line
+	16650 6500 16750 6600
+Wire Wire Line
+	16250 6400 16650 6400
+Wire Wire Line
+	16650 6500 16250 6500
+Wire Wire Line
+	16250 6600 16650 6600
+Wire Wire Line
+	16650 6700 16250 6700
+Entry Wire Line
+	16650 4650 16750 4750
+Entry Wire Line
+	16650 4750 16750 4850
+Entry Wire Line
+	13850 2550 13750 2650
+Entry Wire Line
+	13850 2650 13750 2750
 Wire Bus Line
-	13750 7800 13750 9900
+	13750 2650 13750 9900
 Wire Bus Line
 	-1050 300  -1050 9900
 Wire Bus Line
-	16750 5600 16750 9900
-Connection ~ 16750 9900
-Wire Bus Line
-	16750 9900 17100 9900
+	16750 4750 16750 9900
 $EndSCHEMATC

Commit message: All parts labeled, just need to pick passives basically.
Parts:
- removed C? (x23): 0.1uF, symbol Device:C
- removed R? (x4): R, symbol Device:R
- removed R?: 2K2, symbol Device:R
- removed R?: 4K7, symbol Device:R
- added C172, C173, C174, C175, C176, C177, C178, C179, C180, C181, C182, C183, C184, C185, C186, C187, C188, C189, C190, C191, C192, C193, C194: 0.1uF, Capacitor_SMD:C_0201_0603Metric_Pad0.64x0.40mm_HandSolder, symbol Device:C
- added H1: Conn_02x12_Odd_Even, Connector_PinHeader_1.27mm:PinHeader_2x24_P1.27mm_Vertical, symbol Connector_Generic:Conn_02x12_Odd_Even
- added R104: 2K2, Resistor_SMD:R_0603_1608Metric_Pad0.98x0.95mm_HandSolder, symbol Device:R
- added R105: 4K7, Resistor_SMD:R_0603_1608Metric_Pad0.98x0.95mm_HandSolder, symbol Device:R
- C170, C171: renamed from C?; footprint (none) -> Capacitor_SMD:C_0201_0603Metric_Pad0.64x0.40mm_HandSolder
- JP1: renamed from JP?; footprint (none) -> Connector_PinSocket_2.54mm:PinSocket_1x03_P2.54mm_Vertical
- R100, R101: renamed from R?; value 2K2 -> 2.2K; footprint (none) -> Resistor_SMD:R_0603_1608Metric_Pad0.98x0.95mm_HandSolder
- R102, R103, R106, R107, R108, R109: renamed from R?; footprint (none) -> Resistor_SMD:R_0603_1608Metric_Pad0.98x0.95mm_HandSolder
- SW1: renamed from SW?; footprint (none) -> ?
- TP1: footprint (none) -> TestPoint:TestPoint_Pad_D1.5mm
- U2: renamed from U?; footprint (none) -> ?
Connections:
- net labels added: ADCSOCAO, ADCSOCBO, Bus_Backplane, Bus_FrontBreakout, CLB_OUTPUTX_BAR1, CLB_OUTPUTX_BAR2, CLB_OUTPUTX_BAR3, CLB_OUTPUTX_BAR4, CLB_OUTPUTX_BAR5, CLB_OUTPUTX_BAR6, CLB_OUTPUTX_BAR7, CLB_OUTPUTX_BAR8, Emitter_Enable_Backplane, Emitter_Enable_DSP, OUTPUTXBAR1, OUTPUTXBAR2, OUTPUTXBAR3, OUTPUTXBAR4, OUTPUTXBAR5, OUTPUTXBAR6, OUTPUTXBAR7, OUTPUTXBAR8, SafeState, VDDA, XCLKOUT
- net labels removed: +5V, -5V, DSP_Emitter_Enable, GlobalReset, SEARAY_Emitter_Enable, ToBackplane
- wire segments 368 -> 433
Other:
- note added: "10-19"
- note added: "20-39"
- note added: "200+"
- note added: "40-59"
- note added: "60-69"
- note added: "60-79"
- note added: "GPIO - 20mA max out\n"
- note added: "Place near U1 170-199\n"
- note added: "TODO:\nGPIO sense SafeState?\nadd more testpoints\n\nDone:\nDrop ethercats, switch MMCX to BNC\nADC vrefs\nDAC regs\nCalculate Safe_State Pull Downs\nNew 3.3V reg\nNew 1.2V reg\nNew 3.0V reg\nbreakout purple stuff to duponts (maybe GPIOs?)\nedge connecter"
- note removed: "Lines to break out to Back plane:\nAll ADC cards - 3 cards - 6 l/c - 18 lines\nAll PWM lines - \nSafe_State line\nFO_Enable line\n"
- note removed: "Place near U1"
- note removed: "Seperate 5V,3V3,1V8,1V2,VDD_3V3,VDDA_3V3,VDD_1V2, -5V"
- note removed: "TODO HIGH-PRIORITY:\nADC vrefs\nDAC regs\nDrop ethercats, switch MMCX to BNC, breakout purple stuff to duponts (maybe GPIOs?)\nReset button\n\nTODO LOW-PRIO:\nedge connecter\nDSP GPIO Routing"
- note removed: "actually calculate pulldowns to match DSP current limit\n"
- moved on the sheet: JP1, R100, R101, R102, R103, R106, R107, R108, R109, SW1, TP1, U1A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

Commit message: DSP - added footprints and links to most parts
Parts:
- removed R104: 2K2, Resistor_SMD:R_0603_1608Metric_Pad0.98x0.95mm_HandSolder, symbol Device:R
- removed U2: conn_JTAG_14Pin, ?, symbol DSP_symbols:conn_JTAG_14Pin
- added U2: SBH41-NBPB-D10-ST-BK, mark_footprints:SBH41-NBPB-D10-ST-BK, symbol Connector_Generic:Conn_02x10_Odd_Even
- R100, R101: value 2.2K -> 2K2
- SW1: footprint ? -> mark_footprints:GT12MABE
Connections:
- net +3V3: now also R105.1; no longer R105.2
- net GND: now also U2.10 (Pin_10), U2.12 (Pin_12), U2.16 (Pin_16), U2.17 (Pin_17), U2.18 (Pin_18), U2.19 (Pin_19), U2.20 (Pin_20), U2.4 (Pin_4), U2.8 (Pin_8)
- net EMU0: now reaches R103.1
- net EMU0: now also U2.13 (Pin_13)
- net PD: now reaches R102.1
- net PD: now also U2.5 (Pin_5)
- net FTDI/DSP_TCK renamed RTCK
- net RTCK: now also U2.11 (Pin_11), U2.9 (Pin_9)
- net FTDI/DSP_TDI renamed TDI
- net TDI: now also U2.3 (Pin_3)
- net FTDI/DSP_TDO renamed TDO
- net TDO: now also U2.7 (Pin_7)
- net FTDI/DSP_TMS renamed TMS
- net TMS: now also U2.1 (Pin_1)
- net FTDI/DSP_TRSTn renamed NSRST
- net NSRST: now also U2.15 (Pin_15), U2.2 (Pin_2)
- net SafeState renamed Safe_State
- new net EMU1: R105.2, U2.14 (Pin_14)
Other:
- note added: "80-89\n"
- note added: "TODO:\nGPIO sense SafeState?\nadd more testpoints\npick dsp gpio LEDs\n\nDone:\nDrop ethercats, switch MMCX to BNC\nADC vrefs\nDAC regs\nCalculate Safe_State Pull Downs\nNew 3.3V reg\nNew 1.2V reg\nNew 3.0V reg\nbreakout purple stuff to duponts (maybe GPIOs?)\nedge connecter"
- note removed: "60-69"
- note removed: "TODO:\nGPIO sense SafeState?\nadd more testpoints\n\nDone:\nDrop ethercats, switch MMCX to BNC\nADC vrefs\nDAC regs\nCalculate Safe_State Pull Downs\nNew 3.3V reg\nNew 1.2V reg\nNew 3.0V reg\nbreakout purple stuff to duponts (maybe GPIOs?)\nedge connecter"
- moved on the sheet: R102, R103, R105, R106

Commit message: Removed clock buffer, misc leds, ethernet
Parts:
- added U?: ECS-2520MV-xxx-xx, Oscillator:Oscillator_SMD_ECS_2520MV-xxx-xx-4Pin_2.5x2.0mm, symbol Oscillator:ECS-2520MV-xxx-xx
- C170, C171, C172, C173, C174, C175, C176, C177, C178, C179, C180, C181, C182, C183, C184, C185, C186, C187, C188, C189, C190, C191, C192, C193, C194: footprint Capacitor_SMD:C_0201_0603Metric_Pad0.64x0.40mm_HandSolder -> Capacitor_SMD:C_0603_1608Metric_Pad1.08x0.95mm_HandSolder
- H1: footprint Connector_PinHeader_1.27mm:PinHeader_2x24_P1.27mm_Vertical -> Connector_PinHeader_1.27mm:PinHeader_2x12_P1.27mm_Vertical
Connections:
- net +3V3: now also U?.4 (VDD)
- net GND: now also U?.2 (GND)
- net CLK_25M_DSP renamed 25MHz_clk_DSP
- net 25MHz_clk_DSP: now also U?.3 (OUT)
- net Ethernet/COL: no longer names the net of U1.M2 (GPIO110)
- net Ethernet/CRS: no longer names the net of U1.N2 (GPIO109)
- net Ethernet/MDC: no longer names the net of U1.J3 (GPIO105)
- net Ethernet/MDIO: no longer names the net of U1.L2 (GPIO106)
- net Ethernet/PWDN: no longer names the net of U1.L4 (GPIO108)
- net Ethernet/RX_CLK: no longer names the net of U1.M4 (GPIO111)
- net Ethernet/RX_D0: no longer names the net of U1.N3 (GPIO114)
- net Ethernet/RX_D1: no longer names the net of U1.V12 (GPIO115)
- net Ethernet/RX_D2: no longer names the net of U1.W10 (GPIO116)
- net Ethernet/RX_D3: no longer names the net of U1.U12 (GPIO117)
- net Ethernet/RX_DV: no longer names the net of U1.M3 (GPIO112)
- net Ethernet/RX_ER: no longer names the net of U1.N4 (GPIO113)
- net Ethernet/Reset: no longer names the net of U1.T15 (GPIO119)
- net Ethernet/TX_CLK: no longer names the net of U1.U15 (GPIO120)
- net Ethernet/TX_D0: no longer names the net of U1.W16 (GPIO121)
- net Ethernet/TX_D1: no longer names the net of U1.T8 (GPIO122)
- net Ethernet/TX_D2: no longer names the net of U1.U8 (GPIO123)
- net Ethernet/TX_D3: no longer names the net of U1.V8 (GPIO124)
- net Ethernet/TX_EN: no longer names the net of U1.T12 (GPIO118)
- no-connect marks 6 -> 7
Other:
- note added: "TODO:\nGPIO sense SafeState?\nadd more testpoints\npick dsp gpio LEDs\nFix 12 Mhz clock\nfix clock buffer\n\n\n\nDone:\ndropped ethernet\nDrop ethercats, switch MMCX to BNC\nADC vrefs\nDAC regs\nCalculate Safe_State Pull Downs\nNew 3.3V reg\nNew 1.2V reg\nNew 3.0V reg\nbreakout purple stuff to duponts (maybe GPIOs?)\nedge connecter"
- note removed: "40-59"
- note removed: "TODO:\nGPIO sense SafeState?\nadd more testpoints\npick dsp gpio LEDs\n\nDone:\nDrop ethercats, switch MMCX to BNC\nADC vrefs\nDAC regs\nCalculate Safe_State Pull Downs\nNew 3.3V reg\nNew 1.2V reg\nNew 3.0V reg\nbreakout purple stuff to duponts (maybe GPIOs?)\nedge connecter"

Commit message: added backplane connector, changed right angle headers, added FP for bigger reg caps, all ICs arranged, routed isolated section.
Parts:
- removed H1: Conn_02x12_Odd_Even, Connector_PinHeader_1.27mm:PinHeader_2x12_P1.27mm_Vertical, symbol Connector_Generic:Conn_02x12_Odd_Even
- added C13: 0.1uF, Capacitor_SMD:C_0603_1608Metric_Pad1.08x0.95mm_HandSolder, symbol Device:C
- added D10: WP1384AD/RD, LED_THT:LED_D3.0mm, symbol Device:LED
- added H1, H2, H3: Conn_01x05, Connector_PinSocket_2.54mm:PinSocket_1x05_P2.54mm_Vertical, symbol Connector_Generic:Conn_01x05
- added J1: 374385, 374385:374385, symbol 374385:374385
- added R10: 1K, Resistor_SMD:R_0603_1608Metric_Pad0.98x0.95mm_HandSolder, symbol Device:R_Small_US
- gave numbers to parts that had none: 1
- renumbered TP1 to T1
Connections:
- net +3V3: now also C13.2, R10.1
- net ADCSOCAO: now also H3.4 (Pin_4)
- net ADCSOCBO: now also H3.5 (Pin_5)
- net CLB_OUTPUTX_BAR1: now also H2.1 (Pin_1)
- net CLB_OUTPUTX_BAR2: now also H2.2 (Pin_2)
- net CLB_OUTPUTX_BAR3: now also H2.4 (Pin_4)
- net CLB_OUTPUTX_BAR4: now also H2.5 (Pin_5)
- net GND: now also C13.1, H1.3 (Pin_3), H2.3 (Pin_3), H3.2 (Pin_2), H3.3 (Pin_3)
- net OUTPUTXBAR1: now also H1.1 (Pin_1)
- net OUTPUTXBAR2: now also H1.2 (Pin_2)
- net OUTPUTXBAR3: now also H1.4 (Pin_4)
- net OUTPUTXBAR4: now also H1.5 (Pin_5)
- net Safe_State: now also D10.1 (K)
- net XCLKOUT: now also H3.1 (Pin_1)
- new net: D10.2 (A), R10.2
Other:
- note added: "TODO:\n\nSTRECH:\nadd more testpoints\nFix isolators\nfix USB protection\n\nBUY:\nnew C21,22,28\nright angle header\nbackplane connector\nisolators\nUSB protection\n\nDONE:\ndropped ethernet\nDrop ethercats, switch MMCX to BNC\nADC vrefs\nDAC regs\nCalculate Safe_State Pull Downs\nNew 3.3V reg\nNew 1.2V reg\nNew 3.0V reg\nbreakout purple stuff to duponts (maybe GPIOs?)\nedge connecter\nFix 12 Mhz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"
- note removed: "TODO:\nGPIO sense SafeState?\nadd more testpoints\npick dsp gpio LEDs\nFix 12 Mhz clock\nfix clock buffer\n\n\n\nDone:\ndropped ethernet\nDrop ethercats, switch MMCX to BNC\nADC vrefs\nDAC regs\nCalculate Safe_State Pull Downs\nNew 3.3V reg\nNew 1.2V reg\nNew 3.0V reg\nbreakout purple stuff to duponts (maybe GPIOs?)\nedge connecter"

Commit message: connected DSP signals to BP connector symbol, routed most non-signal traces on PCB
Parts:
- removed J1: 374385, 374385:374385, symbol 374385:374385
- JP1: value Jumper_3_Bridged12 -> EE_Switch
Connections:
- net Emitter_Enable_DSP is gone; now on net +3V3: JP1.1 (A)
- net +3V3: no longer JP1.3 (B)
- net at U1.C2 (GPIO12): now also JP1.3 (B)
- net GPIO14: now reaches U1.D2 (GPIO14)
- net GPIO15: now reaches U1.D3 (GPIO15)
- net GPIO16: now reaches U1.E1 (GPIO16)
- net GPIO18: now reaches U1.E3 (GPIO18)
- net GPIO19: now reaches U1.E4 (GPIO19)
- net GPIO22: now reaches U1.J4 (GPIO22)
- net GPIO44: now reaches U1.K18 (GPIO44)
- net GPIO45: now reaches U1.K19 (GPIO45)
- net GPIO25: now reaches U1.K2 (GPIO25)
- net GPIO24: now reaches U1.K3 (GPIO24)
- net GPIO23: now reaches U1.K4 (GPIO23)
- net GPIO52: now reaches U1.P16 (GPIO52)
- net GPIO53: now reaches U1.P17 (GPIO53)
- net Emitter_Enable_Backplane renamed Emitter_Enable
Other:
- note removed: "GPIO - 20mA max out\n"
- moved on the sheet: C170, C171, C172, C173, C174, C175, C176, C177, C178, C179, C180, C181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
