File: MC-DSP/MC-DSP.sch (KiCad schematic (older format))
At the start: 46 parts, among them SW1 SW_SPDT, T1 ERRORSTS, U1 TMS320F28388DZWT, U10 ECS-2520MV-xxx-xx, U2 SBH41-NBPB-D10-ST-BK

Commit message: Total overhaul of power planes. Routed whole Analog section, middle of digital section.
Parts:
- removed C176, C192, C193, C194: 0.1uF, Capacitor_SMD:C_0603_1608Metric_Pad1.08x0.95mm_HandSolder, symbol Device:C
- C170, C171, C172, C173, C174, C175, C177, C178, C179, C180, C181, C182, C183, C184, C185, C186, C187, C188, C189, C190, C191: footprint Capacitor_SMD:C_0603_1608Metric_Pad1.08x0.95mm_HandSolder -> Capacitor_SMD:C_0402_1005Metric_Pad0.74x0.62mm_HandSolder
Connections:
- net +3V3: no longer C179.2, C180.2, C181.2, C182.2, C183.2, C184.2, C185.2, C186.2, C187.2, C188.2, C189.2, C190.2, C191.2, U1.A18 (VDDIO_A18), U1.A9 (VDDIO_A9), U1.B1 (VDDIO_B1), U1.E10 (VDDIO_E10), U1.E13 (VDDIO_E13), U1.E16 (VDDIO_E16), U1.E7 (VDDIO_E7), U1.F10 (VDDIO_F10), U1.F13 (VDDIO_F13), U1.F16 (VDDIO_F16), U1.F4 (VDDIO_F4), U1.F7 (VDDIO_F7), U1.G4 (VDDIO_G4), U1.G5 (VDDIO_G5), U1.G6 (VDDIO_G6), U1.H16 (VDDOSC_H16), U1.H17 (VDDOSC_H17), U1.H5 (VDDIO_H5), U1.H6 (VDDIO_H6), U1.L14 (VDDIO_L14), U1.L15 (VDDIO_L15), U1.M1 (VDDIO_M1), U1.M5 (VDDIO_M5), U1.M6 (VDDIO_M6), U1.N14 (VDDIO_N14), U1.N15 (VDDIO_N15), U1.P6 (VDDA), U1.P9 (VDDIO_P9), U1.R11 (VDD3VFL_R11), U1.R12 (VDD3VFL_R12), U1.R6 (VDDA), U1.R9 (VDDIO_R9), U1.V19 (VDDIO_V19), U1.W8 (VDDIO_W8)
- net VDD: now also C179.2, C180.2, C181.2, C182.2, C183.2, C184.2, C185.2, C186.2, C187.2, C188.2, C189.2, C190.2, C191.2, U1.A18 (VDDIO_A18), U1.A9 (VDDIO_A9), U1.B1 (VDDIO_B1), U1.E10 (VDDIO_E10), U1.E13 (VDDIO_E13), U1.E16 (VDDIO_E16), U1.E7 (VDDIO_E7), U1.F10 (VDDIO_F10), U1.F13 (VDDIO_F13), U1.F16 (VDDIO_F16), U1.F4 (VDDIO_F4), U1.F7 (VDDIO_F7), U1.G4 (VDDIO_G4), U1.G5 (VDDIO_G5), U1.G6 (VDDIO_G6), U1.H16 (VDDOSC_H16), U1.H17 (VDDOSC_H17), U1.H5 (VDDIO_H5), U1.H6 (VDDIO_H6), U1.L14 (VDDIO_L14), U1.L15 (VDDIO_L15), U1.M1 (VDDIO_M1), U1.M5 (VDDIO_M5), U1.M6 (VDDIO_M6), U1.N14 (VDDIO_N14), U1.N15 (VDDIO_N15), U1.P9 (VDDIO_P9), U1.R11 (VDD3VFL_R11), U1.R12 (VDD3VFL_R12), U1.R9 (VDDIO_R9), U1.V19 (VDDIO_V19), U1.W8 (VDDIO_W8)
- net VDDA: now also U1.P6 (VDDA), U1.R6 (VDDA)
Other:
- note added: "TODO:\n\nSTRECH:\nadd more testpoints\nFix isolators\nfix USB protection\n0402 CAPs\n\n\nZach order:\nright angle header\nC218\nisolators\n\nBUY:\nnew C21,22,28\nbackplane connector\nUSB protection\n\nDONE:\ndropped ethernet\nDrop ethercats, switch MMCX to BNC\nADC vrefs\nDAC regs\nCalculate Safe_State Pull Downs\nNew 3.3V reg\nNew 1.2V reg\nNew 3.0V reg\nbreakout purple stuff to duponts (maybe G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"
- note added: "Unused:"
- note removed: "TODO:\n\nSTRECH:\nadd more testpoints\nFix isolators\nfix USB protection\n\nBUY:\nnew C21,22,28\nright angle header\nbackplane connector\nisolators\nUSB protection\n\nDONE:\ndropped ethernet\nDrop ethercats, switch MMCX to BNC\nADC vrefs\nDAC regs\nCalculate Safe_State Pull Downs\nNew 3.3V reg\nNew 1.2V reg\nNew 3.0V reg\nbreakout purple stuff to duponts (maybe GPIOs?)\nedge connecter\nFix 12 Mhz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"
